Commit message: Separating out simulation

File: husky_description/urdf/base.urdf.xacro (robot description, xacro)
@@ -1,5 +1,5 @@
 <?xml version="1.0"?>
 <!--
-Copyright (c) 2012, Siddhant Ahuja (Sid), Ryan Gariepy
+Copyright (c) 2012, Ryan Gariepy/Clearpath Robotics
 All rights reserved.
 Redistribution and use in source and binary forms, with or without
@@ -158,5 +158,5 @@
     </gazebo>
     <gazebo>
-		<controller:husky_plugin name="husky_diff_controller" plugin="libhusky_description.so">
+		<controller:husky_plugin name="husky_diff_controller" plugin="libhusky_gazebo_plugins.so">
 		        <alwaysOn>true</alwaysOn>
 		        <updateRate>100.0</updateRate>

File: husky_description/urdf/base.urdf_prefuerte.xacro (robot description, xacro)
@@ -1,5 +1,5 @@
 <?xml version="1.0"?>
 <!--
-Copyright (c) 2012, Siddhant Ahuja (Sid), Ryan Gariepy
+Copyright (c) 2012, Siddhant Ahuja/WAVELab, Ryan Gariepy/Clearpath Robotics
 All rights reserved.
 Redistribution and use in source and binary forms, with or without

File: husky_description/urdf/wheel.urdf.xacro (robot description, xacro)
@@ -1,5 +1,5 @@
 <?xml version="1.0"?>
 <!--
-Copyright (c) 2012, Siddhant Ahuja (Sid)
+Copyright (c) 2012, Siddhant Ahuja/WAVELab, Ryan Gariepy/Clearpath Robotics
 All rights reserved.
 Redistribution and use in source and binary forms, with or without
@@ -64,14 +64,17 @@
 			</visual>
 			<collision>
-				<origin xyz="0 0 0" rpy="${flipY*M_PI} 0 0" />
+				<origin xyz="0 0 0" rpy="${flipY*M_PI/2} 0 0" />
 				<geometry>
+				    <cylinder length="${wheel_z_size}" radius="${wheel_x_size/2}" />
+				<!--
 					<mesh filename="package://husky_description/Media/models/wheel.stl" />
+			    -->
 				</geometry>
 			</collision>
 		</link>
 		<gazebo reference="${fb}_${lr}_wheel">
-			<mu1 value="75.0"/>
-			<mu2 value="1.5"/>
-			<kp  value="1000000.0" />
+			<mu1 value="1.0"/>
+			<mu2 value="1.0"/>
+			<kp  value="100000.0" />
 			<kd  value="1.0" />
 			<fdir1 value="1 0 0"/>

Commit message: Moving SDF back into husky_description

File: husky_description/urdf/base.urdf.xacro (robot description, xacro)
@@ -105,5 +105,5 @@
             <origin xyz="0 0 ${base_z_origin_offset}" rpy="0 0 0" />
             <geometry>
-                <mesh filename="package://husky_description/Media/models/base_link.stl" />
+                <mesh filename="package://husky_description/models/husky/meshes/base_link.stl" />
             </geometry>
             <material name="Black" />

File: husky_description/urdf/parts.urdf.xacro (robot description, xacro)
@@ -62,5 +62,5 @@
 				<origin xyz="0 0 0" rpy="0 0 0" />
 				<geometry>
-					<mesh filename="package://husky_description/Media/models/${mesh}.stl" />
+					<mesh filename="package://husky_description/models/husky/meshes/${mesh}.stl" />
 				</geometry>
 				<material name="${colour}" />

File: husky_description/urdf/wheel.urdf.xacro (robot description, xacro)
@@ -59,5 +59,5 @@
 				<origin xyz="0 0 0" rpy="${flipY*M_PI} 0 0" />
 				<geometry>
-					<mesh filename="package://husky_description/Media/models/wheel.stl" />
+					<mesh filename="package://husky_description/models/husky/meshes/wheel.stl" />
 				</geometry>
 				<material name="DarkGray" />
@@ -67,7 +67,4 @@
 				<geometry>
 				    <cylinder length="${wheel_z_size}" radius="${wheel_x_size/2}" />
-				<!--
-					<mesh filename="package://husky_description/Media/models/wheel.stl" />
-			    -->
 				</geometry>
 			</collision>
