Commit message: Add effort limit to wheel joint

File: husky_description/urdf/wheel.urdf.xacro (robot description, xacro)
@@ -69,4 +69,5 @@
 	      <xacro:insert_block name="joint_pose"/>
 	      <axis xyz="0 1 0" rpy="0 0 0" />
+        <limit effort="100" velocity="100"/>
 	    </joint>
 	    <transmission name="${wheel_prefix}_wheel_trans" type="SimpleTransmission">
