Commit message: Added left and right arm for dual config, no positions yet, no top plate mod yet

File: husky_description/urdf/description.xacro (robot description, xacro)
@@ -22,4 +22,5 @@
 -->
 <robot name="husky" xmlns:xacro="http://ros.org/wiki/xacro">
+  <xacro:arg name="dual_ur5_enabled" default="false" />
   <xacro:arg name="laser_enabled" default="false" />
   <xacro:arg name="ur5_enabled" default="false" />

File: husky_description/urdf/husky.urdf.xacro (robot description, xacro)
@@ -107,4 +107,20 @@
     </xacro:husky_wheel>
     <xacro:husky_decorate />
+    <xacro:if value="$(arg dual_ur5_enabled)">
+        <xacro:ur5_robot prefix="l_ur5_arm_" joint_limited="true"/>
+        <xacro:ur5_robot prefix="r_ur5_arm_" joint_limited="true"/>
+        <!-- Join left arm to top plate -->
+        <joint name="l_ur5_arm_base" type="fixed"/>
+            <parent link="modified_top_plate_link"/>
+            <child link="l_ur5_arm_base_link" />
+            <origin xyz="0 0 0" rpy="0 0 0"/>
+        </joint>
+         <!-- Joint right arm to top plate -->
+        <joint name="r_ur5_arm_base" type="fixed">
+            <parent link="modified_top_plate_link"/>
+            <child link="r_ur5_arm_base_link" />
+            <origin xyz="0 0 0" rpy="0 0 0"/>
+        </joint>
+    </xacro>
     <xacro:if value="$(arg ur5_enabled)">
       <xacro:property name="reflect" value="-1" />

Commit message: Added robotiq grippers to dual husky

File: husky_description/urdf/description.xacro (robot description, xacro)
@@ -26,4 +26,5 @@
   <xacro:arg name="ur5_enabled" default="false" />
   <xacro:arg name="kinect_enabled" default="false" />
+  <xacro:arg name="robotiq_grippers_enabled" default="false" />
   <xacro:include filename="$(find husky_description)/urdf/husky.urdf.xacro" />
   <xacro:husky_robot />

File: husky_description/urdf/husky.urdf.xacro (robot description, xacro)
@@ -110,4 +110,21 @@
         <xacro:ur5_robot prefix="l_ur5_arm_" joint_limited="true"/>
         <xacro:ur5_robot prefix="r_ur5_arm_" joint_limited="true"/>
+        <xacro:if value="$(arg robotiq_grippers_enabled)">
+            <xacro:include filename="$(find robotiq_s_model_visualization)/cfg/s-model_articulated_macro.xacro"/>
+            <!-- Left gripper -->
+            <xacro:s-model_articulated prefix="l_"/>
+            <joint name="l_palm_to_l_ur5" type="fixed"/>
+                <parent link="l_ur5_arm_ee_link"/>
+                <child link="l_palm"/>
+                <origin xyz="0 0 0" rpy="0 0 0"/>
+            </joint>
+            <!-- Right gripper -->
+            <xacro:s-model_articulated prefix="r_"/>
+            <joint name="r_palm_to_r_ur5" type="fixed"/>
+                <parent link="r_ur5_arm_ee_link"/>
+                <child link="r_palm"/>
+                <origin xyz="0 0 0" rpy="0 0 0"/>
+            </joint>
+        </xacro:if>
         <!-- Join left arm to top plate -->
         <joint name="l_ur5_arm_base" type="fixed"/>
