Commit message: Added new package with corrected urdf

File: husky_description/urdf/dual_arm_husky.urdf (robot description, URDF)
Before this commit: robot husky, 126 links, 125 joints
Joints:
- joint bumblebee2_mount_joint: origin xyz=-0.07 0.02 -0.13 rpy=0 1.57 0 -> xyz=-0.079 0.02 -0.10 rpy=3.14 1.57 0

Commit message: Generate URDF (old was out of date)

File: husky_description/urdf/dual_arm_husky.urdf (robot description, URDF)
Before this commit: robot husky, 126 links, 125 joints
Joints:
- joint bumblebee2_mount_joint: origin xyz=-0.079 0.02 -0.10 rpy=3.14 1.57 0 -> xyz=0 0 0.00 rpy=0 0 0
- joint husky_ptu_joint: origin xyz=0.365 0 0.221 rpy=0 1.57 3.14 -> xyz=0.365 0 0.221 rpy=0 0 0
- joint l_robotiq_hand_joint: origin xyz=0 0 0 rpy=1.57 0 0 -> xyz=0 0 0.08 rpy=1.57 0 0
- joint r_robotiq_hand_joint: origin xyz=0 0 0 rpy=1.57 0 0 -> xyz=0 0 0.08 rpy=1.57 0 0

Commit message: Update URDF

File: husky_description/urdf/dual_arm_husky.urdf (robot description, URDF)
Before this commit: robot husky, 126 links, 125 joints
Joints:
- joint husky_ptu_joint: origin xyz=0.365 0 0.221 rpy=0 0 0 -> xyz=0.365 0 0.19876 rpy=0 0 0
- joint l_robotiq_hand_joint: origin xyz=0 0 0.08 rpy=1.57 0 0 -> xyz=0 0 0.05398 rpy=1.57 0 0
- joint r_robotiq_hand_joint: origin xyz=0 0 0.08 rpy=1.57 0 0 -> xyz=0 0 0.05398 rpy=1.57 0 0
