Commit message: Fix PTU to Bulkhead joint z-offset (read from CAD model)

File: husky_description/urdf/dual_arm_husky.urdf.xacro (robot description, xacro)
@@ -480,5 +480,5 @@
   <!-- Connect PTU to Husky bulkhead -->
   <joint name="husky_ptu_joint" type="fixed">
-    <origin rpy="0 0 0" xyz="0.365 0 0.221"/>
+    <origin rpy="0 0 0" xyz="0.365 0 0.19876"/>
     <parent link="dual_arm_bulkhead_link"/>
     <child link="husky_ptu_base_link"/>

Commit message: Fix Robotiq hand attachment z-offset (read from palm CAD model)

File: husky_description/urdf/dual_arm_husky.urdf.xacro (robot description, xacro)
@@ -1266,5 +1266,5 @@
   <!-- joint attaching parent link to robotiq hand -->
   <joint name="l_robotiq_hand_joint" type="fixed">
-    <origin rpy="1.57 0 0" xyz="0 0 0.08"/>
+    <origin rpy="1.57 0 0" xyz="0 0 0.05398"/>
     <parent link="l_robotiq_fts300_fts_toolside"/>
     <child link="l_palm"/>
@@ -3034,5 +3034,5 @@
   <!-- joint attaching parent link to robotiq hand -->
   <joint name="r_robotiq_hand_joint" type="fixed">
-    <origin rpy="1.57 0 0" xyz="0 0 0.08"/>
+    <origin rpy="1.57 0 0" xyz="0 0 0.05398"/>
     <parent link="r_robotiq_fts300_fts_toolside"/>
     <child link="r_palm"/>

Commit message: Update inertial link based on information provided by Clearpath support

File: husky_description/urdf/dual_arm_husky.urdf.xacro (robot description, xacro)
@@ -96,7 +96,7 @@
   <link name="inertial_link">
     <inertial>
-      <mass value="33.455"/>
-      <origin xyz="-0.08748 -0.00085 0.09947"/>
-      <inertia ixx="0.6022" ixy="-0.02364" ixz="-0.1197" iyy="1.7386" iyz="-0.001544" izz="2.0296"/>
+      <mass value="48.39054"/>
+      <origin xyz="-0.0648 -0.00059 0.07895"/>
+      <inertia ixx="2.1634275613800003" ixy="-0.055452352110000006" ixz="-0.41083822026" iyy="3.5314689495400002" iyz="-0.004366145530000001" izz="4.4759585875" />
     </inertial>
   </link>

Commit message: Fix gripper mounting orientation approximately Old orientation was off, calibrated visualisation vs real robot approximately to match

File: husky_description/urdf/dual_arm_husky.urdf.xacro (robot description, xacro)
@@ -1266,5 +1266,5 @@
   <!-- joint attaching parent link to robotiq hand -->
   <joint name="l_robotiq_hand_joint" type="fixed">
-    <origin rpy="1.57 0 0" xyz="0 0 0.05398"/>
+    <origin rpy="1.57 0 1.0" xyz="0 0 0.05398"/>
     <parent link="l_robotiq_fts300_fts_toolside"/>
     <child link="l_palm"/>
@@ -3034,5 +3034,5 @@
   <!-- joint attaching parent link to robotiq hand -->
   <joint name="r_robotiq_hand_joint" type="fixed">
-    <origin rpy="1.57 0 0" xyz="0 0 0.05398"/>
+    <origin rpy="1.57 0 2.355" xyz="0 0 0.05398"/>
     <parent link="r_robotiq_fts300_fts_toolside"/>
     <child link="r_palm"/>

Commit message: Fix IMU rotation

File: husky_description/urdf/dual_arm_husky.urdf.xacro (robot description, xacro)
@@ -110,5 +110,6 @@
   <link name="imu_link"/>
   <joint name="imu_joint" type="fixed">
-    <origin rpy="0 -1.5708 3.1416" xyz="0.19 0 0.149"/>
+    <!-- <origin xyz="$(optenv HUSKY_IMU_XYZ 0.19 0 0.149)" rpy="$(optenv HUSKY_IMU_RPY 0 -1.5708 3.1416)" /> -->
+    <origin rpy="-1.5708 0 0" xyz="0.19 0 0.149"/>
     <parent link="base_link"/>
     <child link="imu_link"/>

Commit message: Fix bumblebee2 mount joint z-offset

File: husky_description/urdf/dual_arm_husky.urdf.xacro (robot description, xacro)
@@ -1178,5 +1178,5 @@
   </gazebo>
   <joint name="bumblebee2_mount_joint" type="fixed">
-    <origin rpy="0 0 0" xyz="0 0 0.00"/>
+    <origin rpy="0 0 0" xyz="0 0 0.02224"/>
     <parent link="husky_ptu_mount_link"/>
     <child link="bumblebee2"/>

Commit message: Fix husky_ptu_joint x and y translation. The y translation was taken from the FLIR PTU E46 data sheet and also confirmed via self-observation point clouds. The x translation is guesstimated based on photographs and point cloud self-observation since I'm currently not in the lab. It is much better now and can be seen from the screw locations for the SICK mount for instance.

File: husky_description/urdf/dual_arm_husky.urdf.xacro (robot description, xacro)
@@ -481,5 +481,5 @@
   <!-- Connect PTU to Husky bulkhead -->
   <joint name="husky_ptu_joint" type="fixed">
-    <origin rpy="0 0 0" xyz="0.365 0 0.19876"/>
+    <origin rpy="0 0 0" xyz="0.345 0.010414 0.19876"/><!-- x-translation still needs to be measured -->
     <parent link="dual_arm_bulkhead_link"/>
     <child link="husky_ptu_base_link"/>
