Commit message: Remove the unnecessary args from wherever we include description.launch, add the extra extrusions the integration team uses to mount the VLP16 high enough to avoid "seeing" the sensor arch. Refactor some of the new env var names so they're more consistently-named

File: husky_description/urdf/accessories.urdf.xacro (robot description, xacro)
@@ -4,5 +4,5 @@
   <xacro:include filename="$(find husky_description)/urdf/accessories/intel_realsense.urdf.xacro"/>
   <xacro:include filename="$(find husky_description)/urdf/accessories/sick_lms1xx_mount.urdf.xacro"/>
-  <xacro:include filename="$(find velodyne_description)/urdf/VLP-16.urdf.xacro" />
+  <xacro:include filename="$(find husky_description)/urdf/accessories/vlp16_mount.urdf.xacro"/>
   <xacro:if value="$(optenv HUSKY_LASER 0)">
     <xacro:property name="lidar_model" value="$(optenv HUSKY_LASER_MODEL lms1xx)" />
@@ -31,10 +31,12 @@
   <xacro:if value="$(optenv HUSKY_LASER_3D 0)">
     <xacro:property name="lidar_3d_model" value="$(optenv HUSKY_LASER_3D_MODEL vlp16)" />
-    <xacro:VLP-16 parent="sensor_arch_mount_link" topic="$(optenv HUSKY_LASER_3D_TOPIC ponts)">
-      <origin xyz="$(optenv HUSKY_LASER_3D_OFFSET 0 0 0)" rpy="$(optenv HUSKY_LASER_3D_RPY 0 0 0)" />
-    </xacro:VLP-16>
+    <xacro:if value="${lidar_3d_model == 'vlp16'}">
+      <xacro:vlp16_mount prefix="vlp16" topic="$(optenv HUSKY_LASER_3D_TOPIC points)" parent_link="sensor_arch_mount_link">
+        <origin xyz="$(optenv HUSKY_LASER_3D_OFFSET 0 0 0)" rpy="$(optenv HUSKY_LASER_3D_RPY 0 0 0)" />
+      </xacro:vlp16_mount>
+    </xacro:if>
   </xacro:if>
   <!-- add the intel realsense to the topbar if needed -->
-  <xacro:if value="$(arg realsense_enabled)">
+  <xacro:if value="$(optenv HUSKY_REALSENSE 0)">
     <link name="realsense_mountpoint"/>
     <joint name="realsense_mountpoint_joint" type="fixed">

File: husky_description/urdf/decorations.urdf.xacro (robot description, xacro)
@@ -191,5 +191,5 @@
       <link name="top_plate_rear_link"/>
     </xacro:if>
-    <xacro:if value="$(optenv HUSKY_SENSOR_BAR_ENABLED 0)">
+    <xacro:if value="$(optenv HUSKY_SENSOR_ARCH 0)">
       <xacro:include filename="$(find husky_description)/urdf/accessories/sensor_arch.urdf.xacro"/>
       <xacro:sensor_arch prefix="" parent="top_plate_link">

Commit message: Overhaul the husky_bringup package so it installs an accessories.launch file, which selectively includes the *_config/*.launch files, as the old install script would have. Add launch files for the VLP16, modify the LMS1xx to accept parameters for front/rear. Change the HUSKY_LASER_TOPIC to front/scan by default. Update more launch files to get rid of the deleted arguments for description.launch

File: husky_description/urdf/accessories.urdf.xacro (robot description, xacro)
@@ -1,2 +1,3 @@
+<?xml version="1.0"?>
 <robot xmlns:xacro="http://wiki.ros.org/xacro">
   <xacro:arg name="robot_namespace" default="$(optenv HUSKY_NAMESPACE /" />
@@ -8,10 +9,10 @@
     <xacro:property name="lidar_model" value="$(optenv HUSKY_LASER_MODEL lms1xx)" />
     <xacro:if value="${lidar_model == 'lms1xx'}">
-      <sick_lms1xx_mount prefix="base"/>
-      <sick_lms1xx frame="base_laser" topic="scan" robot_namespace="$(arg robot_namespace)"/>
+      <sick_lms1xx_mount prefix="front"/>
+      <sick_lms1xx frame="front_laser" topic="$(optenv HUSKY_LASER_TOPIC front/scan)" robot_namespace="$(arg robot_namespace)"/>
       <joint name="laser_mount_joint" type="fixed">
         <origin xyz="$(optenv HUSKY_LASER_OFFSET 0.2206 0.0 0.00635)" rpy="$(optenv HUSKY_LASER_RPY 0 0 0)" />
         <parent link="top_plate_link" />
-        <child link="base_laser_mount" />
+        <child link="front_laser_mount" />
       </joint>
     </xacro:if>
@@ -21,5 +22,5 @@
     <xacro:if value="${lidar2_model == 'lms1xx'}">
       <sick_lms1xx_mount prefix="rear"/>
-      <sick_lms1xx frame="rear_laser" topic="rear/scan" robot_namespace="$(arg robot_namespace)"/>
+      <sick_lms1xx frame="rear_laser" topic="$(optenv HUSKY_LASER_SECONDARY_TOPIC rear/scan)" robot_namespace="$(arg robot_namespace)"/>
       <joint name="secondary_laser_mount_joint" type="fixed">
         <origin xyz="$(optenv HUSKY_LASER_SECONDARY_OFFSET -0.2206 0.0 0.00635)" rpy="$(optenv HUSKY_LASER_RPY 0 0 ${M_PI})" />
