Commit message: Added bulkhead as param

File: husky_description/urdf/decorations.urdf.xacro (robot description, xacro)
@@ -79,4 +79,27 @@
       <child link="rear_bumper_link" />
     </joint>
+    <xacro:if value="$(optenv DUAL_ARM_BULKHEAD true)">
+        <!-- Spawn the bulkhead -->
+        <link name="dual_arm_bulkhead_link">
+        <visual>
+          <origin xyz="0 0 0" rpy="0 0 0" />
+          <geometry>
+            <mesh filename="package://husky_description/meshes/dual_arm_bulkhead.dae" />
+          </geometry>
+        </visual>
+        <collision>
+          <origin xyz="0 0 0" rpy="0 0 0"/>
+          <geometry>
+            <mesh filename="package://husky_description/meshes/dual_arm_bulkhead.dae" />
+          </geometry>
+        </collision>
+        </link>
+      <!-- Attach bulkhead -->
+      <joint name="dual_arm_bulkhead_joint" type="fixed">
+        <parent link="base_link" />
+        <child link="dual_arm_bulkhead_link"/>
+        <origin xyz="0.0812 0 0.245" rpy="0 0 0"/>
+      </joint>
+    </xacro:if>
     <xacro:if value="$(optenv HUSKY_TOP_PLATE_ENABLED true)">
       <!-- Spawn the top plate -->

Commit message: Added option to include user rails or not

File: husky_description/urdf/decorations.urdf.xacro (robot description, xacro)
@@ -37,18 +37,20 @@
       <child link="top_chassis_link" />
     </joint>
-    <!-- Spawn user rails -->
-    <link name="user_rail_link">
-      <visual>
-        <geometry>
-          <mesh filename="package://husky_description/meshes/user_rail.dae" />
-        </geometry>
-      </visual>
-    </link>
-    <!-- Attach user rails to base link -->
-    <joint name="user_rail" type="fixed">
-      <origin xyz="0.272 0 0.245" rpy="0 0 0" />
-      <parent link="base_link" />
-      <child link="user_rail_link" />
-    </joint>
+    <xacro:if value="$(optenv HUSKY_USER_RAILS true)">
+	    <!-- Spawn user rails -->
+	    <link name="user_rail_link">
+	      <visual>
+		<geometry>
+		  <mesh filename="package://husky_description/meshes/user_rail.dae" />
+		</geometry>
+	      </visual>
+	    </link>
+	    <!-- Attach user rails to base link -->
+	    <joint name="user_rail" type="fixed">
+	      <origin xyz="0.272 0 0.245" rpy="0 0 0" />
+	      <parent link="base_link" />
+	      <child link="user_rail_link" />
+	    </joint>
+    </xacro:if>
     <!-- Spawn front bumper link -->
     <link name="front_bumper_link">

File: husky_description/urdf/husky.urdf.xacro (robot description, xacro)
@@ -131,5 +131,5 @@
             <parent link="dual_arm_bulkhead_link"/>
             <child link="l_ur5_arm_base_link" />
-            <origin xyz="0 0 0" rpy="0 0 0"/>
+            <origin xyz="0 0 0.5" rpy="0 0 0"/>
         </joint>
          <!-- Joint right arm to top plate -->
@@ -137,5 +137,5 @@
             <parent link="dual_arm_bulkhead_link"/>
             <child link="r_ur5_arm_base_link" />
-            <origin xyz="0 0 0" rpy="0 0 0"/>
+            <origin xyz="0 0 -0.5" rpy="0 0 0"/>
         </joint>
     </xacro:if>

Commit message: Added dual arm positioning

File: husky_description/urdf/decorations.urdf.xacro (robot description, xacro)
@@ -101,5 +101,5 @@
         <parent link="base_link" />
         <child link="dual_arm_bulkhead_link"/>
-        <origin xyz="0.0812 0 0.245" rpy="0 0 0"/>
+        <origin xyz="0.0112 0 0.225" rpy="0 0 0"/>
       </joint>
     </xacro:if>

File: husky_description/urdf/husky.urdf.xacro (robot description, xacro)
@@ -131,5 +131,5 @@
             <parent link="dual_arm_bulkhead_link"/>
             <child link="l_ur5_arm_base_link" />
-            <origin xyz="0 0 0.5" rpy="0 0 0"/>
+            <origin xyz="0.125 -0.15 0.135" rpy="0.785 0 0"/>
         </joint>
          <!-- Joint right arm to top plate -->
@@ -137,5 +137,5 @@
             <parent link="dual_arm_bulkhead_link"/>
             <child link="r_ur5_arm_base_link" />
-            <origin xyz="0 0 -0.5" rpy="0 0 0"/>
+            <origin xyz="0.125 0.15 0.135" rpy="-0.785 0 0"/>
         </joint>
     </xacro:if>

Commit message: Added bulkhead positioning

File: husky_description/urdf/decorations.urdf.xacro (robot description, xacro)
@@ -101,5 +101,5 @@
         <parent link="base_link" />
         <child link="dual_arm_bulkhead_link"/>
-        <origin xyz="0.0112 0 0.225" rpy="0 0 0"/>
+        <origin xyz="0 0 0.225" rpy="0 0 0"/>
       </joint>
     </xacro:if>

Commit message: fix bug

File: husky_description/urdf/decorations.urdf.xacro (robot description, xacro)
@@ -38,19 +38,19 @@
     </joint>
     <!-- Spawn user rails -->
-    <link name="user_rail_link">
-      <visual>
-        <geometry>
-          <mesh filename="package://husky_description/meshes/user_rail.dae" />
-        </geometry>
-      </visual>
-    </link>
-    <xacro:if value="$(optenv HUSKY_USER_RAILS_ENABLED true)">
-    <!-- Attach user rails to base link -->
-    <joint name="user_rail" type="fixed">
-      <origin xyz="0.272 0 0.245" rpy="0 0 0" />
-      <parent link="base_link" />
-      <child link="user_rail_link" />
-    </joint>
-    </xacro:if>
+   <xacro:if value="$(optenv HUSKY_USER_RAILS_ENABLED true)">
+        <link name="user_rail_link">
+          <visual>
+            <geometry>
+              <mesh filename="package://husky_description/meshes/user_rail.dae" />
+            </geometry>
+          </visual>
+        </link>
+        <!-- Attach user rails to base link -->
+        <joint name="user_rail" type="fixed">
+          <origin xyz="0.272 0 0.245" rpy="0 0 0" />
+          <parent link="base_link" />
+          <child link="user_rail_link" />
+        </joint>
+   </xacro:if>
     <!-- Spawn front bumper link -->
     <link name="front_bumper_link">

Commit message: added bumper code removed rail code

File: husky_description/urdf/decorations.urdf.xacro (robot description, xacro)
@@ -38,5 +38,4 @@
     </joint>
     <!-- Spawn user rails -->
-   <xacro:if value="$(optenv HUSKY_USER_RAILS_ENABLED true)">
         <link name="user_rail_link">
           <visual>
@@ -52,5 +51,4 @@
           <child link="user_rail_link" />
         </joint>
-   </xacro:if>
     <!-- Spawn front bumper link -->
     <link name="front_bumper_link">
@@ -61,24 +59,26 @@
       </visual>
     </link>
-    <!-- Attach front bumper -->
-    <joint name="front_bumper" type="fixed">
-      <origin xyz="0.48 0 0.091" rpy="0 0 0" />
-      <parent link="base_link" />
-      <child link="front_bumper_link" />
-    </joint>
-    <!-- Spawn rear bumper link -->
-    <link name="rear_bumper_link">
-      <visual>
-        <geometry>
-          <mesh filename="package://husky_description/meshes/bumper.dae" />
-        </geometry>
-      </visual>
-    </link>
-    <!-- Attach rear bumper -->
-    <joint name="rear_bumper" type="fixed">
-      <origin xyz="-0.48 0 0.091" rpy="0 0 ${M_PI}" />
-      <parent link="base_link" />
-      <child link="rear_bumper_link" />
-    </joint>
+   <xacro:if value="$(optenv HUSKY_BUMPERS_ENABLED true)">
+        <!-- Attach front bumper -->
+        <joint name="front_bumper" type="fixed">
+          <origin xyz="0.48 0 0.091" rpy="0 0 0" />
+          <parent link="base_link" />
+          <child link="front_bumper_link" />
+        </joint>
+        <!-- Spawn rear bumper link -->
+        <link name="rear_bumper_link">
+          <visual>
+            <geometry>
+              <mesh filename="package://husky_description/meshes/bumper.dae" />
+            </geometry>
+          </visual>
+        </link>
+        <!-- Attach rear bumper -->
+        <joint name="rear_bumper" type="fixed">
+          <origin xyz="-0.48 0 0.091" rpy="0 0 ${M_PI}" />
+          <parent link="base_link" />
+          <child link="rear_bumper_link" />
+        </joint>
+    </xacro:if>
     <xacro:if value="$(optenv HUSKY_TOP_PLATE_ENABLED true)">
       <!-- Spawn the top plate -->

Commit message: Added environment variables to enabled or disabled the bumpers and the user rail

File: husky_description/urdf/decorations.urdf.xacro (robot description, xacro)
@@ -37,46 +37,52 @@
       <child link="top_chassis_link" />
     </joint>
-    <!-- Spawn user rails -->
-    <link name="user_rail_link">
-      <visual>
-        <geometry>
-          <mesh filename="package://husky_description/meshes/user_rail.dae" />
-        </geometry>
-      </visual>
-    </link>
-    <!-- Attach user rails to base link -->
-    <joint name="user_rail" type="fixed">
-      <origin xyz="0.272 0 0.245" rpy="0 0 0" />
-      <parent link="base_link" />
-      <child link="user_rail_link" />
-    </joint>
-    <!-- Spawn front bumper link -->
-    <link name="front_bumper_link">
-      <visual>
-        <geometry>
-          <mesh filename="package://husky_description/meshes/bumper.dae" />
-        </geometry>
-      </visual>
-    </link>
-    <!-- Attach front bumper -->
-    <joint name="front_bumper" type="fixed">
-      <origin xyz="0.48 0 0.091" rpy="0 0 0" />
-      <parent link="base_link" />
-      <child link="front_bumper_link" />
-    </joint>
-    <!-- Spawn rear bumper link -->
-    <link name="rear_bumper_link">
-      <visual>
-        <geometry>
-          <mesh filename="package://husky_description/meshes/bumper.dae" />
-        </geometry>
-      </visual>
-    </link>
-    <!-- Attach rear bumper -->
-    <joint name="rear_bumper" type="fixed">
-      <origin xyz="-0.48 0 0.091" rpy="0 0 ${M_PI}" />
-      <parent link="base_link" />
-      <child link="rear_bumper_link" />
-    </joint>
+    <xacro:if value="$(optenv HUSKY_USER_RAIL_ENABLED true)">
+      <!-- Spawn user rails -->
+      <link name="user_rail_link">
+        <visual>
+          <geometry>
+            <mesh filename="package://husky_description/meshes/user_rail.dae" />
+          </geometry>
+        </visual>
+      </link>
+      <!-- Attach user rails to base link -->
+      <joint name="user_rail" type="fixed">
+        <origin xyz="0.272 0 0.245" rpy="0 0 0" />
+        <parent link="base_link" />
+        <child link="user_rail_link" />
+      </joint>
+    </xacro:if>
+    <xacro:if value="$(optenv HUSKY_FRONT_BUMPER_ENABLED true)">
+      <!-- Spawn front bumper link -->
+      <link name="front_bumper_link">
+        <visual>
+          <geometry>
+            <mesh filename="package://husky_description/meshes/bumper.dae" />
+          </geometry>
+        </visual>
+      </link>
+      <!-- Attach front bumper -->
+      <joint name="front_bumper" type="fixed">
+        <origin xyz="0.48 0 0.091" rpy="0 0 0" />
+        <parent link="base_link" />
+        <child link="front_bumper_link" />
+      </joint>
+    </xacro:if>
+    <xacro:if value="$(optenv HUSKY_REAR_BUMPER_ENABLED true)">
+      <!-- Spawn rear bumper link -->
+      <link name="rear_bumper_link">
+        <visual>
+          <geometry>
+            <mesh filename="package://husky_description/meshes/bumper.dae" />
+          </geometry>
+        </visual>
+      </link>
+      <!-- Attach rear bumper -->
+      <joint name="rear_bumper" type="fixed">
+        <origin xyz="-0.48 0 0.091" rpy="0 0 ${M_PI}" />
+        <parent link="base_link" />
+        <child link="rear_bumper_link" />
+      </joint>
+    </xacro:if>
     <xacro:if value="$(optenv HUSKY_TOP_PLATE_ENABLED true)">
       <!-- Spawn the top plate -->

Commit message: Added a large top plate (used for waterproofing upgrade and UR5 upgrade) and an environment variable for controlling it HUSKY_LARGE_TOP_PLATE

File: husky_description/urdf/decorations.urdf.xacro (robot description, xacro)
@@ -81,30 +81,60 @@
     <xacro:if value="$(optenv HUSKY_TOP_PLATE_ENABLED true)">
       <!-- Spawn the top plate -->
-      <link name="top_plate_link">
-        <visual>
-          <origin xyz="0 0 0" rpy="0 0 0" />
-          <geometry>
-            <mesh filename="package://husky_description/meshes/top_plate.dae" />
-          </geometry>
-        </visual>
-        <collision>
-          <origin xyz="0 0 0" rpy="0 0 0"/>
-          <geometry>
-            <mesh filename="package://husky_description/meshes/top_plate.dae" />
-          </geometry>
-        </collision>
-        <collision>
-          <!-- Extra collision tag for widgets on top plate -->
-          <geometry>
-            <box size="0.32 0.41 0.09" rpy="0 0 0"/>
-          </geometry>
-        </collision>
-      </link>
-      <!-- Attach top plate -->
-      <joint name="top_plate_joint" type="fixed">
-        <parent link="base_link" />
-        <child link="top_plate_link"/>
-        <origin xyz="0.0812 0 0.245" rpy="0 0 0"/>
-      </joint>
+      <xacro:if value="$(optenv HUSKY_LARGE_TOP_PLATE false)">
+        <link name="top_plate_link">
+          <visual>
+            <origin xyz="0 0 0" rpy="0 0 0" />
+            <geometry>
+              <mesh filename="package://husky_description/meshes/large_top_plate.dae" />
+            </geometry>
+          </visual>
+          <collision>
+            <origin xyz="0 0 0" rpy="0 0 0"/>
+            <geometry>
+              <mesh filename="package://husky_description/meshes/large_top_plate_collision.stl" />
+            </geometry>
+          </collision>
+          <collision>
+            <!-- Extra collision tag for widgets on top plate -->
+            <geometry>
+              <box size="0.32 0.41 0.09" rpy="0 0 0"/>
+            </geometry>
+          </collision>
+        </link>
+        <!-- Attach top plate -->
+        <joint name="top_plate_joint" type="fixed">
+          <parent link="base_link" />
+          <child link="top_plate_link"/>
+          <origin xyz="0.0812 0 0.225" rpy="0 0 0"/>
+        </joint>
+      </xacro:if>
+      <xacro:unless value="$(optenv HUSKY_LARGE_TOP_PLATE false)">
+        <link name="top_plate_link">
+          <visual>
+            <origin xyz="0 0 0" rpy="0 0 0" />
+            <geometry>
+              <mesh filename="package://husky_description/meshes/top_plate.dae" />
+            </geometry>
+          </visual>
+          <collision>
+            <origin xyz="0 0 0" rpy="0 0 0"/>
+            <geometry>
+              <mesh filename="package://husky_description/meshes/top_plate.dae" />
+            </geometry>
+          </collision>
+          <collision>
+            <!-- Extra collision tag for widgets on top plate -->
+            <geometry>
+              <box size="0.32 0.41 0.09" rpy="0 0 0"/>
+            </geometry>
+          </collision>
+        </link>
+        <!-- Attach top plate -->
+        <joint name="top_plate_joint" type="fixed">
+          <parent link="base_link" />
+          <child link="top_plate_link"/>
+          <origin xyz="0.0812 0 0.245" rpy="0 0 0"/>
+        </joint>
+      </xacro:unless>
     </xacro:if>
   </xacro:macro>

Commit message: Added a large top plate (used for waterproofing upgrade and UR5 upgrade) and an environment variable for controlling it HUSKY_LARGE_TOP_PLATE

File: husky_description/urdf/decorations.urdf.xacro (robot description, xacro)
@@ -87,30 +87,60 @@
     <xacro:if value="$(optenv HUSKY_TOP_PLATE_ENABLED true)">
       <!-- Spawn the top plate -->
-      <link name="top_plate_link">
-        <visual>
-          <origin xyz="0 0 0" rpy="0 0 0" />
-          <geometry>
-            <mesh filename="package://husky_description/meshes/top_plate.dae" />
-          </geometry>
-        </visual>
-        <collision>
-          <origin xyz="0 0 0" rpy="0 0 0"/>
-          <geometry>
-            <mesh filename="package://husky_description/meshes/top_plate.dae" />
-          </geometry>
-        </collision>
-        <collision>
-          <!-- Extra collision tag for widgets on top plate -->
-          <geometry>
-            <box size="0.32 0.41 0.09" rpy="0 0 0"/>
-          </geometry>
-        </collision>
-      </link>
-      <!-- Attach top plate -->
-      <joint name="top_plate_joint" type="fixed">
-        <parent link="base_link" />
-        <child link="top_plate_link"/>
-        <origin xyz="0.0812 0 0.245" rpy="0 0 0"/>
-      </joint>
+      <xacro:if value="$(optenv HUSKY_LARGE_TOP_PLATE false)">
+        <link name="top_plate_link">
+          <visual>
+            <origin xyz="0 0 0" rpy="0 0 0" />
+            <geometry>
+              <mesh filename="package://husky_description/meshes/large_top_plate.dae" />
+            </geometry>
+          </visual>
+          <collision>
+            <origin xyz="0 0 0" rpy="0 0 0"/>
+            <geometry>
+              <mesh filename="package://husky_description/meshes/large_top_plate_collision.stl" />
+            </geometry>
+          </collision>
+          <collision>
+            <!-- Extra collision tag for widgets on top plate -->
+            <geometry>
+              <box size="0.32 0.41 0.09" rpy="0 0 0"/>
+            </geometry>
+          </collision>
+        </link>
+        <!-- Attach top plate -->
+        <joint name="top_plate_joint" type="fixed">
+          <parent link="base_link" />
+          <child link="top_plate_link"/>
+          <origin xyz="0.0812 0 0.225" rpy="0 0 0"/>
+        </joint>
+      </xacro:if>
+      <xacro:unless value="$(optenv HUSKY_LARGE_TOP_PLATE false)">
+        <link name="top_plate_link">
+          <visual>
+            <origin xyz="0 0 0" rpy="0 0 0" />
+            <geometry>
+              <mesh filename="package://husky_description/meshes/top_plate.dae" />
+            </geometry>
+          </visual>
+          <collision>
+            <origin xyz="0 0 0" rpy="0 0 0"/>
+            <geometry>
+              <mesh filename="package://husky_description/meshes/top_plate.dae" />
+            </geometry>
+          </collision>
+          <collision>
+            <!-- Extra collision tag for widgets on top plate -->
+            <geometry>
+              <box size="0.32 0.41 0.09" rpy="0 0 0"/>
+            </geometry>
+          </collision>
+        </link>
+        <!-- Attach top plate -->
+        <joint name="top_plate_joint" type="fixed">
+          <parent link="base_link" />
+          <child link="top_plate_link"/>
+          <origin xyz="0.0812 0 0.245" rpy="0 0 0"/>
+        </joint>
+      </xacro:unless>
     </xacro:if>
   </xacro:macro>

Commit message: Added env var to allow for extendable front bumper

File: husky_description/urdf/decorations.urdf.xacro (robot description, xacro)
@@ -59,10 +59,32 @@
       </visual>
     </link>
-    <!-- Attach front bumper -->
-    <joint name="front_bumper" type="fixed">
-      <origin xyz="0.48 0 0.091" rpy="0 0 0" />
-      <parent link="base_link" />
-      <child link="front_bumper_link" />
-    </joint>
+    <xacro:if value="$(optenv HUSKY_FORWARD_BUMPER_EXTENDED false)">
+      <!-- Attach front bumper -->
+      <joint name="front_bumper" type="fixed">
+        <origin xyz="0.55 0 0.091" rpy="0 0 0" />
+        <parent link="base_link" />
+        <child link="front_bumper_link" />
+      </joint>
+      <link name="front_bumper_extension_link">
+          <visual>
+              <geometry>
+                  <mesh filename="package://husky_description/meshes/bumper_extension.dae" />
+              </geometry>
+          </visual>
+      </link>
+      <joint name="front_bumper_extension" type="fixed">
+        <origin xyz="0.44 0 0.091" rpy="0 0 0" />
+        <parent link="base_link" />
+        <child link="front_bumper_extension_link" />
+      </joint>
+    </xacro:if>
+    <xacro:unless value="$(optenv HUSKY_FORWARD_BUMPER_EXTENDED false)">
+        <!-- Attach front bumper -->
+        <joint name="front_bumper" type="fixed">
+          <origin xyz="0.48 0 0.091" rpy="0 0 0" />
+          <parent link="base_link" />
+          <child link="front_bumper_link" />
+        </joint>
+    </xacro:unless>
     <!-- Spawn rear bumper link -->
     <link name="rear_bumper_link">

Commit message: Allowed for different lengths of bumper extensions

File: husky_description/urdf/decorations.urdf.xacro (robot description, xacro)
@@ -23,4 +23,5 @@
 <robot name="husky_decorations" xmlns:xacro="http://ros.org/wiki/xacro">
   <xacro:macro name="husky_decorate">
+    <xacro:property name="husky_bumper_extend" value="$(optenv HUSKY_FORWARD_BUMPER_EXTEND 0)" />
     <!-- Spawn Husky chassis -->
     <link name="top_chassis_link">
@@ -59,32 +60,24 @@
       </visual>
     </link>
-    <xacro:if value="$(optenv HUSKY_FORWARD_BUMPER_EXTENDED false)">
-      <!-- Attach front bumper -->
-      <joint name="front_bumper" type="fixed">
-        <origin xyz="0.55 0 0.091" rpy="0 0 0" />
-        <parent link="base_link" />
-        <child link="front_bumper_link" />
-      </joint>
+    <!-- Attach front bumper -->
+    <joint name="front_bumper" type="fixed">
+      <origin xyz="${0.48 + husky_bumper_extend / 100.0} 0 0.091" rpy="0 0 0" />
+      <parent link="base_link" />
+      <child link="front_bumper_link" />
+    </joint>
+    <xacro:if value="${husky_bumper_extend}">
       <link name="front_bumper_extension_link">
           <visual>
               <geometry>
-                  <mesh filename="package://husky_description/meshes/bumper_extension.dae" />
+                  <mesh filename="package://husky_description/meshes/bumper_extension.dae" scale="${husky_bumper_extend} 1 1"/>
               </geometry>
           </visual>
       </link>
       <joint name="front_bumper_extension" type="fixed">
-        <origin xyz="0.44 0 0.091" rpy="0 0 0" />
+        <origin xyz="${0.405 + husky_bumper_extend / 200.0} 0 0.091" rpy="0 0 0" />
         <parent link="base_link" />
         <child link="front_bumper_extension_link" />
       </joint>
     </xacro:if>
-    <xacro:unless value="$(optenv HUSKY_FORWARD_BUMPER_EXTENDED false)">
-        <!-- Attach front bumper -->
-        <joint name="front_bumper" type="fixed">
-          <origin xyz="0.48 0 0.091" rpy="0 0 0" />
-          <parent link="base_link" />
-          <child link="front_bumper_link" />
-        </joint>
-    </xacro:unless>
     <!-- Spawn rear bumper link -->
     <link name="rear_bumper_link">
