Commit message: Added env var to allow a 7cm forward bumper extension (#92)
* Added env var to allow for extendable front bumper

* Fix weird spacing

* Uploaded bumper extension meshes

* Allowed for different lengths of bumper extensions

File: husky_description/urdf/decorations.urdf.xacro (robot description, xacro)
@@ -23,4 +23,5 @@
 <robot name="husky_decorations" xmlns:xacro="http://ros.org/wiki/xacro">
   <xacro:macro name="husky_decorate">
+    <xacro:property name="husky_bumper_extend" value="$(optenv HUSKY_FORWARD_BUMPER_EXTEND 0)" />
     <!-- Spawn Husky chassis -->
     <link name="top_chassis_link">
@@ -61,8 +62,22 @@
     <!-- Attach front bumper -->
     <joint name="front_bumper" type="fixed">
-      <origin xyz="0.48 0 0.091" rpy="0 0 0" />
+      <origin xyz="${0.48 + husky_bumper_extend / 100.0} 0 0.091" rpy="0 0 0" />
       <parent link="base_link" />
       <child link="front_bumper_link" />
     </joint>
+    <xacro:if value="${husky_bumper_extend}">
+      <link name="front_bumper_extension_link">
+          <visual>
+              <geometry>
+                  <mesh filename="package://husky_description/meshes/bumper_extension.dae" scale="${husky_bumper_extend} 1 1"/>
+              </geometry>
+          </visual>
+      </link>
+      <joint name="front_bumper_extension" type="fixed">
+        <origin xyz="${0.405 + husky_bumper_extend / 200.0} 0 0.091" rpy="0 0 0" />
+        <parent link="base_link" />
+        <child link="front_bumper_extension_link" />
+      </joint>
+    </xacro:if>
     <!-- Spawn rear bumper link -->
     <link name="rear_bumper_link">

Commit message: Added some additional frames on the top plates and an environment variable for diabling the user rails

File: husky_description/urdf/decorations.urdf.xacro (robot description, xacro)
@@ -38,18 +38,20 @@
       <child link="top_chassis_link" />
     </joint>
-    <!-- Spawn user rails -->
-    <link name="user_rail_link">
-      <visual>
-        <geometry>
-          <mesh filename="package://husky_description/meshes/user_rail.dae" />
-        </geometry>
-      </visual>
-    </link>
-    <!-- Attach user rails to base link -->
-    <joint name="user_rail" type="fixed">
-      <origin xyz="0.272 0 0.245" rpy="0 0 0" />
-      <parent link="base_link" />
-      <child link="user_rail_link" />
-    </joint>
+    <xacro:if value="$(optenv HUSKY_USER_RAIL_ENABLED true)">
+      <!-- Spawn user rails -->
+      <link name="user_rail_link">
+        <visual>
+          <geometry>
+            <mesh filename="package://husky_description/meshes/user_rail.dae" />
+          </geometry>
+        </visual>
+      </link>
+      <!-- Attach user rails to base link -->
+      <joint name="user_rail" type="fixed">
+        <origin xyz="0.272 0 0.245" rpy="0 0 0" />
+        <parent link="base_link" />
+        <child link="user_rail_link" />
+      </joint>
+    </xacro:if>
     <!-- Spawn front bumper link -->
     <link name="front_bumper_link">
@@ -123,4 +125,16 @@
           <origin xyz="0.0812 0 0.225" rpy="0 0 0"/>
         </joint>
+        <!-- Top plate front link -->
+        <joint name="top_plate_front_joint" type="fixed">
+          <parent link="top_plate_link" />
+          <child link="top_plate_front_link"/>
+          <origin xyz="0.4125 0 0.00672" rpy="0 0 0"/>
+        </joint>
+        <!-- Top plate rear link-->
+        <joint name="top_plate_rear_joint" type="fixed">
+          <parent link="top_plate_link" />
+          <child link="top_plate_rear_link"/>
+          <origin xyz="-0.4125 0 0.00672" rpy="0 0 0"/>
+        </joint>
       </xacro:if>
       <xacro:unless value="$(optenv HUSKY_LARGE_TOP_PLATE false)">
@@ -151,5 +165,19 @@
           <origin xyz="0.0812 0 0.245" rpy="0 0 0"/>
         </joint>
+        <!-- Top plate front link -->
+        <joint name="top_plate_front_joint" type="fixed">
+          <parent link="top_plate_link" />
+          <child link="top_plate_front_link"/>
+          <origin xyz="0.36367 0 0.00639" rpy="0 0 0"/>
+        </joint>
+        <!-- Top plate rear link-->
+        <joint name="top_plate_rear_joint" type="fixed">
+          <parent link="top_plate_link" />
+          <child link="top_plate_rear_link"/>
+          <origin xyz="-0.36633 0 0.00639" rpy="0 0 0"/>
+        </joint>
       </xacro:unless>
+      <link name="top_plate_front_link"/>
+      <link name="top_plate_rear_link"/>
     </xacro:if>
   </xacro:macro>

Commit message: Initial Gazebo Classic changes.

File: husky_description/urdf/decorations.urdf.xacro (robot description, xacro)
@@ -16,5 +16,5 @@
         <origin xyz="0 0 0" rpy="0 0 0" />
         <geometry>
-          <mesh filename="package://husky_description/meshes/top_chassis.dae" />
+          <mesh filename="file://$(find husky_description)/meshes/top_chassis.dae" />
         </geometry>
       </visual>
@@ -30,5 +30,5 @@
         <visual>
           <geometry>
-            <mesh filename="package://husky_description/meshes/user_rail.dae" />
+            <mesh filename="file://$(find husky_description)/meshes/user_rail.dae" />
           </geometry>
         </visual>
@@ -45,5 +45,5 @@
       <visual>
         <geometry>
-          <mesh filename="package://husky_description/meshes/bumper.dae" />
+          <mesh filename="file://$(find husky_description)/meshes/bumper.dae" />
         </geometry>
       </visual>
@@ -59,5 +59,5 @@
           <visual>
               <geometry>
-                  <mesh filename="package://husky_description/meshes/bumper_extension.dae" />
+                  <mesh filename="file://$(find husky_description)/meshes/bumper_extension.dae" />
               </geometry>
           </visual>
@@ -73,5 +73,5 @@
       <visual>
         <geometry>
-          <mesh filename="package://husky_description/meshes/bumper.dae" />
+          <mesh filename="file://$(find husky_description)/meshes/bumper.dae" />
         </geometry>
       </visual>
@@ -87,5 +87,5 @@
           <visual>
               <geometry>
-                  <mesh filename="package://husky_description/meshes/bumper_extension.dae" />
+                  <mesh filename="file://$(find husky_description)/meshes/bumper_extension.dae" />
               </geometry>
           </visual>
@@ -104,5 +104,5 @@
             <origin xyz="0 0 0" rpy="0 0 0" />
             <geometry>
-              <mesh filename="package://husky_description/meshes/large_top_plate.dae" />
+              <mesh filename="file://$(find husky_description)/meshes/large_top_plate.dae" />
             </geometry>
           </visual>
@@ -110,5 +110,5 @@
             <origin xyz="0 0 0" rpy="0 0 0"/>
             <geometry>
-              <mesh filename="package://husky_description/meshes/large_top_plate_collision.stl" />
+              <mesh filename="file://$(find husky_description)/meshes/large_top_plate_collision.stl" />
             </geometry>
           </collision>
@@ -138,5 +138,5 @@
             <origin xyz="0 0 0" rpy="0 0 0" />
             <geometry>
-              <mesh filename="package://husky_description/meshes/top_plate.dae" />
+              <mesh filename="file://$(find husky_description)/meshes/top_plate.dae" />
             </geometry>
           </visual>
@@ -144,5 +144,5 @@
             <origin xyz="0 0 0" rpy="0 0 0"/>
             <geometry>
-              <mesh filename="package://husky_description/meshes/top_plate.stl" />
+              <mesh filename="file://$(find husky_description)/meshes/top_plate.stl" />
             </geometry>
           </collision>

File: husky_description/urdf/husky.urdf.xacro (robot description, xacro)
@@ -11,4 +11,5 @@
   <xacro:property name="husky_rear_bumper_extend" value="$(optenv HUSKY_REAR_BUMPER_EXTEND 0)" />
   <xacro:arg name="robot_namespace" default="/" />
+  <xacro:arg name="is_sim" default="false" />
   <xacro:arg name="urdf_extras" default="empty.urdf" />
   <!-- Included URDF/XACRO Files -->
@@ -35,5 +36,5 @@
       <origin xyz="0 0 0" rpy="0 0 0" />
       <geometry>
-        <mesh filename="package://husky_description/meshes/base_link.dae" />
+        <mesh filename="file://$(find husky_description)/meshes/base_link.dae" />
       </geometry>
     </visual>
@@ -125,10 +126,9 @@
     <xacro:intel_realsense_mount prefix="camera" topic="realsense" parent_link="realsense_mountpoint"/>
   </xacro:if> -->
-  <!-- <gazebo>
-    <plugin name="gazebo_ros_control" filename="libgazebo_ros_control.so">
-      <robotNamespace>$(arg robot_namespace)</robotNamespace>
-      <legacyModeNS>true</legacyModeNS>
+  <gazebo>
+    <plugin name="gazebo_ros2_control" filename="libgazebo_ros2_control.so">
+      <parameters>$(find husky_control)/config/control.yaml</parameters>
     </plugin>
-  </gazebo> -->
+  </gazebo>
   <gazebo>
     <plugin name="imu_controller" filename="libhector_gazebo_ros_imu.so">
@@ -160,48 +160,73 @@
     </plugin>
   </gazebo>
-  <ros2_control name="husky_hardware" type="system">
-    <hardware>
-      <plugin>husky_base/HuskyHardware</plugin>
-      <param name="hw_start_duration_sec">2.0</param>
-      <param name="hw_stop_duration_sec">3.0</param>
-      <param name="wheel_diameter">0.3302</param>
-      <param name="max_accel">5.0</param>
-      <param name="max_speed">1.0</param>
-      <param name="polling_timeout">10.0</param>
-      <param name="serial_port">/dev/prolific</param>
-    </hardware>
-    <joint name="front_left_wheel">
-      <command_interface name="velocity">
-        <param name="min">-1</param>
-        <param name="max">1</param>
-      </command_interface>
-      <state_interface name="position"/>
-      <state_interface name="velocity"/>
-    </joint>
-    <joint name="front_right_wheel">
-      <command_interface name="velocity">
-        <param name="min">-1</param>
-        <param name="max">1</param>
-      </command_interface>
-      <state_interface name="position"/>
-      <state_interface name="velocity"/>
-    </joint>
-    <joint name="rear_left_wheel">
-      <command_interface name="velocity">
-        <param name="min">-1</param>
-        <param name="max">1</param>
-      </command_interface>
-      <state_interface name="position"/>
-      <state_interface name="velocity"/>
-    </joint>
-    <joint name="rear_right_wheel">
-      <command_interface name="velocity">
-        <param name="min">-1</param>
-        <param name="max">1</param>
-      </command_interface>
-      <state_interface name="position"/>
-      <state_interface name="velocity"/>
-    </joint>
-  </ros2_control>
+  <xacro:unless value="$(arg is_sim)">
+    <ros2_control name="husky_hardware" type="system">
+      <hardware>
+        <plugin>husky_base/HuskyHardware</plugin>
+        <param name="hw_start_duration_sec">2.0</param>
+        <param name="hw_stop_duration_sec">3.0</param>
+        <param name="wheel_diameter">0.3302</param>
+        <param name="max_accel">5.0</param>
+        <param name="max_speed">1.0</param>
+        <param name="polling_timeout">10.0</param>
+        <param name="serial_port">/dev/prolific</param>
+      </hardware>
+      <joint name="front_left_wheel_joint">
+        <command_interface name="velocity">
+          <param name="min">-1</param>
+          <param name="max">1</param>
+        </command_interface>
+        <state_interface name="position"/>
+        <state_interface name="velocity"/>
+      </joint>
+      <joint name="rear_left_wheel_joint">
+        <command_interface name="velocity">
+          <param name="min">-1</param>
+          <param name="max">1</param>
+        </command_interface>
+        <state_interface name="position"/>
+        <state_interface name="velocity"/>
+      </joint>
+      <joint name="front_right_wheel_joint">
+        <command_interface name="velocity">
+          <param name="min">-1</param>
+          <param name="max">1</param>
+        </command_interface>
+        <state_interface name="position"/>
+        <state_interface name="velocity"/>
+      </joint>
+      <joint name="rear_right_wheel_joint">
+        <command_interface name="velocity">
+          <param name="min">-1</param>
+          <param name="max">1</param>
+        </command_interface>
+        <state_interface name="position"/>
+        <state_interface name="velocity"/>
+      </joint>
+    </ros2_control>
+  </xacro:unless>
+  <xacro:if value="$(arg is_sim)">
+    <ros2_control name="husky_hardware" type="system">
+      <hardware>
+        <plugin>gazebo_ros2_control/GazeboSystem</plugin>
+      </hardware>
+      <joint name="front_left_wheel_joint">
+        <state_interface name="position" />
+        <command_interface name="velocity" />
+      </joint>
+      <joint name="rear_left_wheel_joint">
+        <state_interface name="position" />
+        <command_interface name="velocity" />
+      </joint>
+      <joint name="front_right_wheel_joint">
+        <state_interface name="position" />
+        <command_interface name="velocity" />
+      </joint>
+      <joint name="rear_right_wheel_joint">
+        <state_interface name="position" />
+        <command_interface name="velocity" />
+      </joint>
+    </ros2_control>
+  </xacro:if>
   <!-- Optional custom includes. -->
   <xacro:include filename="$(arg urdf_extras)" />

File: husky_description/urdf/wheel.urdf.xacro (robot description, xacro)
@@ -1,46 +1,37 @@
 <?xml version="1.0"?>
 <robot xmlns:xacro="http://ros.org/wiki/xacro" name="husky_wheel">
-	<xacro:macro name="husky_wheel" params="wheel_prefix *joint_pose">
-		<link name="${wheel_prefix}_wheel_link">
-			<inertial>
-				<mass value="2.637" />
-				<origin xyz="0 0 0" />
-				<inertia  ixx="0.02467" ixy="0" ixz="0" iyy="0.04411" iyz="0" izz="0.02467" />
-			</inertial>
-			<visual>
-				<origin xyz="0 0 0" rpy="0 0 0" />
-				<geometry>
-					<mesh filename="package://husky_description/meshes/wheel.dae" />
-				</geometry>
-			</visual>
-			<collision>
-				<origin xyz="0 0 0" rpy="${M_PI/2} 0 0" />
-				<geometry>
-					<cylinder length="${wheel_length}" radius="${wheel_radius}" />
-				</geometry>
-			</collision>
-		</link>
-		<gazebo reference="${wheel_prefix}_wheel_link">
-			<mu1 value="1.0"/>
-			<mu2 value="1.0"/>
-			<kp value="10000000.0" />
-			<kd value="1.0" />
-			<fdir1 value="1 0 0"/>
-		</gazebo>
-		<joint name="${wheel_prefix}_wheel" type="continuous">
-			<parent link="base_link"/>
-			<child link="${wheel_prefix}_wheel_link"/>
-			<xacro:insert_block name="joint_pose"/>
-			<axis xyz="0 1 0" rpy="0 0 0" />
-		</joint>
-		<transmission name="${wheel_prefix}_wheel_trans" type="SimpleTransmission">
-			<type>transmission_interface/SimpleTransmission</type>
-			<actuator name="${wheel_prefix}_wheel_motor">
-				<mechanicalReduction>1</mechanicalReduction>
-			</actuator>
-			<joint name="${wheel_prefix}_wheel">
-				<hardwareInterface>hardware_interface/VelocityJointInterface</hardwareInterface>
-			</joint>
-		</transmission>
-	</xacro:macro>
+  <xacro:macro name="husky_wheel" params="wheel_prefix *joint_pose">
+    <link name="${wheel_prefix}_wheel">
+      <inertial>
+        <mass value="2.637" />
+        <origin xyz="0 0 0" />
+        <inertia  ixx="0.02467" ixy="0" ixz="0" iyy="0.04411" iyz="0" izz="0.02467" />
+      </inertial>
+      <visual>
+        <origin xyz="0 0 0" rpy="0 0 0" />
+        <geometry>
+          <mesh filename="file://$(find husky_description)/meshes/wheel.dae" />
+        </geometry>
+      </visual>
+      <collision>
+        <origin xyz="0 0 0" rpy="${M_PI/2} 0 0" />
+        <geometry>
+          <cylinder length="${wheel_length}" radius="${wheel_radius}" />
+        </geometry>
+      </collision>
+    </link>
+    <gazebo reference="${wheel_prefix}_wheel">
+      <mu1 value="1.0"/>
+      <mu2 value="1.0"/>
+      <kp value="10000000.0" />
+      <kd value="1.0" />
+      <fdir1 value="1 0 0"/>
+    </gazebo>
+    <joint name="${wheel_prefix}_wheel_joint" type="continuous">
+      <parent link="base_link"/>
+      <child link="${wheel_prefix}_wheel"/>
+      <xacro:insert_block name="joint_pose"/>
+      <axis xyz="0 1 0" rpy="0 0 0" />
+    </joint>
+  </xacro:macro>
 </robot>
