Commit message: Add tf_prefix argument to description
This way, the description can easily used in a multi-robot setup.

File: husky_description/urdf/decorations.urdf.xacro (robot description, xacro)
@@ -29,5 +29,5 @@
   <material name="white"><color rgba="1.0 1.0 1.0 1.0" /></material>
   <material name="red"><color rgba="1.0 0.0 0.0 1.0" /></material>
-  <xacro:macro name="husky_decorate">
+  <xacro:macro name="husky_decorate" params="tf_prefix:=''">
     <xacro:property name="husky_front_bumper_enable"    value="$(optenv HUSKY_FRONT_BUMPER 1)" />
     <xacro:property name="husky_rear_bumper_enable"     value="$(optenv HUSKY_REAR_BUMPER 1)" />
@@ -36,5 +36,5 @@
     <xacro:property name="husky_wibotic_bumper_enable"  value="$(optenv HUSKY_WIBOTIC_BUMPER 0)" />
     <!-- Spawn Husky chassis -->
-    <link name="top_chassis_link">
+    <link name="${tf_prefix}top_chassis_link">
       <visual>
         <origin xyz="0 0 0" rpy="0 0 0" />
@@ -45,11 +45,11 @@
     </link>
     <!-- Attach chassis to the robot -->
-    <joint name="top_chassis_joint" type="fixed">
-      <parent link="base_link" />
-      <child link="top_chassis_link" />
+    <joint name="${tf_prefix}top_chassis_joint" type="fixed">
+      <parent link="${tf_prefix}base_link" />
+      <child link="${tf_prefix}top_chassis_link" />
     </joint>
     <xacro:if value="$(optenv HUSKY_USER_RAIL_ENABLED true)">
       <!-- Spawn user rails -->
-      <link name="user_rail_link">
+      <link name="${tf_prefix}user_rail_link">
         <visual>
           <geometry>
@@ -59,8 +59,8 @@
       </link>
       <!-- Attach user rails to base link -->
-      <joint name="user_rail" type="fixed">
+      <joint name="${tf_prefix}user_rail" type="fixed">
         <origin xyz="0.272 0 0.245" rpy="0 0 0" />
-        <parent link="base_link" />
-        <child link="user_rail_link" />
+        <parent link="${tf_prefix}base_link" />
+        <child link="${tf_prefix}user_rail_link" />
       </joint>
     </xacro:if>
@@ -68,5 +68,5 @@
     <xacro:if value="${husky_front_bumper_enable}">
       <xacro:unless value="${husky_wibotic_bumper_enable}">
-        <link name="front_bumper_link">
+        <link name="${tf_prefix}front_bumper_link">
           <visual>
             <geometry>
@@ -77,5 +77,5 @@
       </xacro:unless>
       <xacro:if value="${husky_wibotic_bumper_enable}">
-        <link name="front_bumper_link">
+        <link name="${tf_prefix}front_bumper_link">
           <visual>
             <material name="black"/>
@@ -87,11 +87,11 @@
       </xacro:if>
       <!-- Attach front bumper -->
-      <joint name="front_bumper" type="fixed">
+      <joint name="${tf_prefix}front_bumper" type="fixed">
         <origin xyz="${0.48 + husky_front_bumper_extend} 0 0.091" rpy="0 0 0" />
-        <parent link="base_link" />
-        <child link="front_bumper_link" />
+        <parent link="${tf_prefix}base_link" />
+        <child link="${tf_prefix}front_bumper_link" />
       </joint>
       <xacro:if value="${husky_front_bumper_extend}">
-        <link name="front_bumper_extension_link">
+        <link name="${tf_prefix}front_bumper_extension_link">
             <visual>
                 <geometry>
@@ -100,8 +100,8 @@
             </visual>
         </link>
-        <joint name="front_bumper_extension" type="fixed">
+        <joint name="${tf_prefix}front_bumper_extension" type="fixed">
           <origin xyz="${0.48 + husky_front_bumper_extend} 0 0.091" rpy="0 0 0" />
-          <parent link="base_link" />
-          <child link="front_bumper_extension_link" />
+          <parent link="${tf_prefix}base_link" />
+          <child link="${tf_prefix}front_bumper_extension_link" />
         </joint>
       </xacro:if>
@@ -109,5 +109,5 @@
     <!-- Spawn rear bumper link -->
     <xacro:if value="${husky_rear_bumper_enable}">
-      <link name="rear_bumper_link">
+      <link name="${tf_prefix}rear_bumper_link">
         <visual>
           <geometry>
@@ -117,11 +117,11 @@
       </link>
       <!-- Attach rear bumper -->
-      <joint name="rear_bumper" type="fixed">
+      <joint name="${tf_prefix}rear_bumper" type="fixed">
         <origin xyz="${-0.48 - husky_rear_bumper_extend} 0 0.091" rpy="0 0 ${M_PI}" />
-        <parent link="base_link" />
-        <child link="rear_bumper_link" />
+        <parent link="${tf_prefix}base_link" />
+        <child link="${tf_prefix}rear_bumper_link" />
       </joint>
       <xacro:if value="${husky_rear_bumper_extend}">
-        <link name="rear_bumper_extension_link">
+        <link name="${tf_prefix}rear_bumper_extension_link">
             <visual>
                 <geometry>
@@ -130,8 +130,8 @@
             </visual>
         </link>
-        <joint name="rear_bumper_extension" type="fixed">
+        <joint name="${tf_prefix}rear_bumper_extension" type="fixed">
           <origin xyz="${-0.48 - husky_rear_bumper_extend} 0 0.091" rpy="0 0 ${M_PI}" />
-          <parent link="base_link" />
-          <child link="rear_bumper_extension_link" />
+          <parent link="${tf_prefix}base_link" />
+          <child link="${tf_prefix}rear_bumper_extension_link" />
         </joint>
       </xacro:if>
@@ -140,5 +140,5 @@
       <!-- Spawn the top plate -->
       <xacro:if value="$(optenv HUSKY_LARGE_TOP_PLATE false)">
-        <link name="top_plate_link">
+        <link name="${tf_prefix}top_plate_link">
           <visual>
             <origin xyz="0 0 0" rpy="0 0 0" />
@@ -155,24 +155,24 @@
         </link>
         <!-- Attach top plate -->
-        <joint name="top_plate_joint" type="fixed">
-          <parent link="base_link" />
-          <child link="top_plate_link"/>
+        <joint name="${tf_prefix}top_plate_joint" type="fixed">
+          <parent link="${tf_prefix}base_link" />
+          <child link="${tf_prefix}top_plate_link"/>
           <origin xyz="0.0812 0 0.225" rpy="0 0 0"/>
         </joint>
         <!-- Top plate front link -->
-        <joint name="top_plate_front_joint" type="fixed">
-          <parent link="top_plate_link" />
-          <child link="top_plate_front_link"/>
+        <joint name="${tf_prefix}top_plate_front_joint" type="fixed">
+          <parent link="${tf_prefix}top_plate_link" />
+          <child link="${tf_prefix}top_plate_front_link"/>
           <origin xyz="0.4125 0 0.00672" rpy="0 0 0"/>
         </joint>
         <!-- Top plate rear link-->
-        <joint name="top_plate_rear_joint" type="fixed">
-          <parent link="top_plate_link" />
-          <child link="top_plate_rear_link"/>
+        <joint name="${tf_prefix}top_plate_rear_joint" type="fixed">
+          <parent link="${tf_prefix}top_plate_link" />
+          <child link="${tf_prefix}top_plate_rear_link"/>
           <origin xyz="-0.4125 0 0.00672" rpy="0 0 0"/>
         </joint>
       </xacro:if>
       <xacro:unless value="$(optenv HUSKY_LARGE_TOP_PLATE false)">
-        <link name="top_plate_link">
+        <link name="${tf_prefix}top_plate_link">
           <visual>
             <origin xyz="0 0 0" rpy="0 0 0" />
@@ -189,24 +189,24 @@
         </link>
         <!-- Attach top plate -->
-        <joint name="top_plate_joint" type="fixed">
-          <parent link="base_link" />
-          <child link="top_plate_link"/>
+        <joint name="${tf_prefix}top_plate_joint" type="fixed">
+          <parent link="${tf_prefix}base_link" />
+          <child link="${tf_prefix}top_plate_link"/>
           <origin xyz="0.0812 0 0.245" rpy="0 0 0"/>
         </joint>
         <!-- Top plate front link -->
-        <joint name="top_plate_front_joint" type="fixed">
-          <parent link="top_plate_link" />
-          <child link="top_plate_front_link"/>
+        <joint name="${tf_prefix}top_plate_front_joint" type="fixed">
+          <parent link="${tf_prefix}top_plate_link" />
+          <child link="${tf_prefix}top_plate_front_link"/>
           <origin xyz="0.36367 0 0.00639" rpy="0 0 0"/>
         </joint>
         <!-- Top plate rear link-->
-        <joint name="top_plate_rear_joint" type="fixed">
-          <parent link="top_plate_link" />
-          <child link="top_plate_rear_link"/>
+        <joint name="${tf_prefix}top_plate_rear_joint" type="fixed">
+          <parent link="${tf_prefix}top_plate_link" />
+          <child link="${tf_prefix}top_plate_rear_link"/>
           <origin xyz="-0.36633 0 0.00639" rpy="0 0 0"/>
         </joint>
       </xacro:unless>
-      <link name="top_plate_front_link"/>
-      <link name="top_plate_rear_link"/>
+      <link name="${tf_prefix}top_plate_front_link"/>
+      <link name="${tf_prefix}top_plate_rear_link"/>
     </xacro:if>
   </xacro:macro>

File: husky_description/urdf/husky.urdf.xacro (robot description, xacro)
@@ -53,4 +53,5 @@
   <xacro:arg name="sensor_arch"         default="$(optenv HUSKY_SENSOR_ARCH 0)" />
   <xacro:arg name="robot_namespace" default="$(optenv ROBOT_NAMESPACE /)" />
+  <xacro:arg name="tf_prefix" default="$(optenv TF_PREFIX)" />
   <xacro:arg name="urdf_extras" default="$(optenv HUSKY_URDF_EXTRAS empty.urdf)" />
   <xacro:arg name="cpr_urdf_extras" default="$(optenv CPR_URDF_EXTRAS empty.urdf)" />
@@ -76,5 +77,5 @@
   <xacro:property name="wheel_radius" value="0.1651" />
   <!-- Base link is the center of the robot's bottom plate -->
-  <link name="base_link">
+  <link name="$(arg tf_prefix)base_link">
     <visual>
       <origin xyz="0 0 0" rpy="0 0 0" />
@@ -97,12 +98,12 @@
   </link>
   <!-- Base footprint is on the ground under the robot -->
-  <link name="base_footprint"/>
-  <joint name="base_footprint_joint" type="fixed">
+  <link name="$(arg tf_prefix)base_footprint"/>
+  <joint name="$(arg tf_prefix)base_footprint_joint" type="fixed">
     <origin xyz="0 0 ${wheel_vertical_offset - wheel_radius}" rpy="0 0 0" />
-    <parent link="base_link" />
-    <child link="base_footprint" />
+    <parent link="$(arg tf_prefix)base_link" />
+    <child link="$(arg tf_prefix)base_footprint" />
   </joint>
   <!-- Inertial link stores the robot's inertial information -->
-  <link name="inertial_link">
+  <link name="$(arg tf_prefix)inertial_link">
     <inertial>
       <mass value="46.034" />
@@ -111,52 +112,52 @@
     </inertial>
   </link>
-  <joint name="inertial_joint" type="fixed">
+  <joint name="$(arg tf_prefix)inertial_joint" type="fixed">
     <origin xyz="0 0 0" rpy="0 0 0" />
-    <parent link="base_link" />
-    <child link="inertial_link" />
+    <parent link="$(arg tf_prefix)base_link" />
+    <child link="$(arg tf_prefix)inertial_link" />
   </joint>
   <!-- IMU Link is the standard mounting position for the UM6 IMU.-->
   <!-- Can be modified with environment variables in /etc/ros/setup.bash -->
-  <link name="imu_link"/>
-  <joint name="imu_joint" type="fixed">
+  <link name="$(arg tf_prefix)imu_link"/>
+  <joint name="$(arg tf_prefix)imu_joint" type="fixed">
     <origin xyz="$(optenv HUSKY_IMU_XYZ 0.19 0 0.149)" rpy="$(optenv HUSKY_IMU_RPY 0 -1.5708 3.1416)" />
-    <parent link="base_link" />
-    <child link="imu_link" />
+    <parent link="$(arg tf_prefix)base_link" />
+    <child link="$(arg tf_prefix)imu_link" />
   </joint>
   <gazebo reference="imu_link">
   </gazebo>
   <!-- Husky wheel macros -->
-  <xacro:husky_wheel wheel_prefix="front_left">
+  <xacro:husky_wheel wheel_prefix="front_left" tf_prefix="$(arg tf_prefix)">
     <origin xyz="${wheelbase/2} ${track/2} ${wheel_vertical_offset}" rpy="0 0 0" />
   </xacro:husky_wheel>
-  <xacro:husky_wheel wheel_prefix="front_right">
+  <xacro:husky_wheel wheel_prefix="front_right" tf_prefix="$(arg tf_prefix)">
     <origin xyz="${wheelbase/2} ${-track/2} ${wheel_vertical_offset}" rpy="0 0 0" />
   </xacro:husky_wheel>
-  <xacro:husky_wheel wheel_prefix="rear_left">
+  <xacro:husky_wheel wheel_prefix="rear_left" tf_prefix="$(arg tf_prefix)">
     <origin xyz="${-wheelbase/2} ${track/2} ${wheel_vertical_offset}" rpy="0 0 0" />
   </xacro:husky_wheel>
-  <xacro:husky_wheel wheel_prefix="rear_right">
+  <xacro:husky_wheel wheel_prefix="rear_right" tf_prefix="$(arg tf_prefix)">
     <origin xyz="${-wheelbase/2} ${-track/2} ${wheel_vertical_offset}" rpy="0 0 0" />
   </xacro:husky_wheel>
-  <xacro:husky_decorate />
+  <xacro:husky_decorate tf_prefix="$(arg tf_prefix)"/>
   <!--
     Add the primary and secondary lasers
   -->
   <xacro:if value="$(arg laser_enabled)">
-    <xacro:sick_lms1xx_mount prefix="base"/>
-    <xacro:sick_lms1xx frame="base_laser" topic="scan" robot_namespace="$(arg robot_namespace)"/>
-    <joint name="laser_mount_joint" type="fixed">
+    <xacro:sick_lms1xx_mount prefix="$(arg tf_prefix)base"/>
+    <xacro:sick_lms1xx frame="$(arg tf_prefix)base_laser" topic="scan" robot_namespace="$(arg robot_namespace)"/>
+    <joint name="$(arg tf_prefix)laser_mount_joint" type="fixed">
       <origin xyz="$(arg laser_xyz)" rpy="$(arg laser_rpy)" />
-      <parent link="top_plate_link" />
-      <child link="base_laser_mount" />
+      <parent link="$(arg tf_prefix)top_plate_link" />
+      <child link="$(arg tf_prefix)base_laser_mount" />
     </joint>
   </xacro:if>
   <xacro:if value="$(arg laser_secondary_enabled)">
-    <xacro:sick_lms1xx_mount prefix="rear"/>
-    <xacro:sick_lms1xx frame="rear_laser" topic="rear/scan" robot_namespace="$(arg robot_namespace)"/>
-    <joint name="laser_secondary_mount_joint" type="fixed">
+    <xacro:sick_lms1xx_mount prefix="$(arg tf_prefix)rear"/>
+    <xacro:sick_lms1xx frame="$(arg tf_prefix)rear_laser" topic="rear/scan" robot_namespace="$(arg robot_namespace)"/>
+    <joint name="$(arg tf_prefix)laser_secondary_mount_joint" type="fixed">
       <origin xyz="$(arg laser_secondary_xyz)" rpy="$(arg laser_secondary_rpy)" />
-      <parent link="top_plate_link" />
-      <child link="rear_laser_mount" />
+      <parent link="$(arg tf_prefix)top_plate_link" />
+      <child link="$(arg tf_prefix)rear_laser_mount" />
     </joint>
   </xacro:if>
@@ -165,10 +166,10 @@
   -->
   <xacro:if value="$(arg laser_ust10_front_enabled)">
-    <xacro:hokuyo_ust10_mount topic="$(arg laser_ust10_front_topic)" prefix="$(arg laser_ust10_front_prefix)" parent_link="$(arg laser_ust10_front_parent)">
+    <xacro:hokuyo_ust10_mount topic="$(arg laser_ust10_front_topic)" prefix="$(arg tf_prefix)$(arg laser_ust10_front_prefix)" parent_link="$(arg tf_prefix)$(arg laser_ust10_front_parent)">
         <origin xyz="$(arg laser_ust10_front_xyz)" rpy="$(arg laser_ust10_front_rpy)" />
       </xacro:hokuyo_ust10_mount>
   </xacro:if>
   <xacro:if value="$(arg laser_ust10_rear_enabled)">
-    <xacro:hokuyo_ust10_mount topic="$(arg laser_ust10_rear_topic)" prefix="$(arg laser_ust10_rear_prefix)" parent_link="$(arg laser_ust10_rear_parent)">
+    <xacro:hokuyo_ust10_mount topic="$(arg laser_ust10_rear_topic)" prefix="$(arg tf_prefix)$(arg laser_ust10_rear_prefix)" parent_link="$(arg tf_prefix)$(arg laser_ust10_rear_parent)">
         <origin xyz="$(arg laser_ust10_rear_xyz)" rpy="$(arg laser_ust10_rear_rpy)" />
       </xacro:hokuyo_ust10_mount>
@@ -182,5 +183,5 @@
   <xacro:property name="sensorbar_needed_lidar"     value="$(arg laser_3d_enabled)" />
   <xacro:if value="${sensorbar_needed_realsense or sensorbar_user_enabled or sensorbar_needed_lidar}">
-    <xacro:sensor_arch prefix="" parent="top_plate_link" size="$(arg sensor_arch_height)">
+    <xacro:sensor_arch prefix="$(arg tf_prefix)" parent="$(arg tf_prefix)top_plate_link" size="$(arg sensor_arch_height)">
         <origin xyz="$(optenv HUSKY_SENSOR_ARCH_OFFSET 0 0 0)" rpy="$(optenv HUSKY_SENSOR_ARCH_RPY 0 0 0)"/>
       </xacro:sensor_arch>
@@ -188,11 +189,11 @@
   <!-- add the intel realsense to the sensor arch if needed -->
   <xacro:if value="$(arg realsense_enabled)">
-    <link name="realsense_mountpoint"/>
-    <joint name="realsense_mountpoint_joint" type="fixed">
+    <link name="$(arg tf_prefix)realsense_mountpoint"/>
+    <joint name="$(arg tf_prefix)realsense_mountpoint_joint" type="fixed">
       <origin xyz="$(arg realsense_xyz)" rpy="$(arg realsense_rpy)" />
-      <parent link="$(arg realsense_mount)"/>
-      <child link="realsense_mountpoint" />
+      <parent link="$(arg tf_prefix)$(arg realsense_mount)"/>
+      <child link="$(arg tf_prefix)realsense_mountpoint" />
     </joint>
-    <xacro:intel_realsense_mount prefix="camera" topic="realsense" parent_link="realsense_mountpoint"/>
+    <xacro:intel_realsense_mount prefix="$(arg tf_prefix)camera" topic="realsense" parent_link="$(arg tf_prefix)realsense_mountpoint"/>
   </xacro:if>
   <!--
@@ -200,5 +201,5 @@
   -->
   <xacro:if value="$(arg laser_3d_enabled)">
-    <xacro:vlp16_mount prefix="" parent_link="sensor_arch_mount_link" topic="$(optenv HUSKY_LASER_3D_TOPIC points)">
+    <xacro:vlp16_mount prefix="$(arg tf_prefix)" parent_link="$(arg tf_prefix)sensor_arch_mount_link" topic="$(optenv HUSKY_LASER_3D_TOPIC points)">
       <origin xyz="$(arg laser_3d_xyz)" rpy="$(arg laser_3d_rpy)" />
     </xacro:vlp16_mount>

File: husky_description/urdf/wheel.urdf.xacro (robot description, xacro)
@@ -22,6 +22,6 @@
 -->
 <robot xmlns:xacro="http://ros.org/wiki/xacro" name="husky_wheel">
-	<xacro:macro name="husky_wheel" params="wheel_prefix *joint_pose">
-		<link name="${wheel_prefix}_wheel_link">
+	<xacro:macro name="husky_wheel" params="wheel_prefix tf_prefix *joint_pose">
+		<link name="${tf_prefix}${wheel_prefix}_wheel_link">
 			<inertial>
 				<mass value="2.637" />
@@ -42,5 +42,5 @@
 			</collision>
 		</link>
-		<gazebo reference="${wheel_prefix}_wheel_link">
+		<gazebo reference="${tf_prefix}${wheel_prefix}_wheel_link">
 			<mu1 value="1.0"/>
 			<mu2 value="1.0"/>
@@ -49,16 +49,16 @@
 			<fdir1 value="1 0 0"/>
 		</gazebo>
-		<joint name="${wheel_prefix}_wheel" type="continuous">
-			<parent link="base_link"/>
-			<child link="${wheel_prefix}_wheel_link"/>
+		<joint name="${tf_prefix}${wheel_prefix}_wheel" type="continuous">
+                  <parent link="${tf_prefix}base_link"/>
+			<child link="${tf_prefix}${wheel_prefix}_wheel_link"/>
 			<xacro:insert_block name="joint_pose"/>
 			<axis xyz="0 1 0" rpy="0 0 0" />
 		</joint>
-		<transmission name="${wheel_prefix}_wheel_trans" type="SimpleTransmission">
+		<transmission name="${tf_prefix}${wheel_prefix}_wheel_trans" type="SimpleTransmission">
 			<type>transmission_interface/SimpleTransmission</type>
-			<actuator name="${wheel_prefix}_wheel_motor">
+			<actuator name="${tf_prefix}${wheel_prefix}_wheel_motor">
 				<mechanicalReduction>1</mechanicalReduction>
 			</actuator>
-			<joint name="${wheel_prefix}_wheel">
+			<joint name="${tf_prefix}${wheel_prefix}_wheel">
 				<hardwareInterface>hardware_interface/VelocityJointInterface</hardwareInterface>
 			</joint>
