Commit message: Add lidar link

File: husky_description/urdf/husky_macro.urdf.xacro (robot description, xacro)
@@ -83,4 +83,10 @@
     <gazebo reference="${prefix}imu_link">
     </gazebo>
+    <link name="${prefix}lidar_link"/>
+    <joint name="${prefix}lidar_joint" type="fixed">
+      <origin xyz="0.375 0 0.321" rpy="0 0 0" />
+      <parent link="${prefix}base_link" />
+      <child link="${prefix}lidar_link" />
+    </joint>
     <!-- Husky wheel macros -->
     <xacro:husky_wheel wheel_prefix="${prefix}front_left">

Commit message: Initial accessories launch file.

File: husky_description/urdf/husky_macro.urdf.xacro (robot description, xacro)
@@ -77,5 +77,5 @@
     <link name="${prefix}imu_link"/>
     <joint name="${prefix}imu_joint" type="fixed">
-      <origin xyz="$(optenv HUSKY_IMU_XYZ 0.19 0 0.149)" rpy="$(optenv HUSKY_IMU_RPY 0 -1.5708 3.1416)" />
+      <origin xyz="$(optenv CPR_IMU_XYZ 0.19 0 0.149)" rpy="$(optenv CPR_IMU_RPY 0 -1.5708 3.1416)" />
       <parent link="${prefix}base_link" />
       <child link="${prefix}imu_link" />

Commit message: Switched to gazebo_plugins for IMU and GPS.

File: husky_description/urdf/husky_macro.urdf.xacro (robot description, xacro)
@@ -73,14 +73,20 @@
       <child link="${prefix}inertial_link" />
     </joint>
-    <!-- IMU Link is the standard mounting position for the UM6 IMU.-->
+    <!-- IMU Link-->
     <!-- Can be modified with environment variables in /etc/ros/setup.bash -->
     <link name="${prefix}imu_link"/>
     <joint name="${prefix}imu_joint" type="fixed">
-      <origin xyz="$(optenv CPR_IMU_XYZ 0.19 0 0.149)" rpy="$(optenv CPR_IMU_RPY 0 -1.5708 3.1416)" />
+      <origin xyz="$(optenv CPR_IMU_XYZ 0 0 0)" rpy="$(optenv CPR_IMU_RPY 0 0 0)" />
       <parent link="${prefix}base_link" />
       <child link="${prefix}imu_link" />
     </joint>
-    <gazebo reference="${prefix}imu_link">
-    </gazebo>
+    <!-- GPS Link-->
+    <!-- Can be modified with environment variables in /etc/ros/setup.bash -->
+    <link name="${prefix}gps_link"/>
+    <joint name="${prefix}gps_joint" type="fixed">
+      <origin xyz="$(optenv CPR_GPS_XYZ 0 0 0)" rpy="$(optenv CPR_GPS_RPY 0 0 0)" />
+      <parent link="${prefix}base_link" />
+      <child link="${prefix}gps_link" />
+    </joint>
     <!-- Husky wheel macros -->
     <xacro:husky_wheel wheel_prefix="${prefix}front_left">

Commit message: Changed URDF to use package rather than file.

File: husky_description/urdf/husky_macro.urdf.xacro (robot description, xacro)
@@ -37,5 +37,5 @@
         <origin xyz="0 0 0" rpy="0 0 0" />
         <geometry>
-          <mesh filename="file://$(find husky_description)/meshes/base_link.dae" />
+          <mesh filename="package://husky_description/meshes/base_link.dae" />
         </geometry>
       </visual>

Commit message: Add missing usage of realsense_xyz and realsense_rpy xacro arguments in realsense joint

File: husky_description/urdf/husky_macro.urdf.xacro (robot description, xacro)
@@ -127,5 +127,5 @@
       <link name="realsense_mountpoint"/>
       <joint name="realsense_mountpoint_joint" type="fixed">
-        <origin xyz="0 0 0" rpy="0 0 -3.14159" />
+        <origin xyz="$(arg realsense_xyz)" rpy="$(arg realsense_rpy)" />
         <parent link="$(arg realsense_mount)"/>
         <child link="realsense_mountpoint" />

Commit message: Changes for IIDT06.

File: husky_description/urdf/husky_macro.urdf.xacro (robot description, xacro)
@@ -1,22 +1,22 @@
 <?xml version="1.0"?>
 <robot xmlns:xacro="http://ros.org/wiki/xacro">
-  <xacro:arg name="laser_enabled" default="false" />
-  <xacro:arg name="laser_xyz" default="$(optenv HUSKY_LMS1XX_XYZ 0.2206 0.0 0.00635)" />
-  <xacro:arg name="laser_rpy" default="$(optenv HUSKY_LMS1XX_RPY 0.0 0.0 0.0)" />
-  <xacro:arg name="realsense_enabled" default="false" />
-  <xacro:arg name="realsense_xyz" default="$(optenv HUSKY_REALSENSE_XYZ 0 0 0)" />
-  <xacro:arg name="realsense_rpy" default="$(optenv HUSKY_REALSENSE_RPY 0 0 0)" />
-  <xacro:arg name="realsense_mount" default="$(optenv HUSKY_REALSENSE_MOUNT_FRAME sensor_arch_mount_link)" />
+  <xacro:arg name="laser_enabled" default="$(optenv CPR_LASER_ENABLED 0)" />
+  <xacro:arg name="laser_xyz" default="$(optenv CPR_LASER_XYZ 0.2206 0.0 0.00635)" />
+  <xacro:arg name="laser_rpy" default="$(optenv CPR_LASER_RPY 0.0 0.0 0.0)" />
+  <xacro:arg name="realsense_enabled" default="$(optenv CPR_REALSENSE 0)" />
+  <xacro:arg name="realsense_xyz" default="$(optenv CPR_REALSENSE_XYZ 0 0 0)" />
+  <xacro:arg name="realsense_rpy" default="$(optenv CPR_REALSENSE_RPY 0 0 0)" />
+  <xacro:arg name="realsense_mount" default="$(optenv CPR_REALSENSE_MOUNT_FRAME sensor_arch_mount_link)" />
   <xacro:property name="husky_front_bumper_extend" value="$(optenv HUSKY_FRONT_BUMPER_EXTEND 0)" />
   <xacro:property name="husky_rear_bumper_extend" value="$(optenv HUSKY_REAR_BUMPER_EXTEND 0)" />
   <xacro:arg name="robot_namespace" default="/" />
   <xacro:arg name="is_sim" default="false" />
-  <xacro:arg name="urdf_extras" default="empty.urdf" />
+  <xacro:arg name="urdf_extras" default="$(optenv CPR_URDF_EXTRAS empty.urdf)" />
   <!-- Included URDF/XACRO Files -->
   <xacro:include filename="$(find husky_description)/urdf/decorations.urdf.xacro" />
   <xacro:include filename="$(find husky_description)/urdf/wheel.urdf.xacro" />
-  <!-- <xacro:include filename="$(find husky_description)/urdf/accessories/intel_realsense.urdf.xacro"/>
-  <xacro:include filename="$(find husky_description)/urdf/accessories/sick_lms1xx_mount.urdf.xacro"/>
-  <xacro:include filename="$(find husky_description)/urdf/accessories/sensor_arch.urdf.xacro"/> -->
+  <xacro:include filename="$(find husky_description)/urdf/accessories/intel_realsense.urdf.xacro"/>
+  <!-- <xacro:include filename="$(find husky_description)/urdf/accessories/sick_lms1xx_mount.urdf.xacro"/> -->
+  <xacro:include filename="$(find husky_description)/urdf/accessories/sensor_arch.urdf.xacro"/>
   <xacro:property name="M_PI" value="3.14159"/>
   <xacro:macro name="husky" params="prefix">
@@ -37,5 +37,5 @@
         <origin xyz="0 0 0" rpy="0 0 0" />
         <geometry>
-          <mesh filename="file://$(find husky_description)/meshes/base_link.dae" />
+          <mesh filename="package://husky_description/meshes/base_link.dae" />
         </geometry>
       </visual>
@@ -124,13 +124,13 @@
     </xacro:if> -->
     <!-- add the intel realsense to the topbar if needed -->
-    <!-- <xacro:if value="$(arg realsense_enabled)">
+    <xacro:if value="$(arg realsense_enabled)">
       <link name="realsense_mountpoint"/>
       <joint name="realsense_mountpoint_joint" type="fixed">
-        <origin xyz="0 0 0" rpy="0 0 -3.14159" />
+        <origin xyz="$(arg realsense_xyz)" rpy="$(arg realsense_rpy)" />
         <parent link="$(arg realsense_mount)"/>
         <child link="realsense_mountpoint" />
       </joint>
       <xacro:intel_realsense_mount prefix="camera" topic="realsense" parent_link="realsense_mountpoint"/>
-    </xacro:if> -->
+    </xacro:if>
     <ros2_control name="${prefix}husky_hardware" type="system">
       <hardware>
