Commit message: Make base_footprint a child of base_link

File: husky_description/urdf/husky.urdf.xacro (robot description, xacro)
@@ -45,15 +45,5 @@
   <xacro:property name="wheel_radius" value="0.17775" />
   <xacro:macro name="husky_robot">
-    <!-- Base link is on the ground under the robot -->
-    <link name="base_footprint"/>
-    <gazebo reference="base_footprint">
-      <material>Gazebo/DarkGrey</material>
-    </gazebo>
-    <joint name="chassis_joint" type="fixed">
-      <origin xyz="0 0 ${wheel_radius - wheel_vertical_offset}" rpy="0 0 0" />
-      <parent link="base_footprint" />
-      <child link="base_link" />
-    </joint>
-    <!-- Chassis link is the center of the robot's bottom plate -->
+    <!-- Base link is the center of the robot's bottom plate -->
     <link name="base_link">
       <visual>
@@ -76,4 +66,17 @@
         </geometry>
       </collision>
+    </link>
+    <gazebo reference="base_link">
+      <material>Gazebo/DarkGrey</material>
+    </gazebo>
+    <!-- Base footprint is on the ground under the robot -->
+    <link name="base_footprint"/>
+    <joint name="base_footprint_joint" type="fixed">
+      <origin xyz="0 0 ${wheel_vertical_offset - wheel_radius}" rpy="0 0 0" />
+      <parent link="base_link" />
+      <child link="base_footprint" />
+    </joint>
+    <!-- Interial link stores the robot's inertial information -->
+    <link name="inertial_link">
       <inertial>
         <mass value="33.455" />
@@ -82,6 +85,9 @@
       </inertial>
     </link>
-    <gazebo reference="base_link">
-    </gazebo>
+    <joint name="inertial_joint" type="fixed">
+      <origin xyz="0 0 0" rpy="0 0 0" />
+      <parent link="base_link" />
+      <child link="inertial_link" />
+    </joint>
     <!-- IMU Link is the standard mounting position for the UM6 IMU.-->
     <!-- Can be modified with environment variables in /etc/ros/setup.bash -->

Commit message: Port *.stl to *.dae format, removing material/gazebo colours

File: husky_description/urdf/husky.urdf.xacro (robot description, xacro)
@@ -24,12 +24,9 @@
   <!-- Included URDF/XACRO Files -->
   <xacro:include filename="$(find husky_description)/urdf/decorations.urdf.xacro" />
+  <xacro:include filename="$(find husky_description)/urdf/wheel.urdf.xacro" />
   <xacro:include filename="$(find husky_description)/urdf/accessories/kinect_camera.urdf.xacro"/>
   <xacro:include filename="$(find husky_description)/urdf/accessories/sick_lms100.urdf.xacro"/>
   <xacro:include filename="$(find husky_description)/urdf/accessories/sensor_arch.urdf.xacro"/>
-  <!-- <xacro:include filename="$(find robotiq_c2_model_visualization)/urdf/robotiq_c2_model_macro.xacro"/> -->
   <xacro:include filename="$(find ur_description)/urdf/ur5.urdf.xacro" />
-  <!-- Included URDF/XACRO Files -->
-  <xacro:include filename="$(find husky_description)/urdf/materials.urdf" />
-  <xacro:include filename="$(find husky_description)/urdf/wheel.urdf.xacro" />
   <property name="M_PI" value="3.14159"/>
   <!-- Base Size -->
@@ -50,7 +47,6 @@
         <origin xyz="0 0 0" rpy="0 0 0" />
         <geometry>
-          <mesh filename="package://husky_description/meshes/base_link.stl" />
+          <mesh filename="package://husky_description/meshes/base_link.dae" />
         </geometry>
-        <material name="Black" />
       </visual>
       <collision>
@@ -67,7 +63,4 @@
       </collision>
     </link>
-    <gazebo reference="base_link">
-      <material>Gazebo/DarkGrey</material>
-    </gazebo>
     <!-- Base footprint is on the ground under the robot -->
     <link name="base_footprint"/>

Commit message: Custom tunining for dual lidar husky.

File: husky_description/urdf/husky.urdf.xacro (robot description, xacro)
@@ -36,9 +36,9 @@
   <!-- Wheel Mounting Positions -->
   <xacro:property name="wheelbase" value="0.5120" />
-  <xacro:property name="track" value="0.5708" />
+  <xacro:property name="track" value="0.5603" />
   <xacro:property name="wheel_vertical_offset" value="0.03282" />
   <!-- Wheel Properties -->
   <xacro:property name="wheel_length" value="0.1143" />
-  <xacro:property name="wheel_radius" value="0.17775" />
+  <xacro:property name="wheel_radius" value="0.16" />
   <xacro:macro name="husky_robot">
     <!-- Base link is the center of the robot's bottom plate -->
@@ -87,5 +87,5 @@
     <link name="imu_link"/>
     <joint name="imu_joint" type="fixed">
-      <origin xyz="$(optenv HUSKY_IMU_XYZ 0.19 0 0.149)" rpy="$(optenv HUSKY_IMU_RPY 0 -1.5708 3.1416)" />
+      <origin xyz="$(optenv HUSKY_IMU_XYZ -0.2 0 0)" rpy="$(optenv HUSKY_IMU_RPY 3.14159 0 0)" />
       <parent link="base_link" />
       <child link="imu_link" />

Commit message: Add 2wheel config option

File: husky_description/urdf/husky.urdf.xacro (robot description, xacro)
@@ -41,5 +41,5 @@
   <xacro:property name="wheel_length" value="0.1143" />
   <xacro:property name="wheel_radius" value="0.17775" />
-  <xacro:macro name="husky_robot">
+  <xacro:macro name="husky_robot" params="wheelconfig">
     <!-- Base link is the center of the robot's bottom plate -->
     <link name="base_link">
@@ -94,16 +94,26 @@
     </gazebo>
     <!-- Husky wheel macros -->
-    <xacro:husky_wheel wheel_prefix="front_left">
+    <xacro:husky_wheel wheel_prefix="front_left" fixed="false">
       <origin xyz="${wheelbase/2} ${track/2} ${wheel_vertical_offset}" rpy="0 0 0" />
     </xacro:husky_wheel>
-    <xacro:husky_wheel wheel_prefix="front_right">
+    <xacro:husky_wheel wheel_prefix="front_right" fixed="false">
       <origin xyz="${wheelbase/2} ${-track/2} ${wheel_vertical_offset}" rpy="0 0 0" />
     </xacro:husky_wheel>
-    <xacro:husky_wheel wheel_prefix="rear_left">
-      <origin xyz="${-wheelbase/2} ${track/2} ${wheel_vertical_offset}" rpy="0 0 0" />
-    </xacro:husky_wheel>
-    <xacro:husky_wheel wheel_prefix="rear_right">
-      <origin xyz="${-wheelbase/2} ${-track/2} ${wheel_vertical_offset}" rpy="0 0 0" />
-    </xacro:husky_wheel>
+    <xacro:if value="${wheelconfig_full}">
+	    <xacro:husky_wheel wheel_prefix="rear_left" fixed="false">
+	      <origin xyz="${-wheelbase/2} ${track/2} ${wheel_vertical_offset}" rpy="0 0 0" />
+	    </xacro:husky_wheel>
+	    <xacro:husky_wheel wheel_prefix="rear_right" fixed="false">
+	      <origin xyz="${-wheelbase/2} ${-track/2} ${wheel_vertical_offset}" rpy="0 0 0" />
+	    </xacro:husky_wheel>
+	  </xacro:if>
+	  <xacro:unless value="${wheelconfig_full}">
+      <xacro:husky_wheel wheel_prefix="rear_left" fixed="true">
+        <origin xyz="${-wheelbase/2} ${track/2} ${wheel_vertical_offset}" rpy="0 0 0" />
+      </xacro:husky_wheel>
+      <xacro:husky_wheel wheel_prefix="rear_right" fixed="true">
+        <origin xyz="${-wheelbase/2} ${-track/2} ${wheel_vertical_offset}" rpy="0 0 0" />
+      </xacro:husky_wheel>
+	  </xacro:unless>
     <xacro:husky_decorate />
     <xacro:if value="$(arg ur5_enabled)">

File: husky_description/urdf/wheel.urdf.xacro (robot description, xacro)
@@ -22,5 +22,5 @@
 -->
 <robot xmlns:xacro="http://ros.org/wiki/xacro" name="husky_wheel">
-	<xacro:macro name="husky_wheel" params="wheel_prefix *joint_pose">
+	<xacro:macro name="husky_wheel" params="wheel_prefix fixed *joint_pose">
 		<link name="${wheel_prefix}_wheel_link">
 			<inertial>
@@ -42,26 +42,42 @@
 			</collision>
 		</link>
-		<gazebo reference="${wheel_prefix}_wheel_link">
-			<mu1 value="1.0"/>
-			<mu2 value="1.0"/>
-			<kp value="10000000.0" />
-			<kd value="1.0" />
-			<fdir1 value="1 0 0"/>
-		</gazebo>
-		<joint name="${wheel_prefix}_wheel" type="continuous">
-			<parent link="base_link"/>
-			<child link="${wheel_prefix}_wheel_link"/>
-			<xacro:insert_block name="joint_pose"/>
-			<axis xyz="0 1 0" rpy="0 0 0" />
-		</joint>
-		<transmission name="${wheel_prefix}_wheel_trans" type="SimpleTransmission">
-			<type>transmission_interface/SimpleTransmission</type>
-			<actuator name="${wheel_prefix}_wheel_motor">
-				<mechanicalReduction>1</mechanicalReduction>
-			</actuator>
-			<joint name="${wheel_prefix}_wheel">
-				<hardwareInterface>VelocityJointInterface</hardwareInterface>
-			</joint>
-		</transmission>
+    <xacro:if value="${fixed}">
+      <gazebo reference="${wheel_prefix}_wheel_link">
+        <mu1 value="0.0"/>
+        <mu2 value="0.0"/>
+        <kp value="10000000.0" />
+        <kd value="1.0" />
+      </gazebo>
+      <joint name="${wheel_prefix}_wheel" type="fixed">
+        <parent link="base_link"/>
+        <child link="${wheel_prefix}_wheel_link"/>
+        <xacro:insert_block name="joint_pose"/>
+        <axis xyz="0 1 0" rpy="0 0 0" />
+      </joint>
+    </xacro:if>
+    <xacro:unless value="${fixed}">
+	    <gazebo reference="${wheel_prefix}_wheel_link">
+	      <mu1 value="1.0"/>
+	      <mu2 value="1.0"/>
+	      <kp value="10000000.0" />
+	      <kd value="1.0" />
+	      <fdir1 value="1 0 0"/>
+	    </gazebo>
+	    <joint name="${wheel_prefix}_wheel" type="continuous">
+	      <parent link="base_link"/>
+	      <child link="${wheel_prefix}_wheel_link"/>
+	      <xacro:insert_block name="joint_pose"/>
+	      <axis xyz="0 1 0" rpy="0 0 0" />
+	    </joint>
+	    <transmission name="${wheel_prefix}_wheel_trans" type="SimpleTransmission">
+	      <type>transmission_interface/SimpleTransmission</type>
+	      <actuator name="${wheel_prefix}_wheel_motor">
+	        <mechanicalReduction>1</mechanicalReduction>
+	      </actuator>
+	      <joint name="${wheel_prefix}_wheel">
+	        <hardwareInterface>VelocityJointInterface</hardwareInterface>
+	      </joint>
+	    </transmission>
+    </xacro:unless>
 	</xacro:macro>
 </robot>

Commit message: remove laser and ur5

File: husky_description/urdf/husky.urdf.xacro (robot description, xacro)
@@ -26,7 +26,5 @@
   <xacro:include filename="$(find husky_description)/urdf/wheel.urdf.xacro" />
   <xacro:include filename="$(find husky_description)/urdf/accessories/kinect_camera.urdf.xacro"/>
-  <xacro:include filename="$(find husky_description)/urdf/accessories/sick_lms1xx_mount.urdf.xacro"/>
   <xacro:include filename="$(find husky_description)/urdf/accessories/sensor_arch.urdf.xacro"/>
-  <xacro:include filename="$(find ur_description)/urdf/ur5.urdf.xacro" />
   <property name="M_PI" value="3.14159"/>
   <!-- Base Size -->
@@ -117,24 +115,4 @@
 	  </xacro:unless>
     <xacro:husky_decorate />
-    <xacro:if value="$(arg ur5_enabled)">
-      <xacro:property name="reflect" value="-1" />
-      <!-- Spawn arm -->
-      <xacro:ur5_robot prefix="ur5_arm_" joint_limited="true"/>
-      <!-- Join arm -->
-      <joint name="ur5_arm_base" type="fixed">
-        <parent link="top_plate_link" />
-        <child link="ur5_arm_base_link" />
-        <origin xyz="0.3058 0 0.0065" rpy="0.0 0.0 -1.57" />
-      </joint>
-    </xacro:if>
-    <xacro:if value="$(arg laser_enabled)">
-      <sick_lms1xx_mount prefix="base" topic="scan"/>
-      <joint name="laser_mount_joint" type="fixed">
-        <origin xyz="$(optenv HUSKY_LMS1XX_XYZ 0.2206 0.0 0.00635)"
-                rpy="$(optenv HUSKY_LMS1XX_RPY 0.0 0.0 0.0)" />
-        <parent link="top_plate_link" />
-        <child link="base_laser_mount" />
-      </joint>
-    </xacro:if>
     <xacro:if value="$(arg kinect_enabled)">
       <xacro:sensor_arch prefix="" parent="top_plate_link">

Commit message: Change inertia link name

File: husky_description/urdf/husky.urdf.xacro (robot description, xacro)
@@ -69,5 +69,5 @@
     </joint>
     <!-- Interial link stores the robot's inertial information -->
-    <link name="inertial_link">
+    <link name="base_link_inertia">
       <inertial>
         <mass value="33.455" />
@@ -79,5 +79,5 @@
       <origin xyz="0 0 0" rpy="0 0 0" />
       <parent link="base_link" />
-      <child link="inertial_link" />
+      <child link="base_link_inertia" />
     </joint>
     <!-- IMU Link is the standard mounting position for the UM6 IMU.-->

Commit message: Added the joints for the bulkheead to arm

File: husky_description/urdf/husky.urdf.xacro (robot description, xacro)
@@ -129,5 +129,5 @@
         <!-- Join left arm to top plate -->
         <joint name="l_ur5_arm_base" type="fixed"/>
-            <parent link="modified_top_plate_link"/>
+            <parent link="dual_arm_bulkhead_link"/>
             <child link="l_ur5_arm_base_link" />
             <origin xyz="0 0 0" rpy="0 0 0"/>
@@ -135,5 +135,5 @@
          <!-- Joint right arm to top plate -->
         <joint name="r_ur5_arm_base" type="fixed">
-            <parent link="modified_top_plate_link"/>
+            <parent link="dual_arm_bulkhead_link"/>
             <child link="r_ur5_arm_base_link" />
             <origin xyz="0 0 0" rpy="0 0 0"/>

Commit message: fixed slash syntax

File: husky_description/urdf/husky.urdf.xacro (robot description, xacro)
@@ -114,5 +114,5 @@
             <!-- Left gripper -->
             <xacro:s-model_articulated prefix="l_"/>
-            <joint name="l_palm_to_l_ur5" type="fixed"/>
+            <joint name="l_palm_to_l_ur5" type="fixed">
                 <parent link="l_ur5_arm_ee_link"/>
                 <child link="l_palm"/>
@@ -121,5 +121,5 @@
             <!-- Right gripper -->
             <xacro:s-model_articulated prefix="r_"/>
-            <joint name="r_palm_to_r_ur5" type="fixed"/>
+            <joint name="r_palm_to_r_ur5" type="fixed">
                 <parent link="r_ur5_arm_ee_link"/>
                 <child link="r_palm"/>
@@ -128,5 +128,5 @@
         </xacro:if>
         <!-- Join left arm to top plate -->
-        <joint name="l_ur5_arm_base" type="fixed"/>
+        <joint name="l_ur5_arm_base" type="fixed">
             <parent link="dual_arm_bulkhead_link"/>
             <child link="l_ur5_arm_base_link" />

Commit message: Right arm positioned correctly

File: husky_description/urdf/husky.urdf.xacro (robot description, xacro)
@@ -128,13 +128,13 @@
         </xacro:if>
         <!-- Join left arm to top plate -->
+        <joint name="r_ur5_arm_base" type="fixed">
+            <parent link="dual_arm_bulkhead_link"/>
+            <child link="r_ur5_arm_base_link" />
+            <origin xyz="0.125 -0.15 0.135" rpy="0 0.785 -1.57"/>
+        </joint>
+         <!-- Joint right arm to top plate -->
         <joint name="l_ur5_arm_base" type="fixed">
             <parent link="dual_arm_bulkhead_link"/>
             <child link="l_ur5_arm_base_link" />
-            <origin xyz="0.125 -0.15 0.135" rpy="0.785 0 0"/>
-        </joint>
-         <!-- Joint right arm to top plate -->
-        <joint name="r_ur5_arm_base" type="fixed">
-            <parent link="dual_arm_bulkhead_link"/>
-            <child link="r_ur5_arm_base_link" />
             <origin xyz="0.125 0.15 0.135" rpy="-0.785 0 0"/>
         </joint>

Commit message: Positioned left arm for gazebo

File: husky_description/urdf/husky.urdf.xacro (robot description, xacro)
@@ -137,5 +137,5 @@
             <parent link="dual_arm_bulkhead_link"/>
             <child link="l_ur5_arm_base_link" />
-            <origin xyz="0.125 0.15 0.135" rpy="-0.785 0 0"/>
+            <origin xyz="0.125 0.15 0.135" rpy="0 -0.785 -1.57"/>
         </joint>
     </xacro:if>

Commit message: positioned grippers

File: husky_description/urdf/husky.urdf.xacro (robot description, xacro)
@@ -118,5 +118,5 @@
                 <parent link="l_ur5_arm_ee_link"/>
                 <child link="l_palm"/>
-                <origin xyz="0 0 0" rpy="0 0 0"/>
+                <origin xyz="0 0 0" rpy="0 0 -1.57"/>
             </joint>
             <!-- Right gripper -->
@@ -124,5 +124,5 @@
                 <parent link="r_ur5_arm_ee_link"/>
                 <child link="r_palm"/>
-                <origin xyz="0 0 0" rpy="0 0 0"/>
+                <origin xyz="0 0 0" rpy="0 0 -1.57"/>
             </joint>
         </xacro:if>

Commit message: Changed to use a different hand with a gazebo plugin

File: husky_description/urdf/husky.urdf.xacro (robot description, xacro)
@@ -29,5 +29,5 @@
   <xacro:include filename="$(find husky_description)/urdf/accessories/sensor_arch.urdf.xacro"/>
   <xacro:include filename="$(find ur_description)/urdf/ur5.urdf.xacro" />
-  <xacro:include filename="$(find robotiq_s_model_visualization)/cfg/s-model_articulated_macro.xacro"/>
+  <xacro:include filename="$(find robotiq_s_model_visualization)/cfg/robotiq_hand_macro.urdf.xacro"/>
   <property name="M_PI" value="3.14159"/>
   <!-- Base Size -->
@@ -112,18 +112,10 @@
         <xacro:ur5_robot prefix="r_ur5_arm_" joint_limited="true"/>
         <xacro:if value="$(arg robotiq_grippers_enabled)">
-            <xacro:s-model_articulated prefix="l_"/>
-            <xacro:s-model_articulated prefix="r_"/>
-            <!-- Left gripper -->
-            <joint name="l_palm_to_l_ur5" type="fixed">
-                <parent link="l_ur5_arm_ee_link"/>
-                <child link="l_palm"/>
-                <origin xyz="0 0 0" rpy="0 0 -1.57"/>
-            </joint>
-            <!-- Right gripper -->
-            <joint name="r_palm_to_r_ur5" type="fixed">
-                <parent link="r_ur5_arm_ee_link"/>
-                <child link="r_palm"/>
-                <origin xyz="0 0 0" rpy="0 0 -1.57"/>
-            </joint>
+            <xacro:robotiq_hand prefix="l_" reflect="1" parent="l_ur5_arm_ee_link">
+                <origin xyz="0 0 0" rpy="0 0 0"/>
+            </xacro:robotiq_hand>
+            <xacro:robotiq_hand prefix="r_" reflect="-1" parent="r_ur5_arm_ee_link">
+                <origin xyz="0 0 0" rpy="0 0 0"/>
+            </xacro:robotiq_hand>
         </xacro:if>
         <!-- Join left arm to top plate -->

Commit message: Updated position of grippers

File: husky_description/urdf/husky.urdf.xacro (robot description, xacro)
@@ -113,8 +113,8 @@
         <xacro:if value="$(arg robotiq_grippers_enabled)">
             <xacro:robotiq_hand prefix="l_" reflect="1" parent="l_ur5_arm_ee_link">
-                <origin xyz="0 0 0" rpy="0 0 0"/>
+                <origin xyz="0 0 0" rpy="0 0 -1.57"/>
             </xacro:robotiq_hand>
-            <xacro:robotiq_hand prefix="r_" reflect="-1" parent="r_ur5_arm_ee_link">
-                <origin xyz="0 0 0" rpy="0 0 0"/>
+            <xacro:robotiq_hand prefix="r_" reflect="1" parent="r_ur5_arm_ee_link">
+                <origin xyz="0 0 0" rpy="0 0 -1.57"/>
             </xacro:robotiq_hand>
         </xacro:if>

Commit message: Updated grpiper position for ft

File: husky_description/urdf/husky.urdf.xacro (robot description, xacro)
@@ -113,8 +113,8 @@
         <xacro:if value="$(arg robotiq_grippers_enabled)">
             <xacro:robotiq_hand prefix="l_" reflect="1" parent="l_ur5_arm_ee_link">
-                <origin xyz="0 0 0" rpy="0 0 -1.57"/>
+                <origin xyz="0.062 0 0" rpy="0 0 -1.57"/>
             </xacro:robotiq_hand>
             <xacro:robotiq_hand prefix="r_" reflect="1" parent="r_ur5_arm_ee_link">
-                <origin xyz="0 0 0" rpy="0 0 -1.57"/>
+                <origin xyz="0.062 0 0" rpy="0 0 -1.57"/>
             </xacro:robotiq_hand>
         </xacro:if>

Commit message: Added description

File: husky_description/urdf/husky.urdf.xacro (robot description, xacro)
@@ -30,4 +30,5 @@
   <xacro:include filename="$(find ur_description)/urdf/ur5.urdf.xacro" />
   <xacro:include filename="$(find robotiq_s_model_visualization)/cfg/robotiq_hand_macro.urdf.xacro"/>
+  <xacro:include filename="$(find robotiq_force_torque_sensor)/urdf/robotiq_fts150.urdf.xacro"/>
   <property name="M_PI" value="3.14159"/>
   <!-- Base Size -->
@@ -112,9 +113,15 @@
         <xacro:ur5_robot prefix="r_ur5_arm_" joint_limited="true"/>
         <xacro:if value="$(arg robotiq_grippers_enabled)">
-            <xacro:robotiq_hand prefix="l_" reflect="1" parent="l_ur5_arm_ee_link">
-                <origin xyz="0.062 0 0" rpy="0 0 -1.57"/>
+            <xacro:robotiq_fts150 parent="l_ur5_arm_ee_link" prefix="l_">
+                <origin xyz="0 0 0" rpy="0 0 -1.57"/>
+            </xacro:robotiq_fts150>
+            <xacro:robotiq_fts150 parent="r_ur_arm_ee_link" prefix="r_">
+                <origin xyz="0 0 0" rpy="0 0 -1.57"/>
+            </xacro:robotiq_fts150>
+            <xacro:robotiq_hand prefix="l_" reflect="1" parent="l_fts_toolside">
+                <origin xyz="0 0 0" rpy="0 0 -1.57"/>
             </xacro:robotiq_hand>
-            <xacro:robotiq_hand prefix="r_" reflect="1" parent="r_ur5_arm_ee_link">
-                <origin xyz="0.062 0 0" rpy="0 0 -1.57"/>
+            <xacro:robotiq_hand prefix="r_" reflect="1" parent="r_fts_toolside">
+                <origin xyz="0 0 0" rpy="0 0 -1.57"/>
             </xacro:robotiq_hand>
         </xacro:if>

Commit message: updatd

File: husky_description/urdf/husky.urdf.xacro (robot description, xacro)
@@ -30,5 +30,5 @@
   <xacro:include filename="$(find ur_description)/urdf/ur5.urdf.xacro" />
   <xacro:include filename="$(find robotiq_s_model_visualization)/cfg/robotiq_hand_macro.urdf.xacro"/>
-  <xacro:include filename="$(find robotiq_force_torque_sensor)/urdf/robotiq_fts150.urdf.xacro"/>
+ <!-- <xacro:include filename="$(find robotiq_force_torque_sensor)/urdf/robotiq_fts150.urdf.xacro"/> -->
   <property name="M_PI" value="3.14159"/>
   <!-- Base Size -->
@@ -113,15 +113,9 @@
         <xacro:ur5_robot prefix="r_ur5_arm_" joint_limited="true"/>
         <xacro:if value="$(arg robotiq_grippers_enabled)">
-            <xacro:robotiq_fts150 parent="l_ur5_arm_ee_link" prefix="l_">
-                <origin xyz="0 0 0" rpy="0 0 -1.57"/>
-            </xacro:robotiq_fts150>
-            <xacro:robotiq_fts150 parent="r_ur5_arm_ee_link" prefix="r_">
-                <origin xyz="0 0 0" rpy="0 0 -1.57"/>
-            </xacro:robotiq_fts150>
-            <xacro:robotiq_hand prefix="l_" reflect="1" parent="l_fts_toolside">
-                <origin xyz="0 0 0" rpy="0 0 -1.57"/>
+            <xacro:robotiq_hand prefix="l_" reflect="1" parent="l_ur5_arm_ee_link">
+                <origin xyz="0.062 0 0" rpy="0 0 -1.57"/>
             </xacro:robotiq_hand>
-            <xacro:robotiq_hand prefix="r_" reflect="1" parent="r_fts_toolside">
-                <origin xyz="0 0 0" rpy="0 0 -1.57"/>
+            <xacro:robotiq_hand prefix="r_" reflect="1" parent="r_ur5_arm_ee_link">
+                <origin xyz="0.062 0 0" rpy="0 0 -1.57"/>
             </xacro:robotiq_hand>
         </xacro:if>
