Commit message: upd

File: husky_description/urdf/husky.urdf.xacro (robot description, xacro)
@@ -31,4 +31,5 @@
   <xacro:include filename="$(find robotiq_s_model_visualization)/cfg/robotiq_hand_macro.urdf.xacro"/>
  <!-- <xacro:include filename="$(find robotiq_force_torque_sensor)/urdf/robotiq_fts150.urdf.xacro"/> -->
+  <xacro:include filename="$(find flir_ptu_description)/urdf/d46.urdf.xacro"/>
   <property name="M_PI" value="3.14159"/>
   <!-- Base Size -->
@@ -109,4 +110,13 @@
     </xacro:husky_wheel>
     <xacro:husky_decorate />
+    <xacro:if value="$(optenv FLIR_PTU_ENABLED false)">
+         <xacro:ptu_d46 name="husky_ptu_"/>
+        <!-- Connect PTU to Husky bulkhead -->
+         <joint name="husky_ptu_joint" type="fixed">
+             <origin xyz="0 0 0" rpy="0 0 0"/>
+             <parent link="dual_arm_bulkhead_link" />
+             <child link="husky_ptu_base_link" />
+         </joint>
+    </xacro:if>
     <xacro:if value="$(arg dual_ur5_enabled)">
         <xacro:ur5_robot prefix="l_ur5_arm_" joint_limited="true"/>

Commit message: update ptu pos

File: husky_description/urdf/husky.urdf.xacro (robot description, xacro)
@@ -111,8 +111,8 @@
     <xacro:husky_decorate />
     <xacro:if value="$(optenv FLIR_PTU_ENABLED false)">
-         <xacro:ptu_d46 name="husky_ptu_"/>
+         <xacro:ptu_d46 name="husky_ptu"/>
         <!-- Connect PTU to Husky bulkhead -->
          <joint name="husky_ptu_joint" type="fixed">
-             <origin xyz="0 0 0" rpy="0 0 0"/>
+             <origin xyz="0.2 0 0.22" rpy="0 1.57 0"/>
              <parent link="dual_arm_bulkhead_link" />
              <child link="husky_ptu_base_link" />

Commit message: positioned ptu

File: husky_description/urdf/husky.urdf.xacro (robot description, xacro)
@@ -114,5 +114,5 @@
         <!-- Connect PTU to Husky bulkhead -->
          <joint name="husky_ptu_joint" type="fixed">
-             <origin xyz="0.2 0 0.22" rpy="0 1.57 0"/>
+             <origin xyz="0.365 0 0.221" rpy="0 1.57 3.14"/>
              <parent link="dual_arm_bulkhead_link" />
              <child link="husky_ptu_base_link" />

Commit message: Updated

File: husky_description/urdf/husky.urdf.xacro (robot description, xacro)
@@ -111,7 +111,7 @@
     <xacro:husky_decorate />
     <xacro:if value="$(optenv FLIR_PTU_ENABLED false)">
-         <xacro:ptu_d46 name="husky_ptu"/>
-        <!-- Connect PTU to Husky bulkhead -->
-         <joint name="husky_ptu_joint" type="fixed">
+          <xacro:ptu_d46 name="husky_ptu"/>
+          <!-- Connect PTU to Husky bulkhead -->
+          <joint name="husky_ptu_joint" type="fixed">
              <origin xyz="0.365 0 0.221" rpy="0 1.57 3.14"/>
              <parent link="dual_arm_bulkhead_link" />

Commit message: Added ft300

File: husky_description/urdf/husky.urdf.xacro (robot description, xacro)
@@ -30,5 +30,5 @@
   <xacro:include filename="$(find ur_description)/urdf/ur5.urdf.xacro" />
   <xacro:include filename="$(find robotiq_s_model_visualization)/cfg/robotiq_hand_macro.urdf.xacro"/>
- <!-- <xacro:include filename="$(find robotiq_force_torque_sensor)/urdf/robotiq_fts150.urdf.xacro"/> -->
+  <xacro:include filename="$(find robotiq_force_torque_sensor)/urdf/robotiq_fts300.urdf.xacro"/>
   <xacro:include filename="$(find flir_ptu_description)/urdf/d46.urdf.xacro"/>
   <property name="M_PI" value="3.14159"/>
@@ -122,10 +122,17 @@
         <xacro:ur5_robot prefix="l_ur5_arm_" joint_limited="true"/>
         <xacro:ur5_robot prefix="r_ur5_arm_" joint_limited="true"/>
+        <!-- Add force torque model FT300 -->
+        <xacro:robotiq_fts300 parent="l_ur5_arm_ee_link" prefix="l_robotiq_fts300_">
+           <origin xyz="0 0 0" rpy="0 1.57 0"/>
+        </xacro:robotiq_fts300>
+        <xacro:robotiq_fts300 parent="r_ur5_arm_ee_link" prefix="r_robotiq_fts300_">
+           <origin xyz="0 0 0" rpy="0 1.57 0"/>
+        </xacro:robotiq_fts300>
         <xacro:if value="$(arg robotiq_grippers_enabled)">
-            <xacro:robotiq_hand prefix="l_" reflect="1" parent="l_ur5_arm_ee_link">
-                <origin xyz="0.062 0 0" rpy="0 0 -1.57"/>
+            <xacro:robotiq_hand prefix="l_" reflect="1" parent="l_robotiq_fts300_fts_toolside">
+                <origin xyz="0 0 0" rpy="1.57 0 0"/>
             </xacro:robotiq_hand>
-            <xacro:robotiq_hand prefix="r_" reflect="1" parent="r_ur5_arm_ee_link">
-                <origin xyz="0.062 0 0" rpy="0 0 -1.57"/>
+            <xacro:robotiq_hand prefix="r_" reflect="1" parent="r_robotiq_fts300_fts_toolside">
+                <origin xyz="0 0 0" rpy="1.57 0 0"/>
             </xacro:robotiq_hand>
         </xacro:if>

Commit message: Added dnyamic naming for laser pos

File: husky_description/urdf/husky.urdf.xacro (robot description, xacro)
@@ -166,5 +166,5 @@
         <origin xyz="$(optenv HUSKY_LMS1XX_XYZ 0.2206 0.0 0.00635)"
                 rpy="$(optenv HUSKY_LMS1XX_RPY 0.0 0.0 0.0)" />
-        <parent link="top_plate_link" />
+        <parent link="$(optenv HUSKY_LASER_PARENT_LINK top_plate_link)" />
         <child link="base_laser_mount" />
       </joint>

Commit message: Added laser

File: husky_description/urdf/husky.urdf.xacro (robot description, xacro)
@@ -122,4 +122,12 @@
         <xacro:ur5_robot prefix="l_ur5_arm_" joint_limited="true"/>
         <xacro:ur5_robot prefix="r_ur5_arm_" joint_limited="true"/>
+        <!-- Add laser specifically for this mode -->
+        <sick_lms1xx frame="base_laser" topic="scan" />
+        <!-- This offset is from the base of the bracket to the LIDAR's focal point. -->
+        <joint name="base_laser_joint" type="fixed">
+           <origin xyz="0.45 0 0" rpy="${M_PI} 0 0" />
+           <parent link="dual_arm_bulkhead_link" />
+           <child link="base_laser" />
+        </joint>
         <!-- Add force torque model FT300 -->
         <xacro:robotiq_fts300 parent="l_ur5_arm_ee_link" prefix="l_robotiq_fts300_">

Commit message: Laser positioned and added

File: husky_description/urdf/husky.urdf.xacro (robot description, xacro)
@@ -126,5 +126,5 @@
         <!-- This offset is from the base of the bracket to the LIDAR's focal point. -->
         <joint name="base_laser_joint" type="fixed">
-           <origin xyz="0.45 0 0" rpy="${M_PI} 0 0" />
+           <origin xyz="0.465 0 -0.085" rpy="${M_PI} 0 0" />
            <parent link="dual_arm_bulkhead_link" />
            <child link="base_laser" />

Commit message: added camera

File: husky_description/urdf/husky.urdf.xacro (robot description, xacro)
@@ -32,4 +32,5 @@
   <xacro:include filename="$(find robotiq_force_torque_sensor)/urdf/robotiq_fts300.urdf.xacro"/>
   <xacro:include filename="$(find flir_ptu_description)/urdf/d46.urdf.xacro"/>
+  <xacro:include filename="$(find pointgrey_camera_description)/urdf/pointgrey_bumblebee2.urdf.xacro"/>
   <property name="M_PI" value="3.14159"/>
   <!-- Base Size -->
@@ -130,4 +131,11 @@
            <child link="base_laser" />
         </joint>
+        <!-- Add bumblebee camera -->
+       <BB2-08S2C-38 frame="bumblebee2" name="bumblebee2" />
+        <joint name="bumblebee2_mount_joint" type="fixed">
+           <origin xyz="0 0 0" rpy="0 0 0" />
+           <parent link="husky_ptu_mount_link" />
+           <child link="bumblebee2" />
+        </joint>
         <!-- Add force torque model FT300 -->
         <xacro:robotiq_fts300 parent="l_ur5_arm_ee_link" prefix="l_robotiq_fts300_">

Commit message: Positioned camera

File: husky_description/urdf/husky.urdf.xacro (robot description, xacro)
@@ -134,5 +134,5 @@
        <BB2-08S2C-38 frame="bumblebee2" name="bumblebee2" />
         <joint name="bumblebee2_mount_joint" type="fixed">
-           <origin xyz="0 0 0" rpy="0 0 0" />
+           <origin xyz="-0.09 0.02 -0.11" rpy="0 0 0" />
            <parent link="husky_ptu_mount_link" />
            <child link="bumblebee2" />

Commit message: Positoined bb

File: husky_description/urdf/husky.urdf.xacro (robot description, xacro)
@@ -134,5 +134,5 @@
        <BB2-08S2C-38 frame="bumblebee2" name="bumblebee2" />
         <joint name="bumblebee2_mount_joint" type="fixed">
-           <origin xyz="-0.09 0.02 -0.11" rpy="0 0 0" />
+           <origin xyz="-0.075 0.02 -0.10" rpy="0 1.57 0" />
            <parent link="husky_ptu_mount_link" />
            <child link="bumblebee2" />

Commit message: upd

File: husky_description/urdf/husky.urdf.xacro (robot description, xacro)
@@ -134,5 +134,5 @@
        <BB2-08S2C-38 frame="bumblebee2" name="bumblebee2" />
         <joint name="bumblebee2_mount_joint" type="fixed">
-           <origin xyz="-0.075 0.02 -0.10" rpy="0 1.57 0" />
+           <origin xyz="-0.080 0.02 -0.10" rpy="0 1.57 0" />
            <parent link="husky_ptu_mount_link" />
            <child link="bumblebee2" />

Commit message: Camera now upright

File: husky_description/urdf/husky.urdf.xacro (robot description, xacro)
@@ -134,5 +134,5 @@
        <BB2-08S2C-38 frame="bumblebee2" name="bumblebee2" />
         <joint name="bumblebee2_mount_joint" type="fixed">
-           <origin xyz="-0.080 0.02 -0.10" rpy="0 1.57 0" />
+           <origin xyz="-0.080 0.02 -0.10" rpy="3.14 1.57 0" />
            <parent link="husky_ptu_mount_link" />
            <child link="bumblebee2" />

Commit message: Positioned camera so its not tilted

File: husky_description/urdf/husky.urdf.xacro (robot description, xacro)
@@ -134,5 +134,5 @@
        <BB2-08S2C-38 frame="bumblebee2" name="bumblebee2" />
         <joint name="bumblebee2_mount_joint" type="fixed">
-           <origin xyz="-0.080 0.02 -0.10" rpy="3.14 1.57 0" />
+           <origin xyz="-0.079 0.02 -0.10" rpy="3.14 1.57 0" />
            <parent link="husky_ptu_mount_link" />
            <child link="bumblebee2" />

Commit message: positioned bumblebee

File: husky_description/urdf/husky.urdf.xacro (robot description, xacro)
@@ -115,5 +115,5 @@
           <!-- Connect PTU to Husky bulkhead -->
           <joint name="husky_ptu_joint" type="fixed">
-             <origin xyz="0.365 0 0.221" rpy="0 1.57 3.14"/>
+             <origin xyz="0.365 0 0.221" rpy="0 0 0"/>
              <parent link="dual_arm_bulkhead_link" />
              <child link="husky_ptu_base_link" />
@@ -134,5 +134,5 @@
        <BB2-08S2C-38 frame="bumblebee2" name="bumblebee2" />
         <joint name="bumblebee2_mount_joint" type="fixed">
-           <origin xyz="-0.079 0.02 -0.10" rpy="3.14 1.57 0" />
+           <origin xyz="0 0 0.00" rpy="0 0 0" />
            <parent link="husky_ptu_mount_link" />
            <child link="bumblebee2" />

Commit message: Added spacing for grippers

File: husky_description/urdf/husky.urdf.xacro (robot description, xacro)
@@ -147,8 +147,8 @@
         <xacro:if value="$(optenv ROBOTIQ_GRIPPERS_ENABLED false)">
             <xacro:robotiq_hand prefix="l_" reflect="1" parent="l_robotiq_fts300_fts_toolside">
-                <origin xyz="0 0 0" rpy="1.57 0 0"/>
+                <origin xyz="0 0 0.08" rpy="1.57 0 0"/>
             </xacro:robotiq_hand>
             <xacro:robotiq_hand prefix="r_" reflect="1" parent="r_robotiq_fts300_fts_toolside">
-                <origin xyz="0 0 0" rpy="1.57 0 0"/>
+                <origin xyz="0 0 0.08" rpy="1.57 0 0"/>
             </xacro:robotiq_hand>
         </xacro:if>

Commit message: fixed position of ptu

File: husky_description/urdf/husky.urdf.xacro (robot description, xacro)
@@ -115,5 +115,5 @@
           <!-- Connect PTU to Husky bulkhead -->
           <joint name="husky_ptu_joint" type="fixed">
-             <origin xyz="0.365 0 0.221" rpy="0 0 0"/>
+             <origin xyz="0.365 0 0.20" rpy="0 0 0"/>
              <parent link="dual_arm_bulkhead_link" />
              <child link="husky_ptu_base_link" />

Commit message: update

File: husky_description/urdf/husky.urdf.xacro (robot description, xacro)
@@ -115,5 +115,5 @@
           <!-- Connect PTU to Husky bulkhead -->
           <joint name="husky_ptu_joint" type="fixed">
-             <origin xyz="0.365 0 0.221" rpy="0 0 0"/>
+             <origin xyz="0.365 0 0.15" rpy="0 0 0"/>
              <parent link="dual_arm_bulkhead_link" />
              <child link="husky_ptu_base_link" />

Commit message: merged

File: husky_description/urdf/husky.urdf.xacro (robot description, xacro)
@@ -115,9 +115,5 @@
           <!-- Connect PTU to Husky bulkhead -->
           <joint name="husky_ptu_joint" type="fixed">
-<<<<<<< HEAD
-             <origin xyz="0.365 0 0.15" rpy="0 0 0"/>
-=======
              <origin xyz="0.365 0 0.20" rpy="0 0 0"/>
->>>>>>> c7f0ce6cad03176c492bf3487e6330e5ffa1e847
              <parent link="dual_arm_bulkhead_link" />
              <child link="husky_ptu_base_link" />

Commit message: added xacro code

File: husky_description/urdf/husky.urdf.xacro (robot description, xacro)
@@ -140,7 +140,19 @@
     <!-- Enables a back LMS1XX for the Husky. Mainly used in autonomy core config. Laser is spawned inverted. -->
     <xacro:if value="$(optenv BACK_LASER_ENABLED false)">
+     <sick_lms1xx_mount prefix="back" topic="back_scan"/>
+ <joint name="back_laser_mount_joint" type="fixed">
+        <origin xyz="$(optenv HUSKY_LMS1XX_BACK_XYZ 0.1 -0.1 0.1)" rpy="$(optenv HUSKY_LMS1XX_BACK_RPY 0 0 0" />
+        <parent link="base_link"/>
+        <child link="back_laser_mount"/>
+      </joint>
     </xacro:if>
     <!-- Enables a front mounted LMS1xx for the Husky. Mainly used in autonomy core config. Laser is spawned inverted. -->
     <xacro:if value="$(optenv FRONT_LASER_ENABLED false)">
+      <sick_lms1xx_mount prefix="front" topic="front_scan"/>
+      <joint name="front_laser_mount_joint" type="fixed">
+        <origin xyz="$(optenv HUSKY_LMS1XX_FRONT_XYZ 0.1 0.1 0.1)" rpy="$(optenv HUSKY_LMS1XX_FRONT_RPY 0 0 0" />
+        <parent link="base_link"/>
+        <child link="front_laser_mount"/>
+      </joint>
     </xacro:if>
   </xacro:macro>

Commit message: updated position

File: husky_description/urdf/husky.urdf.xacro (robot description, xacro)
@@ -142,5 +142,5 @@
      <sick_lms1xx_mount prefix="back" topic="back_scan"/>
  <joint name="back_laser_mount_joint" type="fixed">
-        <origin xyz="$(optenv HUSKY_LMS1XX_BACK_XYZ 0.1 -0.1 0.1)" rpy="$(optenv HUSKY_LMS1XX_BACK_RPY 0 0 0" />
+        <origin xyz="$(optenv HUSKY_LMS1XX_BACK_XYZ 0.1 -0.1 0.1)" rpy="$(optenv HUSKY_LMS1XX_BACK_RPY 0 0 0)" />
         <parent link="base_link"/>
         <child link="back_laser_mount"/>
@@ -151,5 +151,5 @@
       <sick_lms1xx_mount prefix="front" topic="front_scan"/>
       <joint name="front_laser_mount_joint" type="fixed">
-        <origin xyz="$(optenv HUSKY_LMS1XX_FRONT_XYZ 0.1 0.1 0.1)" rpy="$(optenv HUSKY_LMS1XX_FRONT_RPY 0 0 0" />
+        <origin xyz="$(optenv HUSKY_LMS1XX_FRONT_XYZ 0.1 0.1 0.1)" rpy="$(optenv HUSKY_LMS1XX_FRONT_RPY 0 0 0)" />
         <parent link="base_link"/>
         <child link="front_laser_mount"/>

Commit message: added standard position for autonomy lidars

File: husky_description/urdf/husky.urdf.xacro (robot description, xacro)
@@ -142,5 +142,5 @@
      <sick_lms1xx_mount prefix="back" topic="back_scan"/>
  <joint name="back_laser_mount_joint" type="fixed">
-        <origin xyz="$(optenv HUSKY_LMS1XX_BACK_XYZ 0.1 -0.1 0.1)" rpy="$(optenv HUSKY_LMS1XX_BACK_RPY 0 0 0)" />
+        <origin xyz="$(optenv HUSKY_LMS1XX_BACK_XYZ -0.43 0 -0.1)" rpy="$(optenv HUSKY_LMS1XX_BACK_RPY 0 0 3.14)" />
         <parent link="base_link"/>
         <child link="back_laser_mount"/>
@@ -151,5 +151,5 @@
       <sick_lms1xx_mount prefix="front" topic="front_scan"/>
       <joint name="front_laser_mount_joint" type="fixed">
-        <origin xyz="$(optenv HUSKY_LMS1XX_FRONT_XYZ 0.1 0.1 0.1)" rpy="$(optenv HUSKY_LMS1XX_FRONT_RPY 0 0 0)" />
+        <origin xyz="$(optenv HUSKY_LMS1XX_FRONT_XYZ 0.43 0 -0.1)" rpy="$(optenv HUSKY_LMS1XX_FRONT_RPY 0 0 0)" />
         <parent link="base_link"/>
         <child link="front_laser_mount"/>
