Commit message: Move models directory up to root

File: urdf/base.urdf.xacro (robot description, xacro)
@@ -105,5 +105,5 @@
             <origin xyz="0 0 ${base_z_origin_offset}" rpy="0 0 0" />
             <geometry>
-                <mesh filename="package://husky_description/Media/models/base_link.stl" />
+                <mesh filename="package://husky_description/models/base_link.stl" />
             </geometry>
             <material name="Black" />

File: urdf/parts.urdf.xacro (robot description, xacro)
@@ -62,5 +62,5 @@
 				<origin xyz="0 0 0" rpy="0 0 0" />
 				<geometry>
-					<mesh filename="package://husky_description/Media/models/${mesh}.stl" />
+					<mesh filename="package://husky_description/models/${mesh}.stl" />
 				</geometry>
 				<material name="${colour}" />

File: urdf/wheel.urdf.xacro (robot description, xacro)
@@ -59,5 +59,5 @@
 				<origin xyz="0 0 0" rpy="${flipY*M_PI} 0 0" />
 				<geometry>
-					<mesh filename="package://husky_description/Media/models/wheel.stl" />
+					<mesh filename="package://husky_description/models/wheel.stl" />
 				</geometry>
 				<material name="DarkGray" />
@@ -68,5 +68,5 @@
 				    <cylinder length="${wheel_z_size}" radius="${wheel_x_size/2}" />
 				<!--
-					<mesh filename="package://husky_description/Media/models/wheel.stl" />
+					<mesh filename="package://husky_description/models/wheel.stl" />
 			    -->
 				</geometry>

Commit message: renamed /models folder to /meshes to follow the convention of other gazebo simulation packages. Changed the base.urdf.xacro to use base_footprint as the parent frame. For some reason, the new Gazebo paints all parts the same color as base_link if I use base_link as the parent.

File: urdf/base.urdf.xacro (robot description, xacro)
@@ -1,29 +1,3 @@
 <?xml version="1.0"?>
-<!--
-Copyright (c) 2012, Ryan Gariepy/Clearpath Robotics
-All rights reserved.
-Redistribution and use in source and binary forms, with or without
-modification, are permitted provided that the following conditions are met:
-    * Redistributions of source code must retain the above copyright
-      notice, this list of conditions and the following disclaimer.
-    * Redistributions in binary form must reproduce the above copyright
-      notice, this list of conditions and the following disclaimer in the
-      documentation and/or other materials provided with the distribution.
-    * Neither the name of Clearpath Robotics nor the
-      names of its contributors may be used to endorse or promote products
-      derived from this software without specific prior written permission.
-THIS SOFTWARE IS PROVIDED BY THE COPYRIGHT HOLDERS AND CONTRIBUTORS "AS IS" AND
-ANY EXPRESS OR IMPLIED WARRANTIES, INCLUDING, BUT NOT LIMITED TO, THE IMPLIED
-WARRANTIES OF MERCHANTABILITY AND FITNESS FOR A PARTICULAR PURPOSE ARE
-DISCLAIMED. IN NO EVENT SHALL THE COPYRIGHT HOLDERS BE LIABLE FOR ANY
-DIRECT, INDIRECT, INCIDENTAL, SPECIAL, EXEMPLARY, OR CONSEQUENTIAL DAMAGES
-(INCLUDING, BUT NOT LIMITED TO, PROCUREMENT OF SUBSTITUTE GOODS OR SERVICES;
-LOSS OF USE, DATA, OR PROFITS; OR BUSINESS INTERRUPTION) HOWEVER CAUSED AND
-ON ANY THEORY OF LIABILITY, WHETHER IN CONTRACT, STRICT LIABILITY, OR TORT
-(INCLUDING NEGLIGENCE OR OTHERWISE) ARISING IN ANY WAY OUT OF THE USE OF THIS
-SOFTWARE, EVEN IF ADVISED OF THE POSSIBILITY OF SUCH DAMAGE.
-This program contains the description of the robot base model for the Clearpath
-Husky A200
--->
 <robot
 	xmlns:xi="http://www.w3.org/2001/XInclude"
@@ -83,9 +57,8 @@
     </link>
     <gazebo reference="base_footprint">
-        <material>Gazebo/Green</material>
         <turnGravityOff>false</turnGravityOff>
     </gazebo>
     <joint name="base_footprint_joint" type="fixed">
-		<origin xyz="0 0 ${wheel_x_size/2 - base_z_origin_to_wheel_origin - base_z_origin_offset - base_z_origin_offset}" rpy="0 0 0" />
+		<origin xyz="0 0 ${wheel_x_size/2 - base_z_origin_to_wheel_origin}" rpy="0 0 0" />
         <parent link="base_footprint"/>
         <child link="base_link" />
@@ -103,7 +76,7 @@
         </inertial>
         <visual>
-            <origin xyz="0 0 ${base_z_origin_offset}" rpy="0 0 0" />
+            <origin xyz="0 0 0" rpy="0 0 0" />
             <geometry>
-                <mesh filename="package://husky_description/models/base_link.stl" />
+                <mesh filename="package://husky_description/meshes/base_link.stl" />
             </geometry>
             <material name="Black" />
@@ -127,46 +100,46 @@
     <!-- DECORATIONS -->
     <!-- Top Plate -->
-    <husky_part parent="base_link" name="top_plate" mesh="top_plate"
+    <husky_part parent="base_footprint" name="top_plate" mesh="top_plate"
           colour="Yellow"
-          translateX="0.0" translateY="0.0" translateZ="0.005"
+          translateX="0.0" translateY="0.0" translateZ="${wheel_x_size/2 - base_z_origin_to_wheel_origin}"
           rotateX="0.0" rotateY="0.0" rotateZ="0.0"/>
-    <gazebo reference="base_link_top_plate_part">
+    <gazebo reference="base_footprint_top_plate_part">
         <material>Gazebo/Yellow</material>
     </gazebo>
     <!-- User Rail -->
-    <husky_part parent="base_link" name="user_rail" mesh="user_rail"
+    <husky_part parent="base_footprint" name="user_rail" mesh="user_rail"
           colour="DarkGray"
-          translateX="0.272" translateY="0.0" translateZ="0.245"
+          translateX="0.272" translateY="0.0" translateZ="${0.245 + wheel_x_size/2 - base_z_origin_to_wheel_origin}"
           rotateX="0.0" rotateY="0.0" rotateZ="0.0"/>
-    <gazebo reference="base_link_user_rail_part">
+    <gazebo reference="base_footprint_user_rail_part">
         <material>Gazebo/Grey</material>
     </gazebo>
     <!-- Bumpers -->
-    <husky_part parent="base_link" name="front_bumper" mesh="bumper"
+    <husky_part parent="base_footprint" name="front_bumper" mesh="bumper"
           colour="DarkGray"
-          translateX="0.490" translateY="0.0" translateZ="0.091"
+          translateX="0.490" translateY="0.0" translateZ="${0.091 + wheel_x_size/2 - base_z_origin_to_wheel_origin}"
           rotateX="0.0" rotateY="0.0" rotateZ="0.0"/>
-    <gazebo reference="base_link_front_bumper_part">
+    <gazebo reference="base_footprint_front_bumper_part">
         <material>Gazebo/FlatBlack</material>
     </gazebo>
-    <husky_part parent="base_link" name="rear_bumper" mesh="bumper"
+    <husky_part parent="base_footprint" name="rear_bumper" mesh="bumper"
           colour="DarkGray"
-          translateX="-0.48" translateY="0.0" translateZ="0.091"
+          translateX="-0.48" translateY="0.0" translateZ="${0.091 + wheel_x_size/2 - base_z_origin_to_wheel_origin}"
           rotateX="0.0" rotateY="0.0" rotateZ="3.14"/>
-    <gazebo reference="base_link_rear_bumper_part">
+    <gazebo reference="base_footprint_rear_bumper_part">
         <material>Gazebo/FlatBlack</material>
     </gazebo>
     <gazebo>
-		<controller:husky_plugin name="husky_diff_controller" plugin="libhusky_gazebo_plugins.so">
-		        <alwaysOn>true</alwaysOn>
-		        <updateRate>100.0</updateRate>
-		        <backLeftJoint>joint_back_left_wheel</backLeftJoint>
-		        <backRightJoint>joint_back_right_wheel</backRightJoint>
-		        <frontLeftJoint>joint_front_left_wheel</frontLeftJoint>
-		        <frontRightJoint>joint_front_right_wheel</frontRightJoint>
-		        <wheelSeparation>${base_y_size}</wheelSeparation>
-		        <wheelDiameter>${wheel_x_size}</wheelDiameter>
-		        <torque>35</torque>
-        </controller:husky_plugin>
-	</gazebo>
+	    <plugin name="husky_diff_controller" filename="libhusky_gazebo_plugins.so">
+		    <alwaysOn>true</alwaysOn>
+            <updateRate>100.0</updateRate>
+            <backLeftJoint>joint_back_left_wheel</backLeftJoint>
+            <backRightJoint>joint_back_right_wheel</backRightJoint>
+            <frontLeftJoint>joint_front_left_wheel</frontLeftJoint>
+            <frontRightJoint>joint_front_right_wheel</frontRightJoint>
+            <wheelSeparation>${base_y_size}</wheelSeparation>
+            <wheelDiameter>${wheel_x_size}</wheelDiameter>
+            <torque>35</torque>
+        </plugin>
+    </gazebo>
 </robot>

File: urdf/parts.urdf.xacro (robot description, xacro)
@@ -46,10 +46,4 @@
 	<property name="izz_com_cs" value="0.01" /> <!-- at center of mass aligned with coordinate system, kg*m^2-->
 	<xacro:macro name="husky_part" params="parent name mesh colour translateX translateY translateZ rotateX rotateY rotateZ">
-		<joint name="${parent}_${name}_joint" type="fixed">
-		    <origin xyz="${translateX} ${translateY} ${translateZ}"
-		            rpy="${rotateX} ${rotateY} ${rotateZ}" />
-		    <parent link="${parent}" />
-		    <child link="${parent}_${name}_part" />
-		</joint>
 		<link name="${parent}_${name}_part">
 			<inertial>
@@ -62,5 +56,5 @@
 				<origin xyz="0 0 0" rpy="0 0 0" />
 				<geometry>
-					<mesh filename="package://husky_description/models/${mesh}.stl" />
+					<mesh filename="package://husky_description/meshes/${mesh}.stl" />
 				</geometry>
 				<material name="${colour}" />
@@ -73,4 +67,10 @@
 			</collision>
 		</link>
+		<joint name="${parent}_${name}_joint" type="fixed">
+		    <origin xyz="${translateX} ${translateY} ${translateZ}"
+		            rpy="${rotateX} ${rotateY} ${rotateZ}" />
+		    <parent link="${parent}" />
+		    <child link="${parent}_${name}_part" />
+		</joint>
   	</xacro:macro>
 </robot>

File: urdf/wheel.urdf.xacro (robot description, xacro)
@@ -47,5 +47,4 @@
 	<property name="base_y_origin_to_wheel_origin" value="0.285475" />
 	<property name="base_z_origin_to_wheel_origin" value="0.03282508" />
-	<property name="base_z_origin_offset" value="0.00317500" /> <!-- origin is offset in + z direction by 3.175mm, so need to bring it back down for visual and collision-->
 	<xacro:macro name="husky_wheel" params="fb lr parent translateX translateY flipY"> <!--fb : front, back ; lr: left, right -->
 		<link name="${fb}_${lr}_wheel">
@@ -59,5 +58,5 @@
 				<origin xyz="0 0 0" rpy="${flipY*M_PI} 0 0" />
 				<geometry>
-					<mesh filename="package://husky_description/models/wheel.stl" />
+					<mesh filename="package://husky_description/meshes/wheel.stl" />
 				</geometry>
 				<material name="DarkGray" />
@@ -67,7 +66,4 @@
 				<geometry>
 				    <cylinder length="${wheel_z_size}" radius="${wheel_x_size/2}" />
-				<!--
-					<mesh filename="package://husky_description/models/wheel.stl" />
-			    -->
 				</geometry>
 			</collision>
@@ -76,5 +72,5 @@
 			<mu1 value="1.0"/>
 			<mu2 value="1.0"/>
-			<kp  value="100000.0" />
+			<kp  value="10000000.0" />
 			<kd  value="1.0" />
 			<fdir1 value="1 0 0"/>
