Commit message: adding lidar viewing

File: urdf/base.sensors.urdf.xacro (robot description, xacro)
@@ -173,8 +173,8 @@
           </inertial>
             <visual>
-                <origin xyz="0 0 0" rpy="0 0 0"/>
+                <origin xyz="0 0 0.1" rpy="1.5705 0 -1.5705"/>
                 <geometry>
-                    <box size="0.05 0.05 0.1" />
-                    <!--mesh filename="package://husky_description/meshes/sick_lidar.stl" /-->
+                    <!--box size="0.05 0.05 0.1" /-->
+                    <mesh filename="package://husky_description/meshes/lidar.stl" />
                 </geometry>
             </visual>
@@ -182,6 +182,6 @@
                 <origin xyz="0 0 0" rpy="0 0 0"/>
                 <geometry>
-                  <box size="0.05 0.05 0.1" />
-                  <!--mesh filename="package://husky_description/meshes/sick_lidar.stl" /-->
+                  <!--box size="0.05 0.05 0.1" /-->
+                  <mesh filename="package://husky_description/meshes/lidar.stl" />
                 </geometry>
             </collision>

Commit message: adding basic gps and formalizing gps sick laser models, adding user plate

File: urdf/base.sensors.urdf.xacro (robot description, xacro)
@@ -115,4 +115,11 @@
         <material>Gazebo/Grey</material>
     </gazebo>
+    <husky_part parent="base_footprint" name="user_plate" mesh="user_plate"
+          colour="DarkGray"
+          translateX="-0.35" translateY="-0.325" translateZ="${0.165 + wheel_x_size/2 - base_z_origin_to_wheel_origin}"
+          rotateX="1.5705" rotateY="0.0" rotateZ="1.5705"/>
+    <gazebo reference="base_footprint_user_plate_part">
+        <material>Gazebo/FlatBlack</material>
+    </gazebo>
     <!-- Bumpers -->
     <husky_part parent="base_footprint" name="front_bumper" mesh="bumper"
@@ -152,38 +159,9 @@
       </plugin>
     </gazebo>
+    <xacro:include filename="$(find husky_description)/urdf/sensors/gps.urdf.xacro" />
+    <novatel_gps_sensor name="gps" gps_topic="gps" velocity_topic="gps_vel" lat="48" lon="-8.0" />
     <!-- This adds the laser macro, including the scan for gazebo and link name -->
-    <include filename="$(find husky_description)/urdf/sensors/sick_laser.urdf.xacro" />
-    <xacro:sick_laser_v0 name="laser_scan" parent="base" ros_topic="scan"
-        update_rate="20" min_angle="-1.57" max_angle="1.57" >
-            <origin xyz="${0.4 - 0.01 - 0.04} 0 0.3" rpy="0 0 0" />
-        </xacro:sick_laser_v0>
-        <!-- This adds a visual box to allow us to see the Hokuyo in rviz/gazebo -->
-        <joint name="laser_scan_joint" type="fixed">
-          <origin xyz="${0.4 - 0.01 - 0.04} 0 0.3" rpy="0 0 0" />
-          <parent link="base_link" />
-          <child link="laser_scan_link"/>
-        </joint>
-       <link name="laser_scan_link">
-          <inertial>
-            <mass value="0.01" />
-            <origin xyz="0 0 0" />
-            <inertia ixx="0.001"  ixy="0.0"  ixz="0.0"
-            iyy="0.001"  iyz="0.0"
-                izz="0.001" />
-          </inertial>
-            <visual>
-                <origin xyz="0 0 0.1" rpy="1.5705 0 -1.5705"/>
-                <geometry>
-                    <!--box size="0.05 0.05 0.1" /-->
-                    <mesh filename="package://husky_description/meshes/lidar.stl" />
-                </geometry>
-            </visual>
-            <collision>
-                <origin xyz="0 0 0" rpy="0 0 0"/>
-                <geometry>
-                  <!--box size="0.05 0.05 0.1" /-->
-                  <mesh filename="package://husky_description/meshes/lidar.stl" />
-                </geometry>
-            </collision>
-        </link>
+    <xacro:include filename="$(find husky_description)/urdf/sensors/sick_laser.urdf.xacro" />
+    <sick_laser_v0 name="laser_scan" parent="base" ros_topic="scan"
+        update_rate="20" min_angle="-1.57" max_angle="1.57" />
 </robot>

File: urdf/sensors/sick_laser.urdf.xacro (robot description, xacro)
@@ -5,31 +5,32 @@
        xmlns:xacro="http://ros.org/wiki/xacro">
        <xacro:include filename="$(find husky_description)/urdf/sensors/sick_laser.gazebo.xacro" />
-  <xacro:macro name="sick_laser_v0" params="name parent *origin ros_topic update_rate min_angle max_angle">
-    <!--joint name="${name}_joint" type="fixed">
-      <axis xyz="0 1 0" />
-      <insert_block name="origin" />
-      <parent link="${parent}_link"/>
-      <child link="${name}_link"/>
-    </joint-->
-    <!--link name="${name}_link" type="laser">
-        <visual>
-            <origin xyz="0 0 0" rpy="0 0 0"/>
-            <geometry>
-              <box size="0.05 0.05 0.1" />
-              <mesh filename="package://husky_description/meshes/sick_lidar.stl" />
-            </geometry>
-          </visual>
-        <collision>
-            <origin xyz="0 0 0" rpy="0 0 0"/>
-            <geometry>
-              <box size="0.05 0.05 0.1" />
-            </geometry>
-          </collision>
-      <inertial>
-        <mass value="0.001" />
-        <origin xyz="0 0 0" rpy="0 0 0" />
-        <inertia ixx="0.0001" ixy="0" ixz="0" iyy="0.000001" iyz="0" izz="0.0001" />
-      </inertial>
-    </link-->
+  <xacro:macro name="sick_laser_v0" params="name parent ros_topic update_rate min_angle max_angle">
+        <!-- This adds a visual box to allow us to see the Hokuyo in rviz/gazebo -->
+        <joint name="laser_scan_joint" type="fixed">
+          <origin xyz="0.43 0 0.2" rpy="0 0 0" />
+          <parent link="base_link" />
+          <child link="laser_scan_link"/>
+        </joint>
+       <link name="laser_scan_link">
+          <inertial>
+            <mass value="0.01" />
+            <origin xyz="0 0 0" />
+            <inertia ixx="0.001"  ixy="0.0"  ixz="0.0"
+            iyy="0.001"  iyz="0.0"
+                izz="0.001" />
+          </inertial>
+            <visual>
+                <origin xyz="0 0 0.1" rpy="1.5705 0 -1.5705"/>
+                <geometry>
+                    <mesh filename="package://husky_description/meshes/lidar.stl" />
+                </geometry>
+            </visual>
+            <collision>
+                <origin xyz="0 0 0" rpy="0 0 0"/>
+                <geometry>
+                  <mesh filename="package://husky_description/meshes/lidar.stl" />
+                </geometry>
+            </collision>
+        </link>
     <!-- gazebo extensions -->
     <xacro:sick_laser_gazebo_v0 name="${name}" ros_topic="${ros_topic}" update_rate="${update_rate}" min_angle="${min_angle}" max_angle="${max_angle}" />

Commit message: gps was setup incorrectly. re-jigged to fix it. xacro files needs to be modularized

File: urdf/base.sensors.urdf.xacro (robot description, xacro)
@@ -159,6 +159,21 @@
       </plugin>
     </gazebo>
-    <xacro:include filename="$(find husky_description)/urdf/sensors/gps.urdf.xacro" />
-    <novatel_gps_sensor name="gps" gps_topic="gps" velocity_topic="gps_vel" lat="48" lon="-8.0" />
+    <gazebo>
+       <plugin name="gps_plugin" filename="libhusky_tudarmstadt_gps_plugin.so">
+	    <alwaysOn>true</alwaysOn>
+            <updateRate>4.0</updateRate>
+            <bodyName>base_link</bodyName>
+            <topicName>fix</topicName>
+            <velocityTopicName>fix_velocity</velocityTopicName>
+            <drift>5.0 5.0 5.0</drift>
+            <gaussianNoise>0.1 0.1 0.1</gaussianNoise>
+            <velocityDrift>0 0 0</velocityDrift>
+            <velocityGaussianNoise>0.1 0.1 0.1</velocityGaussianNoise>
+	    <referenceLatitude>43.0</referenceLatitude>
+	    <referenceLongitude>-80.0</referenceLongitude>
+	</plugin>
+    </gazebo>
+    <!--xacro:include filename="$(find husky_description)/urdf/sensors/gps.urdf.xacro" />
+    <novatel_gps_sensor name="gps" gps_topic="gps" velocity_topic="gps_vel" lat="48" lon="-8.0" / -->
     <!-- This adds the laser macro, including the scan for gazebo and link name -->
     <xacro:include filename="$(find husky_description)/urdf/sensors/sick_laser.urdf.xacro" />

File: urdf/sensors/gps.urdf.xacro (robot description, xacro)
@@ -32,7 +32,6 @@
             </collision>
         </link>
-   <xacro:macro name="gps_sensor" params="name gps_topic velocity_topic lat lon">
-    <gazebo reference="${name}_link">
-       <plugin name="gps_plugin" filename="libhusky_tudarmstadt_gps_plugin.so">
+    <gazebo>
+       <controller:husky_gps_plugin name="gps_plugin" filename="libhusky_tudarmstadt_gps_plugin.so">
 	<frameId>${name}_link</frameId>
 	<topicName>${gps_topic}</topicName>
@@ -40,7 +39,6 @@
 	<referenceLatitude>${lat}</referenceLatitude>
 	<referenceLongitude>${lon}</referenceLongitude>
-      </plugin>
+      </controller:husky_gps_plugin>
     </gazebo>
   </xacro:macro>
-  </xacro:macro>
 </robot>
