Commit message: working gps sensor, re-jigged to resuse base.xacro design

File: urdf/base.sensors.urdf.xacro (robot description, xacro)
@@ -1,182 +1,45 @@
 <?xml version="1.0"?>
 <robot
-	xmlns:xi="http://www.w3.org/2001/XInclude"
-	xmlns:gazebo="http://playerstage.sourceforge.net/gazebo/xmlschema/#gz"
-    xmlns:model="http://playerstage.sourceforge.net/gazebo/xmlschema/#model"
-	xmlns:sensor="http://playerstage.sourceforge.net/gazebo/xmlschema/#sensor"
-	xmlns:body="http://playerstage.sourceforge.net/gazebo/xmlschema/#body"
-    xmlns:geom="http://playerstage.sourceforge.net/gazebo/xmlschema/#geom"
-    xmlns:joint="http://playerstage.sourceforge.net/gazebo/xmlschema/#joint"
-	xmlns:controller="http://playerstage.sourceforge.net/gazebo/xmlschema/#controller"
-	xmlns:interface="http://playerstage.sourceforge.net/gazebo/xmlschema/#interface"
-	xmlns:rendering="http://playerstage.sourceforge.net/gazebo/xmlschema/#rendering"
-    xmlns:renderable="http://playerstage.sourceforge.net/gazebo/xmlschema/#renderable"
-    xmlns:physics="http://playerstage.sourceforge.net/gazebo/xmlschema/#physics"
+  xmlns:gazebo="http://playerstage.sourceforge.net/gazebo/xmlschema/#gz"
+  xmlns:plugin="http://playerstage.sourceforge.net/gazebo/xmlschema/#plugin"
 	xmlns:xacro="http://ros.org/wiki/xacro" name="husky">
-	<!-- Included URDF/XACRO Files -->
-    <xacro:include filename="$(find husky_description)/urdf/materials.urdf.xacro" />
-    <xacro:include filename="$(find husky_description)/urdf/wheel.urdf.xacro" />
-    <xacro:include filename="$(find husky_description)/urdf/parts.urdf.xacro" />
-	<!-- PROPERTY LIST -->
-    <!--All units in m-kg-s-radians unit system -->
-    <property name="M_PI" value="3.1415926535897931" />
-    <!-- Main Body-base-->
-    <!-- Location of com : center of mass -->
-    <property name="base_x_com" value="-0.08748000" />
-    <property name="base_y_com" value="-0.00085000" />
-    <property name="base_z_com" value="0.09947000" />
-    <!-- Size of the base-->
-    <property name="base_x_size" value="0.98740000" />
-    <property name="base_y_size" value="0.57090000" />
-    <property name="base_z_size" value="0.24750000" />
-    <!--Weight of the base-->
-    <property name="base_mass" value="33.45489000" /> <!-- in kg-->
-    <!--Inertial values for the base at center of mass, aligned with coordinate system. Units are kg*m^2-->
-    <property name="base_ixx_com_cs" value="0.60216370" />
-    <property name="base_ixy_com_cs" value="-0.02364198" />
-    <property name="base_ixz_com_cs" value="-0.11972132" />
-    <property name="base_iyy_com_cs" value="1.73859574" />
-    <property name="base_iyz_com_cs" value="-0.00154437" />
-    <property name="base_izz_com_cs" value="2.02955229" />
-<!-- BASE-FOOTPRINT -->
-    <!-- base_footprint is a fictitious link(frame) that is on the ground right below base_link origin, navigation stack depends on this frame -->
-    <link name="base_footprint">
-        <inertial>
-            <mass value="0.0001" />
-            <origin xyz="0 0 0" />
-            <inertia ixx="0.0001" ixy="0.0" ixz="0.0"
-                iyy="0.0001" iyz="0.0"
-                izz="0.0001" />
-        </inertial>
-        <visual>
-            <origin xyz="0 0 0" rpy="0 0 0" />
-            <geometry>
-                <box size="0.001 0.001 0.001" />
-            </geometry>
-        </visual>
-    </link>
-    <gazebo reference="base_footprint">
-        <turnGravityOff>false</turnGravityOff>
-    </gazebo>
-    <joint name="base_footprint_joint" type="fixed">
-		<origin xyz="0 0 ${wheel_x_size/2 - base_z_origin_to_wheel_origin}" rpy="0 0 0" />
-        <parent link="base_footprint"/>
-        <child link="base_link" />
-    </joint>
-    <!-- BASE-LINK -->
-    <!--Actual body/chassis of the robot-->
-    <link name="base_link">
-        <inertial>
-            <mass value="${base_mass}" />
-            <!--This is the pose of the inertial reference frame, relative to the link reference frame. The origin of the inertial reference frame needs to be at the center of gravity. The axes of the inertial reference frame do not need to be aligned with the principal axes of the inertia.-->
-            <origin xyz="${base_x_com} ${base_y_com} ${base_z_com}" />
-            <!--The 3x3 rotational inertia matrix. Because the rotational inertia matrix is symmetric, only 6 above-diagonal elements of this matrix are specified here, using the attributes ixx, ixy, ixz, iyy, iyz, izz.-->
-            <inertia ixx="${base_ixx_com_cs}" ixy="${base_ixy_com_cs}" ixz="${base_ixz_com_cs}"
-                iyy="${base_iyy_com_cs}" iyz="${base_iyz_com_cs}" izz="${base_izz_com_cs}" />
-        </inertial>
-        <visual>
-            <origin xyz="0 0 0" rpy="0 0 0" />
-            <geometry>
-                <mesh filename="package://husky_description/meshes/base_link.stl" />
-            </geometry>
-            <material name="Black" />
-        </visual>
-		<collision>
-			<origin xyz="0 0 ${wheel_x_size/2 - base_z_origin_to_wheel_origin - 0.02}" rpy="0 0 0 " />
-			<geometry>
-				<box size = "${base_x_size+0.02} ${base_y_size} ${base_z_size + 0.02}"/> <!--making it slightly bigger in x and z direction-->
-			</geometry>
-		</collision>
-    </link>
-    <gazebo reference="base_link">
-        <material>Gazebo/FlatBlack</material>
-        <turnGravityOff>false</turnGravityOff>
-    </gazebo>
-    <!-- WHEEL macros -->
-	<husky_wheel fb="back" lr="left" parent="base_link" translateX="-1" translateY="1" flipY="-1"/>
-	<husky_wheel fb="back" lr="right" parent="base_link" translateX="-1" translateY="-1" flipY="-1"/>
-	<husky_wheel fb="front" lr="left" parent="base_link" translateX="1" translateY="1" flipY="-1"/>
-	<husky_wheel fb="front" lr="right" parent="base_link" translateX="1" translateY="-1" flipY="-1"/>
-    <!-- DECORATIONS -->
-    <!-- Top Plate -->
-    <husky_part parent="base_footprint" name="top_plate" mesh="top_plate"
-          colour="Yellow"
-          translateX="0.0" translateY="0.0" translateZ="${wheel_x_size/2 - base_z_origin_to_wheel_origin}"
-          rotateX="0.0" rotateY="0.0" rotateZ="0.0"/>
-    <gazebo reference="base_footprint_top_plate_part">
-        <material>Gazebo/Yellow</material>
-    </gazebo>
-    <!-- User Rail -->
-    <husky_part parent="base_footprint" name="user_rail" mesh="user_rail"
-          colour="DarkGray"
-          translateX="0.272" translateY="0.0" translateZ="${0.245 + wheel_x_size/2 - base_z_origin_to_wheel_origin}"
-          rotateX="0.0" rotateY="0.0" rotateZ="0.0"/>
-    <gazebo reference="base_footprint_user_rail_part">
-        <material>Gazebo/Grey</material>
-    </gazebo>
-    <husky_part parent="base_footprint" name="user_plate" mesh="user_plate"
-          colour="DarkGray"
-          translateX="-0.35" translateY="-0.325" translateZ="${0.165 + wheel_x_size/2 - base_z_origin_to_wheel_origin}"
-          rotateX="1.5705" rotateY="0.0" rotateZ="1.5705"/>
-    <gazebo reference="base_footprint_user_plate_part">
-        <material>Gazebo/FlatBlack</material>
-    </gazebo>
-    <!-- Bumpers -->
-    <husky_part parent="base_footprint" name="front_bumper" mesh="bumper"
-          colour="DarkGray"
-          translateX="0.490" translateY="0.0" translateZ="${0.091 + wheel_x_size/2 - base_z_origin_to_wheel_origin}"
-          rotateX="0.0" rotateY="0.0" rotateZ="0.0"/>
-    <gazebo reference="base_footprint_front_bumper_part">
-        <material>Gazebo/FlatBlack</material>
-    </gazebo>
-    <husky_part parent="base_footprint" name="rear_bumper" mesh="bumper"
-          colour="DarkGray"
-          translateX="-0.48" translateY="0.0" translateZ="${0.091 + wheel_x_size/2 - base_z_origin_to_wheel_origin}"
-          rotateX="0.0" rotateY="0.0" rotateZ="3.14"/>
-    <gazebo reference="base_footprint_rear_bumper_part">
-        <material>Gazebo/FlatBlack</material>
-    </gazebo>
-    <gazebo>
-	    <plugin name="husky_diff_controller" filename="libhusky_gazebo_plugins.so">
-		    <alwaysOn>true</alwaysOn>
-            <updateRate>100.0</updateRate>
-            <backLeftJoint>joint_back_left_wheel</backLeftJoint>
-            <backRightJoint>joint_back_right_wheel</backRightJoint>
-            <frontLeftJoint>joint_front_left_wheel</frontLeftJoint>
-            <frontRightJoint>joint_front_right_wheel</frontRightJoint>
-            <wheelSeparation>${base_y_size}</wheelSeparation>
-            <wheelDiameter>${wheel_x_size}</wheelDiameter>
-            <torque>35</torque>
-        </plugin>
-      </gazebo>
-    <gazebo>
-      <plugin name="imu_plugin" filename="libgazebo_ros_imu.so">
-        <alwaysOn>true</alwaysOn>
+    <!-- Included URDF/XACRO Files -->
+  <xacro:include filename="$(find husky_description)/urdf/base.urdf.xacro" />
+  <xacro:include filename="$(find husky_description)/urdf/sensors/sick_laser.urdf.xacro" />
+  <xacro:include filename="$(find husky_description)/urdf/sensors/gps.urdf.xacro" />
+  <gazebo>
+    <plugin name="imu_plugin" filename="libgazebo_ros_imu.so">
+      <alwaysOn>true</alwaysOn>
+      <bodyName>base_link</bodyName>
+      <topicName>imu_data</topicName>
+      <serviceName>imu_service</serviceName>
+      <gaussianNoise>0.01</gaussianNoise>
+    </plugin>
+  </gazebo>
+  <husky_part parent="base_footprint" name="user_plate" mesh="user_plate"
+    colour="DarkGray"
+    translateX="-0.35" translateY="-0.325" translateZ="${0.165 + wheel_x_size/2 - base_z_origin_to_wheel_origin}"
+    rotateX="1.5705" rotateY="0.0" rotateZ="1.5705"/>
+  <gazebo reference="base_footprint_user_plate_part">
+    <material>Gazebo/FlatBlack</material>
+  </gazebo>
+  <gazebo>
+    <plugin name="gps_plugin" filename="libhusky_tudarmstadt_gps_plugin.so">
+    <alwaysOn>true</alwaysOn>
+        <updateRate>4.0</updateRate>
         <bodyName>base_link</bodyName>
-        <topicName>imu_data</topicName>
-        <serviceName>imu_service</serviceName>
-        <gaussianNoise>0.01</gaussianNoise>
-      </plugin>
-    </gazebo>
-    <gazebo>
-       <plugin name="gps_plugin" filename="libhusky_tudarmstadt_gps_plugin.so">
-	    <alwaysOn>true</alwaysOn>
-            <updateRate>4.0</updateRate>
-            <bodyName>base_link</bodyName>
-            <topicName>fix</topicName>
-            <velocityTopicName>fix_velocity</velocityTopicName>
-            <drift>5.0 5.0 5.0</drift>
-            <gaussianNoise>0.1 0.1 0.1</gaussianNoise>
-            <velocityDrift>0 0 0</velocityDrift>
-            <velocityGaussianNoise>0.1 0.1 0.1</velocityGaussianNoise>
-	    <referenceLatitude>43.0</referenceLatitude>
-	    <referenceLongitude>-80.0</referenceLongitude>
-	</plugin>
-    </gazebo>
-    <!--xacro:include filename="$(find husky_description)/urdf/sensors/gps.urdf.xacro" />
-    <novatel_gps_sensor name="gps" gps_topic="gps" velocity_topic="gps_vel" lat="48" lon="-8.0" / -->
-    <!-- This adds the laser macro, including the scan for gazebo and link name -->
-    <xacro:include filename="$(find husky_description)/urdf/sensors/sick_laser.urdf.xacro" />
-    <sick_laser_v0 name="laser_scan" parent="base" ros_topic="scan"
-        update_rate="20" min_angle="-1.57" max_angle="1.57" />
+        <topicName>fix</topicName>
+        <velocityTopicName>fix_velocity</velocityTopicName>
+        <drift>5.0 5.0 5.0</drift>
+        <gaussianNoise>0.1 0.1 0.1</gaussianNoise>
+        <velocityDrift>0 0 0</velocityDrift>
+        <velocityGaussianNoise>0.1 0.1 0.1</velocityGaussianNoise>
+        <referenceLatitude>37.0003</referenceLatitude>
+        <referenceLongitude>-76.4107</referenceLongitude>
+    </plugin>
+  </gazebo>
+  <!--novatel_gps_sensor name="gps" gps_topic="gps" velocity_topic="gps_vel" lat="48" lon="-8.0" /-->
+  <!-- This adds the laser macro, including the scan for gazebo and link name -->
+  <sick_laser_v0 name="laser_scan" parent="base" ros_topic="scan"
+    update_rate="20" min_angle="-1.57" max_angle="1.57" />
 </robot>

File: urdf/sensors/gps.urdf.xacro (robot description, xacro)
@@ -3,42 +3,34 @@
        xmlns:controller="http://playerstage.sourceforge.net/gazebo/xmlschema/#controller"
        xmlns:interface="http://playerstage.sourceforge.net/gazebo/xmlschema/#interface"
+      xmlns:plugin="http://playerstage.sourceforge.net/gazebo/xmlschema/#plugin"
        xmlns:xacro="http://ros.org/wiki/xacro">
   <xacro:macro name="novatel_gps_sensor" params="name gps_topic velocity_topic lat lon">
-        <!-- This adds a visual box to allow us to see the GPS in rviz/gazebo -->
-        <joint name="gps_joint" type="fixed">
-          <origin xyz="0.39 0.385 0.10" rpy="-1.5705 -1.5705 0" />
-          <parent link="base_footprint_user_plate_part" />
-          <child link="gps_link"/>
-        </joint>
-       <link name="gps_link">
-          <inertial>
-            <mass value="0.01" />
-            <origin xyz="0 0 0" />
-            <inertia ixx="0.001"  ixy="0.0"  ixz="0.0"
-            iyy="0.001"  iyz="0.0"
-                izz="0.001" />
-          </inertial>
-            <visual>
-                <origin xyz="0 0 0.1" rpy="1.5705 0 -1.5705"/>
-                <geometry>
-                    <mesh filename="package://husky_description/meshes/gps.stl" />
-                </geometry>
-            </visual>
-            <collision>
-                <origin xyz="0 0 0" rpy="0 0 0"/>
-                <geometry>
-                  <mesh filename="package://husky_description/meshes/gps.stl" />
-                </geometry>
-            </collision>
-        </link>
-    <gazebo>
-       <controller:husky_gps_plugin name="gps_plugin" filename="libhusky_tudarmstadt_gps_plugin.so">
-	<frameId>${name}_link</frameId>
-	<topicName>${gps_topic}</topicName>
-	<velocityTopicName>${velocity_topic}</velocityTopicName>
-	<referenceLatitude>${lat}</referenceLatitude>
-	<referenceLongitude>${lon}</referenceLongitude>
-      </controller:husky_gps_plugin>
-    </gazebo>
+  <!-- This adds a visual box to allow us to see the GPS in rviz/gazebo -->
+    <joint name="gps_joint" type="fixed">
+      <origin xyz="0.39 0.385 0.10" rpy="-1.5705 -1.5705 0" />
+      <parent link="base_footprint_user_plate_part" />
+      <child link="gps_link"/>
+    </joint>
+    <link name="gps_link">
+      <inertial>
+        <mass value="0.01" />
+        <origin xyz="0 0 0" />
+        <inertia ixx="0.001"  ixy="0.0"  ixz="0.0"
+        iyy="0.001"  iyz="0.0"
+        izz="0.001" />
+      </inertial>
+      <visual>
+        <origin xyz="0 0 0.1" rpy="1.5705 0 -1.5705"/>
+        <geometry>
+        <mesh filename="package://husky_description/meshes/gps.stl" />
+        </geometry>
+      </visual>
+      <collision>
+        <origin xyz="0 0 0" rpy="0 0 0"/>
+        <geometry>
+        <mesh filename="package://husky_description/meshes/gps.stl" />
+        </geometry>
+      </collision>
+    </link>
   </xacro:macro>
 </robot>

Commit message: modifications to the laser plugin to standardize the laser link name and fix the LIDAR parameters for SICK

File: urdf/base.sensors.urdf.xacro (robot description, xacro)
@@ -41,5 +41,5 @@
   <!--novatel_gps_sensor name="gps" gps_topic="gps" velocity_topic="gps_vel" lat="48" lon="-8.0" /-->
   <!-- This adds the laser macro, including the scan for gazebo and link name -->
-  <sick_laser_v0 name="laser_scan" parent="base" ros_topic="scan"
+  <sick_laser_v0 name="laser" parent="base" ros_topic="scan"
     update_rate="20" min_angle="-1.57" max_angle="1.57" />
 </robot>

File: urdf/sensors/sick_laser.gazebo.xacro (robot description, xacro)
@@ -11,5 +11,5 @@
           <scan>
             <horizontal>
-              <samples>640</samples>
+              <samples>720</samples>
               <resolution>1</resolution>
               <min_angle>${min_angle}</min_angle>
@@ -19,5 +19,5 @@
           <range>
             <min>0.08</min>
-            <max>10.0</max>
+            <max>50.0</max>
             <resolution>0.01</resolution>
           </range>

File: urdf/sensors/sick_laser.urdf.xacro (robot description, xacro)
@@ -8,9 +8,9 @@
         <!-- This adds a visual box to allow us to see the Hokuyo in rviz/gazebo -->
         <joint name="laser_scan_joint" type="fixed">
-          <origin xyz="0.43 0 0.2" rpy="0 0 0" />
+          <origin xyz="0.3 0 0.4" rpy="0 0 0" />
           <parent link="base_link" />
-          <child link="laser_scan_link"/>
+          <child link="${name}_link"/>
         </joint>
-       <link name="laser_scan_link">
+       <link name="${name}_link">
           <inertial>
             <mass value="0.01" />
