Commit message: RP-272 Switch to NED orientation for UM6 standard package

File: urdf/husky.urdf.xacro (robot description, xacro)
@@ -80,5 +80,5 @@
     <link name="imu_link"/>
     <joint name="imu_joint" type="fixed">
-      <origin xyz="$(optenv HUSKY_IMU_XYZ 0.19 0 0.149)" rpy="$(optenv HUSKY_IMU_RPY 1.5708 0 -1.5708)" />
+      <origin xyz="$(optenv HUSKY_IMU_XYZ 0.19 0 0.149)" rpy="$(optenv HUSKY_IMU_RPY 0 -1.5708 3.1416)" />
       <parent link="chassis_link" />
       <child link="imu_link" />

Commit message: Updated kinect to have optenv

File: urdf/husky.urdf.xacro (robot description, xacro)
@@ -23,12 +23,13 @@
 <robot name="husky_robot" xmlns:xacro="http://ros.org/wiki/xacro">
   <!-- Included URDF/XACRO Files -->
-  <xacro:include filename="$(find husky_description)/urdf/materials.urdf" />
-  <xacro:include filename="$(find husky_description)/urdf/wheel.urdf.xacro" />
   <xacro:include filename="$(find husky_description)/urdf/decorations.urdf.xacro" />
   <xacro:include filename="$(find husky_description)/urdf/accessories/kinect_camera.urdf.xacro"/>
   <xacro:include filename="$(find husky_description)/urdf/accessories/sick_lms100.urdf.xacro"/>
   <xacro:include filename="$(find husky_description)/urdf/accessories/sensor_arch.urdf.xacro"/>
-  <xacro:include filename="$(find robotiq_c2_model_visualization)/urdf/robotiq_c2_model_macro.xacro"/>
+  <!-- <xacro:include filename="$(find robotiq_c2_model_visualization)/urdf/robotiq_c2_model_macro.xacro"/> -->
   <xacro:include filename="$(find ur_description)/urdf/ur5.urdf.xacro" />
+  <!-- Included URDF/XACRO Files -->
+  <xacro:include filename="$(find husky_description)/urdf/materials.urdf" />
+  <xacro:include filename="$(find husky_description)/urdf/wheel.urdf.xacro" />
   <property name="M_PI" value="3.14159"/>
   <!-- Base Size -->
@@ -108,5 +109,5 @@
     </xacro:husky_wheel>
     <xacro:husky_decorate />
-    <xacro:if value="$(arg gripper_enabled)">
+    <!-- <xacro:if value="$(arg gripper_enabled)">
 	    <xacro:robotiq_c2_model prefix=""/>
 	    <joint name="ur5_arm_ee_joint" type="fixed">
@@ -115,5 +116,5 @@
 	       <origin xyz="0 0 0" rpy="0 0 0"/>
 	    </joint>
-    </xacro:if>
+    </xacro:if> -->
     <xacro:if value="$(arg ur5_enabled)">
       <xacro:property name="reflect" value="-1" />
@@ -124,5 +125,5 @@
         <parent link="top_plate_link" />
         <child link="ur5_arm_base_link" />
-        <origin xyz="0.3058 0 0.0065" rpy="0.0 0.0 0.0" />
+        <origin xyz="0.3058 0 0.0065" rpy="0.0 0.0 -1.57" />
       </joint>
     </xacro:if>
@@ -140,5 +141,5 @@
         </xacro:sensor_arch>
         <joint name="kinect_frame_joint" type="fixed">
-          <origin xyz="0 0 0" rpy="0 ${M_PI/8} ${M_PI}"/>
+          <origin xyz="$(optenv HUSKY_KINECT_XYZ 0 0 0)" rpy="$(optenv HUSKY_KINECT_RPY 0 0.3925 3.14)" />
           <parent link="sensor_arch_mount_link"/>
           <child link="camera_link"/>
