Commit message: Cleanup and remove all gripper code

File: urdf/description.xacro (robot description, xacro)
@@ -25,5 +25,4 @@
   <xacro:arg name="ur5_enabled" default="false" />
   <xacro:arg name="kinect_enabled" default="false" />
-  <xacro:arg name="gripper_enabled" default="false" />
   <xacro:include filename="$(find husky_description)/urdf/husky.urdf.xacro" />
   <xacro:husky_robot />

File: urdf/husky.urdf.xacro (robot description, xacro)
@@ -109,12 +109,4 @@
     </xacro:husky_wheel>
     <xacro:husky_decorate />
-    <!-- <xacro:if value="$(arg gripper_enabled)">
-	    <xacro:robotiq_c2_model prefix=""/>
-	    <joint name="ur5_arm_ee_joint" type="fixed">
-	       <parent link="ur5_arm_ee_link"/>
-	       <child link="robotiq_85_adapter_link"/>
-	       <origin xyz="0 0 0" rpy="0 0 0"/>
-	    </joint>
-    </xacro:if> -->
     <xacro:if value="$(arg ur5_enabled)">
       <xacro:property name="reflect" value="-1" />
