Commit message: RP-264 Remove multirobot changes, experiment later

File: urdf/decorations.urdf.xacro (robot description, xacro)
@@ -3,5 +3,5 @@
 Software License Agreement (BSD)
 \file      decorations.urdf.xacro
-\authors   Paul Bovbel <pbovbel@clearpathrobotics.com
+\authors   Paul Bovbel <pbovbel@clearpathrobotics.com>
 \copyright Copyright (c) 2015, Clearpath Robotics, Inc., All rights reserved.
 Redistribution and use in source and binary forms, with or without modification, are permitted provided that
@@ -22,30 +22,6 @@
 -->
 <robot name="husky_decorations" xmlns:xacro="http://ros.org/wiki/xacro">
-  <material name="Black">
-    <color rgba="0.1 0.1 0.1 1.0"/>
-  </material>
-  <material name="Blue">
-    <color rgba="0.0 0.0 0.8 1.0"/>
-  </material>
-  <material name="Green">
-    <color rgba="0.0 0.8 0.0 1.0"/>
-  </material>
-  <material name="Grey">
-    <color rgba="0.7 0.7 0.7 1.0"/>
-  </material>
-  <material name="DarkGrey">
-    <color rgba="0.3 0.3 0.3 1.0"/>
-  </material>
-  <material name="Red">
-    <color rgba="0.8 0.0 0.0 1.0"/>
-  </material>
-  <material name="White">
-    <color rgba="1.0 1.0 1.0 1.0"/>
-  </material>
-  <material name="Yellow">
-    <color rgba="0.8 0.8 0.0 1.0"/>
-  </material>
-  <xacro:macro name="husky_decorate" params="prefix">
-    <link name="${prefix}top_plate_link">
+  <xacro:macro name="husky_decorate">
+    <link name="top_plate_link">
       <visual>
         <origin xyz="0 0 0" rpy="0 0 0" />
@@ -56,13 +32,13 @@
       </visual>
     </link>
-    <joint name="${prefix}top_plate" type="fixed">
-      <parent link="${prefix}chassis_link" />
-      <child link="${prefix}top_plate_link" />
+    <joint name="top_plate" type="fixed">
+      <parent link="chassis_link" />
+      <child link="top_plate_link" />
     </joint>
-    <gazebo reference="${prefix}top_plate_link">
+    <gazebo reference="top_plate_link">
       <material>Gazebo/Yellow</material>
       <turnGravityOff>false</turnGravityOff>
     </gazebo>
-    <link name="${prefix}user_rail_link">
+    <link name="user_rail_link">
       <visual>
         <geometry>
@@ -72,14 +48,14 @@
       </visual>
     </link>
-    <joint name="${prefix}user_rail" type="fixed">
+    <joint name="user_rail" type="fixed">
       <origin xyz="0.272 0 0.245" rpy="0 0 0" />
-      <parent link="${prefix}chassis_link" />
-      <child link="${prefix}user_rail_link" />
+      <parent link="chassis_link" />
+      <child link="user_rail_link" />
     </joint>
-    <gazebo reference="${prefix}user_rail_link">
+    <gazebo reference="user_rail_link">
       <material>Gazebo/DarkGrey</material>
       <turnGravityOff>false</turnGravityOff>
     </gazebo>
-    <link name="${prefix}front_bumper_link">
+    <link name="front_bumper_link">
       <visual>
         <geometry>
@@ -89,14 +65,14 @@
       </visual>
     </link>
-    <joint name="${prefix}front_bumper" type="fixed">
+    <joint name="front_bumper" type="fixed">
       <origin xyz="0.48 0 0.091" rpy="0 0 0" />
-      <parent link="${prefix}chassis_link" />
-      <child link="${prefix}front_bumper_link" />
+      <parent link="chassis_link" />
+      <child link="front_bumper_link" />
     </joint>
-    <gazebo reference="${prefix}front_bumper_link">
+    <gazebo reference="front_bumper_link">
       <material>Gazebo/DarkGrey</material>
       <turnGravityOff>false</turnGravityOff>
     </gazebo>
-    <link name="${prefix}rear_bumper_link">
+    <link name="rear_bumper_link">
       <visual>
         <geometry>
@@ -106,10 +82,10 @@
       </visual>
     </link>
-    <joint name="${prefix}rear_bumper" type="fixed">
+    <joint name="rear_bumper" type="fixed">
       <origin xyz="-0.48 0 0.091" rpy="0 0 ${M_PI}" />
-      <parent link="${prefix}chassis_link" />
-      <child link="${prefix}rear_bumper_link" />
+      <parent link="chassis_link" />
+      <child link="rear_bumper_link" />
     </joint>
-    <gazebo reference="${prefix}rear_bumper_link">
+    <gazebo reference="rear_bumper_link">
       <material>Gazebo/DarkGrey</material>
       <turnGravityOff>false</turnGravityOff>

File: urdf/husky.urdf.xacro (robot description, xacro)
@@ -3,5 +3,5 @@
 Software License Agreement (BSD)
 \file      husky.urdf.xacro
-\authors   Paul Bovbel <pbovbel@clearpathrobotics.com
+\authors   Paul Bovbel <pbovbel@clearpathrobotics.com>
 \copyright Copyright (c) 2015, Clearpath Robotics, Inc., All rights reserved.
 Redistribution and use in source and binary forms, with or without modification, are permitted provided that
@@ -23,4 +23,5 @@
 <robot name="husky_robot" xmlns:xacro="http://ros.org/wiki/xacro">
   <!-- Included URDF/XACRO Files -->
+  <xacro:include filename="$(find husky_description)/urdf/materials.urdf" />
   <xacro:include filename="$(find husky_description)/urdf/wheel.urdf.xacro" />
   <xacro:include filename="$(find husky_description)/urdf/decorations.urdf.xacro" />
@@ -37,18 +38,18 @@
   <xacro:property name="wheel_length" value="0.1143" />
   <xacro:property name="wheel_radius" value="0.17775" />
-  <xacro:macro name="husky_robot" params="prefix">
+  <xacro:macro name="husky_robot">
     <!-- Base link is on the ground under the robot -->
-    <link name="${prefix}base_link"/>
-    <gazebo reference="${prefix}base_link">
+    <link name="base_link"/>
+    <gazebo reference="base_link">
       <material>Gazebo/DarkGrey</material>
       <turnGravityOff>false</turnGravityOff>
     </gazebo>
-    <joint name="${prefix}chassis_joint" type="fixed">
+    <joint name="chassis_joint" type="fixed">
       <origin xyz="0 0 ${wheel_radius - wheel_vertical_offset}" rpy="0 0 0" />
-      <parent link="${prefix}base_link" />
-      <child link="${prefix}chassis_link" />
+      <parent link="base_link" />
+      <child link="chassis_link" />
     </joint>
     <!-- Chassis link is the center of the robot's bottom plate -->
-    <link name="${prefix}chassis_link">
+    <link name="chassis_link">
       <visual>
         <origin xyz="0 0 0" rpy="0 0 0" />
@@ -72,31 +73,32 @@
        </inertial>
      </link>
-     <gazebo reference="${prefix}chassis_link">
+     <gazebo reference="chassis_link">
       <turnGravityOff>false</turnGravityOff>
     </gazebo>
     <!-- IMU Link is the standard mounting position for the UM6 IMU.-->
     <!-- Can be modified with environment variables in /etc/ros/setup.bash -->
-    <link name="${prefix}imu_link"/>
-    <joint name="${prefix}imu_joint" type="fixed">
+    <link name="imu_link"/>
+    <joint name="imu_joint" type="fixed">
       <origin xyz="$(optenv HUSKY_IMU_XYZ 0.19 0 0.149)" rpy="$(optenv HUSKY_IMU_RPY 1.5708 0 -1.5708)" />
-      <parent link="${prefix}chassis_link" />
-      <child link="${prefix}imu_link" />
+      <parent link="chassis_link" />
+      <child link="imu_link" />
     </joint>
-    <gazebo reference="${prefix}imu_link">
+    <gazebo reference="imu_link">
       <turnGravityOff>false</turnGravityOff>
     </gazebo>
-    <xacro:husky_wheel prefix="${prefix}" wheel_prefix="front_left">
+    <!-- Husky wheel macros -->
+    <xacro:husky_wheel wheel_prefix="front_left">
       <origin xyz="${wheelbase/2} ${track/2} ${wheel_vertical_offset}" rpy="0 0 0" />
     </xacro:husky_wheel>
-    <xacro:husky_wheel wheel_prefix="front_right" prefix="${prefix}">
+    <xacro:husky_wheel wheel_prefix="front_right">
       <origin xyz="${wheelbase/2} ${-track/2} ${wheel_vertical_offset}" rpy="0 0 0" />
     </xacro:husky_wheel>
-    <xacro:husky_wheel wheel_prefix="rear_left" prefix="${prefix}">
+    <xacro:husky_wheel wheel_prefix="rear_left">
       <origin xyz="${-wheelbase/2} ${track/2} ${wheel_vertical_offset}" rpy="0 0 0" />
     </xacro:husky_wheel>
-    <xacro:husky_wheel wheel_prefix="rear_right" prefix="${prefix}">
+    <xacro:husky_wheel wheel_prefix="rear_right">
       <origin xyz="${-wheelbase/2} ${-track/2} ${wheel_vertical_offset}" rpy="0 0 0" />
     </xacro:husky_wheel>
-    <xacro:husky_decorate prefix="${prefix}"/>
+    <xacro:husky_decorate />
   </xacro:macro>
 </robot>

File: urdf/wheel.urdf.xacro (robot description, xacro)
@@ -3,5 +3,5 @@
 Software License Agreement (BSD)
 \file      wheel.urdf.xacro
-\authors   Paul Bovbel <pbovbel@clearpathrobotics.com
+\authors   Paul Bovbel <pbovbel@clearpathrobotics.com>
 \copyright Copyright (c) 2015, Clearpath Robotics, Inc., All rights reserved.
 Redistribution and use in source and binary forms, with or without modification, are permitted provided that
@@ -22,6 +22,6 @@
 -->
 <robot xmlns:xacro="http://ros.org/wiki/xacro" name="husky_wheel">
-	<xacro:macro name="husky_wheel" params="prefix wheel_prefix *joint_pose">
-		<link name="${prefix}${wheel_prefix}_wheel_link">
+	<xacro:macro name="husky_wheel" params="wheel_prefix *joint_pose">
+		<link name="${wheel_prefix}_wheel_link">
 			<inertial>
 				<mass value="2.637" />
@@ -43,5 +43,5 @@
 			</collision>
 		</link>
-		<gazebo reference="${prefix}${wheel_prefix}_wheel_link">
+		<gazebo reference="${wheel_prefix}_wheel_link">
 			<mu1 value="1.0"/>
 			<mu2 value="1.0"/>
@@ -52,16 +52,16 @@
 			<turnGravityOff>false</turnGravityOff>
 		</gazebo>
-		<joint name="${prefix}${wheel_prefix}_wheel" type="continuous">
-			<parent link="${prefix}chassis_link"/>
-			<child link="${prefix}${wheel_prefix}_wheel_link"/>
+		<joint name="${wheel_prefix}_wheel" type="continuous">
+			<parent link="chassis_link"/>
+			<child link="${wheel_prefix}_wheel_link"/>
 			<xacro:insert_block name="joint_pose"/>
 			<axis xyz="0 1 0" rpy="0 0 0" />
 		</joint>
-		<transmission name="${prefix}${wheel_prefix}_wheel_trans" type="SimpleTransmission">
+		<transmission name="${wheel_prefix}_wheel_trans" type="SimpleTransmission">
 			<type>transmission_interface/SimpleTransmission</type>
-			<actuator name="${prefix}${wheel_prefix}_wheel_motor">
+			<actuator name="${wheel_prefix}_wheel_motor">
 				<mechanicalReduction>1</mechanicalReduction>
 			</actuator>
-			<joint name="${prefix}${wheel_prefix}_wheel">
+			<joint name="${wheel_prefix}_wheel">
 				<hardwareInterface>VelocityJointInterface</hardwareInterface>
 			</joint>

Commit message: RP-264 Get rid of chassis_link, switch to base_footprint and base_link

File: urdf/decorations.urdf.xacro (robot description, xacro)
@@ -33,5 +33,5 @@
     </link>
     <joint name="top_plate" type="fixed">
-      <parent link="chassis_link" />
+      <parent link="base_link" />
       <child link="top_plate_link" />
     </joint>
@@ -49,5 +49,5 @@
     <joint name="user_rail" type="fixed">
       <origin xyz="0.272 0 0.245" rpy="0 0 0" />
-      <parent link="chassis_link" />
+      <parent link="base_link" />
       <child link="user_rail_link" />
     </joint>
@@ -65,5 +65,5 @@
     <joint name="front_bumper" type="fixed">
       <origin xyz="0.48 0 0.091" rpy="0 0 0" />
-      <parent link="chassis_link" />
+      <parent link="base_link" />
       <child link="front_bumper_link" />
     </joint>
@@ -81,5 +81,5 @@
     <joint name="rear_bumper" type="fixed">
       <origin xyz="-0.48 0 0.091" rpy="0 0 ${M_PI}" />
-      <parent link="chassis_link" />
+      <parent link="base_link" />
       <child link="rear_bumper_link" />
     </joint>

File: urdf/husky.urdf.xacro (robot description, xacro)
@@ -40,15 +40,15 @@
   <xacro:macro name="husky_robot">
     <!-- Base link is on the ground under the robot -->
-    <link name="base_link"/>
-    <gazebo reference="base_link">
+    <link name="base_footprint"/>
+    <gazebo reference="base_footprint">
       <material>Gazebo/DarkGrey</material>
     </gazebo>
     <joint name="chassis_joint" type="fixed">
       <origin xyz="0 0 ${wheel_radius - wheel_vertical_offset}" rpy="0 0 0" />
-      <parent link="base_link" />
-      <child link="chassis_link" />
+      <parent link="base_footprint" />
+      <child link="base_link" />
     </joint>
     <!-- Chassis link is the center of the robot's bottom plate -->
-    <link name="chassis_link">
+    <link name="base_link">
       <visual>
         <origin xyz="0 0 0" rpy="0 0 0" />
@@ -72,5 +72,5 @@
        </inertial>
      </link>
-     <gazebo reference="chassis_link">
+     <gazebo reference="base_link">
     </gazebo>
     <!-- IMU Link is the standard mounting position for the UM6 IMU.-->
@@ -79,5 +79,5 @@
     <joint name="imu_joint" type="fixed">
       <origin xyz="$(optenv HUSKY_IMU_XYZ 0.19 0 0.149)" rpy="$(optenv HUSKY_IMU_RPY 0 -1.5708 3.1416)" />
-      <parent link="chassis_link" />
+      <parent link="base_link" />
       <child link="imu_link" />
     </joint>

File: urdf/wheel.urdf.xacro (robot description, xacro)
@@ -53,5 +53,5 @@
 		</gazebo>
 		<joint name="${wheel_prefix}_wheel" type="continuous">
-			<parent link="chassis_link"/>
+			<parent link="base_link"/>
 			<child link="${wheel_prefix}_wheel_link"/>
 			<xacro:insert_block name="joint_pose"/>

Commit message: Add UR5 and Kinect to description

File: urdf/decorations.urdf.xacro (robot description, xacro)
@@ -3,5 +3,5 @@
 Software License Agreement (BSD)
 \file      decorations.urdf.xacro
-\authors   Paul Bovbel <pbovbel@clearpathrobotics.com>
+\authors   Paul Bovbel <pbovbel@clearpathrobotics.com>, Devon Ash <dash@clearpathrobotics.com>
 \copyright Copyright (c) 2015, Clearpath Robotics, Inc., All rights reserved.
 Redistribution and use in source and binary forms, with or without modification, are permitted provided that
@@ -23,20 +23,54 @@
 <robot name="husky_decorations" xmlns:xacro="http://ros.org/wiki/xacro">
   <xacro:macro name="husky_decorate">
-    <link name="top_plate_link">
+    <!-- Spawn Husky chassis -->
+    <link name="top_chassis_link">
       <visual>
         <origin xyz="0 0 0" rpy="0 0 0" />
         <geometry>
-          <mesh filename="package://husky_description/meshes/top_plate.stl" />
+          <mesh filename="package://husky_description/meshes/top_chassis.stl" />
         </geometry>
         <material name="Yellow" />
       </visual>
+      <collision>
+        <origin xyz="0 0 0" rpy="0 0 0"/>
+        <geometry>
+          <mesh filename="package://husky_description/meshes/top_chassis.stl" />
+        </geometry>
+      </collision>
     </link>
-    <joint name="top_plate" type="fixed">
+    <!-- Attach chassis to the robot -->
+    <joint name="top_chassis_joint" type="fixed">
       <parent link="base_link" />
-      <child link="top_plate_link" />
+      <child link="top_chassis_link" />
     </joint>
-    <gazebo reference="top_plate_link">
+    <gazebo reference="top_chassis_link">
       <material>Gazebo/Yellow</material>
     </gazebo>
+     <!-- Spawn the top plate -->
+     <link name="top_plate_link" type="fixed">
+	  <visual>
+		<origin xyz="0 0 0" rpy="0 0 0" />
+		<geometry>
+		<mesh filename="package://husky_description/meshes/top_plate.stl" />
+		</geometry>
+		<material name="Black" />
+	</visual>
+	<collision>
+		<origin xyz="0 0 0" rpy="0 0 0"/>
+		<geometry>
+                  <mesh filename="package://husky_description/meshes/top_plate.stl" />
+		</geometry>
+	</collision>
+    </link>
+    <gazebo reference="top_plate_link">
+      <material>Gazebo/DarkGrey</material>
+    </gazebo>
+   <!-- Attach custom top plate to Husky model -->
+   <joint name="top_plate_joint" type="fixed">
+      <parent link="base_link" />
+      <child link="top_plate_link"/>
+      <origin xyz="0.0812 0 0.245" rpy="0 0 0"/>
+   </joint>
+    <!-- Spawn user rails -->
     <link name="user_rail_link">
       <visual>
@@ -47,4 +81,5 @@
       </visual>
     </link>
+    <!-- Attach user rails to base link -->
     <joint name="user_rail" type="fixed">
       <origin xyz="0.272 0 0.245" rpy="0 0 0" />
@@ -55,4 +90,5 @@
       <material>Gazebo/DarkGrey</material>
     </gazebo>
+    <!-- Spawn front bumper link -->
     <link name="front_bumper_link">
       <visual>
@@ -63,4 +99,5 @@
       </visual>
     </link>
+    <!-- Attach front bumper -->
     <joint name="front_bumper" type="fixed">
       <origin xyz="0.48 0 0.091" rpy="0 0 0" />
@@ -71,4 +108,5 @@
       <material>Gazebo/DarkGrey</material>
     </gazebo>
+    <!-- Spawn rear bumper link -->
     <link name="rear_bumper_link">
       <visual>
@@ -79,4 +117,5 @@
       </visual>
     </link>
+    <!-- Attach rear bumper -->
     <joint name="rear_bumper" type="fixed">
       <origin xyz="-0.48 0 0.091" rpy="0 0 ${M_PI}" />

File: urdf/description.xacro (robot description, xacro)
@@ -3,5 +3,5 @@
 Software License Agreement (BSD)
 \file      description.urdf.xacro
-\authors   Paul Bovbel <pbovbel@clearpathrobotics.com>
+\authors   Paul Bovbel <pbovbel@clearpathrobotics.com>, Devon Ash <dash@clearpathrobotics.com>
 \copyright Copyright (c) 2015, Clearpath Robotics, Inc., All rights reserved.
 Redistribution and use in source and binary forms, with or without modification, are permitted provided that
@@ -22,4 +22,7 @@
 -->
 <robot name="husky" xmlns:xacro="http://ros.org/wiki/xacro">
+  <xacro:if value="$(arg ur5_enabled)">
+      <xacro:include filename="$(find husky_description)/urdf/ur5_arm.urdf.xacro"/>
+  </xacro:if>
   <xacro:include filename="$(find husky_description)/urdf/husky.urdf.xacro" />
   <xacro:husky_robot />

File: urdf/husky.urdf.xacro (robot description, xacro)
@@ -3,5 +3,5 @@
 Software License Agreement (BSD)
 \file      husky.urdf.xacro
-\authors   Paul Bovbel <pbovbel@clearpathrobotics.com>
+\authors   Paul Bovbel <pbovbel@clearpathrobotics.com>, Devon Ash <dash@clearpathrobotics.com>
 \copyright Copyright (c) 2015, Clearpath Robotics, Inc., All rights reserved.
 Redistribution and use in source and binary forms, with or without modification, are permitted provided that

Commit message: Changed name of parent link

File: urdf/decorations.urdf.xacro (robot description, xacro)
@@ -102,5 +102,5 @@
     </gazebo>
     <!-- Spawn the top plate -->
-    <link name="top_plate_link" type="fixed">
+    <link name="top_plate_link">
       <visual>
         <origin xyz="0 0 0" rpy="0 0 0" />
@@ -126,4 +126,27 @@
       <origin xyz="0.0812 0 0.245" rpy="0 0 0"/>
     </joint>
+    <!-- Spawn top plate widgets collision -->
+    <!-- Note this is so the UR5 arm does not collide with the top plate of the husky or plan through the widgets -->
+    <link name="top_plate_widgets">
+         <visual>
+         <origin xyz="0 0 0" rpy="0 0 0" />
+          <geometry>
+            <box size="0 0 0" rpy="0 0 0"/>
+          </geometry>
+        <material name="Black" />
+      </visual>
+      <collision>
+        <origin xyz="0 0 0" rpy="0 0 0"/>
+        <geometry>
+            <box size="0.32 0.41 0.09" rpy="0 0 0"/>
+          </geometry>
+      </collision>
+    </link>
+   <!-- Attach top plate widgets box -->
+   <joint name="top_plate_widgets_joint" type="fixed">
+       <parent link="top_plate_link" />
+      <child link="top_plate_widgets"/>
+      <origin xyz="0 0 0" rpy="0 0 0"/>
+   </joint>
   </xacro:macro>
 </robot>

Commit message: Indentation; Merge top plate collisions

File: urdf/decorations.urdf.xacro (robot description, xacro)
@@ -105,7 +105,7 @@
       <visual>
         <origin xyz="0 0 0" rpy="0 0 0" />
-          <geometry>
-            <mesh filename="package://husky_description/meshes/top_plate.stl" />
-          </geometry>
+        <geometry>
+          <mesh filename="package://husky_description/meshes/top_plate.stl" />
+        </geometry>
         <material name="Black" />
       </visual>
@@ -114,4 +114,10 @@
         <geometry>
           <mesh filename="package://husky_description/meshes/top_plate.stl" />
+        </geometry>
+      </collision>
+      <collision>
+        <!-- Extra collision tag for widgets typically attached to top plate -->
+        <geometry>
+          <box size="0.32 0.41 0.09" rpy="0 0 0"/>
         </geometry>
       </collision>
@@ -126,27 +132,4 @@
       <origin xyz="0.0812 0 0.245" rpy="0 0 0"/>
     </joint>
-    <!-- Spawn top plate widgets collision -->
-    <!-- Note this is so the UR5 arm does not collide with the top plate of the husky or plan through the widgets -->
-    <link name="top_plate_widgets">
-         <visual>
-         <origin xyz="0 0 0" rpy="0 0 0" />
-          <geometry>
-            <box size="0 0 0" rpy="0 0 0"/>
-          </geometry>
-        <material name="Black" />
-      </visual>
-      <collision>
-        <origin xyz="0 0 0" rpy="0 0 0"/>
-        <geometry>
-            <box size="0.32 0.41 0.09" rpy="0 0 0"/>
-          </geometry>
-      </collision>
-    </link>
-   <!-- Attach top plate widgets box -->
-   <joint name="top_plate_widgets_joint" type="fixed">
-       <parent link="top_plate_link" />
-      <child link="top_plate_widgets"/>
-      <origin xyz="0 0 0" rpy="0 0 0"/>
-   </joint>
   </xacro:macro>
 </robot>

File: urdf/husky.urdf.xacro (robot description, xacro)
@@ -79,14 +79,13 @@
         <mass value="33.455" />
         <origin xyz="-0.08748 -0.00085 0.09947" />
-        <inertia ixx="0.6022" ixy="-0.02364" ixz="-0.1197"
-         iyy="1.7386" iyz="-0.001544" izz="2.0296" />
-       </inertial>
-     </link>
-     <gazebo reference="base_link">
-     </gazebo>
-     <!-- IMU Link is the standard mounting position for the UM6 IMU.-->
-     <!-- Can be modified with environment variables in /etc/ros/setup.bash -->
-     <link name="imu_link"/>
-     <joint name="imu_joint" type="fixed">
+        <inertia ixx="0.6022" ixy="-0.02364" ixz="-0.1197" iyy="1.7386" iyz="-0.001544" izz="2.0296" />
+      </inertial>
+    </link>
+    <gazebo reference="base_link">
+    </gazebo>
+    <!-- IMU Link is the standard mounting position for the UM6 IMU.-->
+    <!-- Can be modified with environment variables in /etc/ros/setup.bash -->
+    <link name="imu_link"/>
+    <joint name="imu_joint" type="fixed">
       <origin xyz="$(optenv HUSKY_IMU_XYZ 0.19 0 0.149)" rpy="$(optenv HUSKY_IMU_RPY 0 -1.5708 3.1416)" />
       <parent link="base_link" />
@@ -129,13 +128,13 @@
     </xacro:if>
     <xacro:if value="$(arg kinect_enabled)">
-        <xacro:sensor_arch prefix="" parent="top_plate_link">
-            <origin xyz="-0.35 0 0.51" rpy="0 0 -3.14"/>
-        </xacro:sensor_arch>
-        <joint name="kinect_frame_joint" type="fixed">
-          <origin xyz="$(optenv HUSKY_KINECT_XYZ 0 0 0)" rpy="$(optenv HUSKY_KINECT_RPY 0 0.3925 3.14)" />
-          <parent link="sensor_arch_mount_link"/>
-          <child link="camera_link"/>
-        </joint>
-        <xacro:kinect_camera prefix="camera"/>
+      <xacro:sensor_arch prefix="" parent="top_plate_link">
+        <origin xyz="-0.35 0 0.51" rpy="0 0 -3.14"/>
+      </xacro:sensor_arch>
+      <joint name="kinect_frame_joint" type="fixed">
+        <origin xyz="$(optenv HUSKY_KINECT_XYZ 0 0 0)" rpy="$(optenv HUSKY_KINECT_RPY 0 0.3925 3.14)" />
+        <parent link="sensor_arch_mount_link"/>
+        <child link="camera_link"/>
+      </joint>
+      <xacro:kinect_camera prefix="camera"/>
     </xacro:if>
   </xacro:macro>
