Commit message: Pretty big refactor of URDF

File: urdf/accessories/kinect_camera.urdf.xacro (robot description, xacro)
@@ -1,5 +1,6 @@
 <?xml version="1.0"?>
 <!--
-Copyright (c) 2011, Siddhant Ahuja/WAVELab, Ryan Gariepy/Clearpath Robotics
+Copyright (c) 2013, Goncalo Cabrita, ISR University of Coimbra
+Copyright (c) 2014, Clearpath Robotics
 All rights reserved.
 Redistribution and use in source and binary forms, with or without
@@ -23,24 +24,24 @@
 (INCLUDING NEGLIGENCE OR OTHERWISE) ARISING IN ANY WAY OUT OF THE USE OF THIS
 SOFTWARE, EVEN IF ADVISED OF THE POSSIBILITY OF SUCH DAMAGE.
-This program contains the model file for a ground plane in Gazebo
 -->
- <!-- ground plane -->
- <model:physical name="g_plane">
-    <xyz>0 0 0</xyz>
-    <rpy>0 0 0</rpy>
-    <static>true</static>
-    <body:plane name="plane">
-      <geom:plane name="plane">
-        <laserRetro>2000.0</laserRetro>
-        <mu1>50.0</mu1> <!--friction coeficients-->
-        <mu2>50.0</mu2> <!--friction coeficients-->
-        <kp>1000000000.0</kp> <!--contact spring coeficients-->
-        <kd>1.0</kd> <!--contact spring coeficients-->
-        <normal>0 0 1</normal>
-        <size>102.4 102.4</size>
-        <segments>10 10</segments>
-        <uvTile>100 100</uvTile>
-        <material>Gazebo/GrayGrid</material>
-      </geom:plane>
-    </body:plane>
-  </model:physical>
+<robot xmlns:xacro="http://ros.org/wiki/xacro" name="kinect_camera">
+  <xacro:macro name="kinect_camera" params="prefix:=camera">
+    <!-- Create kinect reference frame -->
+    <!-- Add mesh for kinect -->
+    <link name="${prefix}_link">
+      <origin xyz="0 0 0" rpy="0 0 0"/>
+      <visual>
+        <origin xyz="0 0 0" rpy="0 0 ${M_PI/2}"/>
+        <geometry>
+          <mesh filename="package://husky_description/meshes/accessories/kinect.dae" />
+        </geometry>
+      </visual>
+      <!-- TODO switch to box -->
+      <collision>
+        <geometry>
+          <mesh filename="package://husky_description/meshes/accessories/kinect.dae" />
+        </geometry>
+      </collision>
+    </link>
+  </xacro:macro>
+</robot>

File: urdf/decorations.urdf.xacro (robot description, xacro)
@@ -22,4 +22,5 @@
 -->
 <robot name="husky_decorations" xmlns:xacro="http://ros.org/wiki/xacro">
+  <!-- TODO Move gazebo to husky_gazebo -->
   <xacro:macro name="husky_decorate">
     <!-- Spawn Husky chassis -->
@@ -47,29 +48,4 @@
       <material>Gazebo/Yellow</material>
     </gazebo>
-     <!-- Spawn the top plate -->
-     <link name="top_plate_link" type="fixed">
-	  <visual>
-		<origin xyz="0 0 0" rpy="0 0 0" />
-		<geometry>
-		<mesh filename="package://husky_description/meshes/top_plate.stl" />
-		</geometry>
-		<material name="Black" />
-	</visual>
-	<collision>
-		<origin xyz="0 0 0" rpy="0 0 0"/>
-		<geometry>
-                  <mesh filename="package://husky_description/meshes/top_plate.stl" />
-		</geometry>
-	</collision>
-    </link>
-    <gazebo reference="top_plate_link">
-      <material>Gazebo/DarkGrey</material>
-    </gazebo>
-   <!-- Attach custom top plate to Husky model -->
-   <joint name="top_plate_joint" type="fixed">
-      <parent link="base_link" />
-      <child link="top_plate_link"/>
-      <origin xyz="0.0812 0 0.245" rpy="0 0 0"/>
-   </joint>
     <!-- Spawn user rails -->
     <link name="user_rail_link">
@@ -126,4 +102,29 @@
       <material>Gazebo/DarkGrey</material>
     </gazebo>
+    <!-- Spawn the top plate -->
+    <link name="top_plate_link" type="fixed">
+      <visual>
+        <origin xyz="0 0 0" rpy="0 0 0" />
+          <geometry>
+            <mesh filename="package://husky_description/meshes/top_plate.stl" />
+          </geometry>
+        <material name="Black" />
+      </visual>
+      <collision>
+        <origin xyz="0 0 0" rpy="0 0 0"/>
+        <geometry>
+          <mesh filename="package://husky_description/meshes/top_plate.stl" />
+        </geometry>
+      </collision>
+    </link>
+    <gazebo reference="top_plate_link">
+      <material>Gazebo/DarkGrey</material>
+    </gazebo>
+    <!-- Attach top plate -->
+    <joint name="top_plate_joint" type="fixed">
+      <parent link="base_link" />
+      <child link="top_plate_link"/>
+      <origin xyz="0.0812 0 0.245" rpy="0 0 0"/>
+    </joint>
   </xacro:macro>
 </robot>

File: urdf/description.xacro (robot description, xacro)
@@ -22,7 +22,7 @@
 -->
 <robot name="husky" xmlns:xacro="http://ros.org/wiki/xacro">
-  <xacro:if value="$(arg ur5_enabled)">
-      <xacro:include filename="$(find husky_description)/urdf/ur5_arm.urdf.xacro"/>
-  </xacro:if>
+  <xacro:arg name="laser_enabled" default="true" />
+  <xacro:arg name="ur5_enabled" default="false" />
+  <xacro:arg name="kinect_enabled" default="false" />
   <xacro:include filename="$(find husky_description)/urdf/husky.urdf.xacro" />
   <xacro:husky_robot />

File: urdf/husky.urdf.xacro (robot description, xacro)
@@ -26,4 +26,8 @@
   <xacro:include filename="$(find husky_description)/urdf/wheel.urdf.xacro" />
   <xacro:include filename="$(find husky_description)/urdf/decorations.urdf.xacro" />
+  <xacro:include filename="$(find husky_description)/urdf/accessories/kinect_camera.urdf.xacro"/>
+  <xacro:include filename="$(find husky_description)/urdf/accessories/sick_lms100.urdf.xacro"/>
+  <xacro:include filename="$(find husky_description)/urdf/accessories/sensor_arch.urdf.xacro"/>
+  <xacro:include filename="$(find ur_description)/urdf/ur5.urdf.xacro" />
   <property name="M_PI" value="3.14159"/>
   <!-- Base Size -->
@@ -73,9 +77,9 @@
      </link>
      <gazebo reference="base_link">
-    </gazebo>
-    <!-- IMU Link is the standard mounting position for the UM6 IMU.-->
-    <!-- Can be modified with environment variables in /etc/ros/setup.bash -->
-    <link name="imu_link"/>
-    <joint name="imu_joint" type="fixed">
+     </gazebo>
+     <!-- IMU Link is the standard mounting position for the UM6 IMU.-->
+     <!-- Can be modified with environment variables in /etc/ros/setup.bash -->
+     <link name="imu_link"/>
+     <joint name="imu_joint" type="fixed">
       <origin xyz="$(optenv HUSKY_IMU_XYZ 0.19 0 0.149)" rpy="$(optenv HUSKY_IMU_RPY 0 -1.5708 3.1416)" />
       <parent link="base_link" />
@@ -98,4 +102,44 @@
     </xacro:husky_wheel>
     <xacro:husky_decorate />
+    <xacro:if value="$(arg ur5_enabled)">
+      <xacro:property name="reflect" value="-1" />
+      <!-- Spawn arm -->
+      <xacro:ur5_robot prefix="ur5_arm_" joint_limited="true"/>
+      <!-- Join arm -->
+      <joint name="ur5_arm_base" type="fixed">
+        <parent link="top_plate_link" />
+        <child link="ur5_arm_base_link" />
+        <origin xyz="0.3058 0 0.0065" rpy="0.0 0.0 0.0" />
+      </joint>
+    </xacro:if>
+    <xacro:if value="$(arg laser_enabled)">
+      <link name="base_laser_mount_link">
+        <visual>
+          <geometry>
+            <mesh filename="package://husky_description/meshes/accessories/lidar_mount.stl" />
+          </geometry>
+          <material name="DarkGrey" />
+        </visual>
+      </link>
+      <!-- TODO find better place for laser -->
+      <joint name="base_laser_mount" type="fixed">
+        <origin xyz="-0.12 0 0" rpy="0 0 0" />
+        <parent link="front_bumper_link" />
+        <child link="base_laser_mount_link" />
+      </joint>
+      <xacro:sick_lms100 prefix="base" />
+    </xacro:if>
+    <xacro:if value="$(arg kinect_enabled)">
+        <xacro:sensor_arch prefix="" parent="top_plate_link">
+            <origin xyz="-0.35 0 0.51" rpy="0 0 -3.14"/>
+        </xacro:sensor_arch>
+        <joint name="kinect_frame_joint" type="fixed">
+          <!-- TODO Fix x y z so kinect is not floating -->
+          <origin xyz="0 0 0" rpy="0 ${M_PI/8} ${M_PI}"/>
+          <parent link="sensor_arch_mount_link"/>
+          <child link="camera_link"/>
+        </joint>
+        <xacro:kinect_camera prefix="camera"/>
+    </xacro:if>
   </xacro:macro>
 </robot>

Commit message: Cleanup

File: urdf/accessories/kinect_camera.urdf.xacro (robot description, xacro)
@@ -40,5 +40,6 @@
       <collision>
         <geometry>
-          <mesh filename="package://husky_description/meshes/accessories/kinect.dae" />
+          <!-- <mesh filename="package://husky_description/meshes/accessories/kinect.dae" /> -->
+          <box size="0.07 0.3 0.09"/>
         </geometry>
       </collision>

File: urdf/accessories/sensor_arch.urdf.xacro (robot description, xacro)
@@ -19,5 +19,4 @@
              </collision>
         </link>
-        <!-- TODO move gazebo -->
         <gazebo reference="${prefix}sensor_arch_mount_link">
             <material>Gazebo/DarkGrey</material>

File: urdf/decorations.urdf.xacro (robot description, xacro)
@@ -22,5 +22,4 @@
 -->
 <robot name="husky_decorations" xmlns:xacro="http://ros.org/wiki/xacro">
-  <!-- TODO Move gazebo to husky_gazebo -->
   <xacro:macro name="husky_decorate">
     <!-- Spawn Husky chassis -->

File: urdf/husky.urdf.xacro (robot description, xacro)
@@ -124,5 +124,5 @@
       <!-- TODO find better place for laser -->
       <joint name="base_laser_mount" type="fixed">
-        <origin xyz="-0.12 0 0" rpy="0 0 0" />
+        <origin xyz="0 0 -0.05" rpy="0 0 0" />
         <parent link="front_bumper_link" />
         <child link="base_laser_mount_link" />

Commit message: Fix whitespace; Fix laser position; Fix collision model for husky base

File: urdf/accessories/kinect_camera.urdf.xacro (robot description, xacro)
@@ -37,8 +37,6 @@
         </geometry>
       </visual>
-      <!-- TODO switch to box -->
       <collision>
         <geometry>
-          <!-- <mesh filename="package://husky_description/meshes/accessories/kinect.dae" /> -->
           <box size="0.07 0.3 0.09"/>
         </geometry>

File: urdf/accessories/sensor_arch.urdf.xacro (robot description, xacro)
@@ -11,5 +11,4 @@
                  <material name="Grey" />
              </visual>
-             <!--TODO collision box-->
              <collision>
                  <origin xyz="0 0 0" rpy="0 0 0"/>

File: urdf/accessories/sick_lms100.urdf.xacro (robot description, xacro)
@@ -30,21 +30,13 @@
   <xacro:property name="laser_z" value="0.152" />
   <xacro:property name="laser_mass" value="1.1" />
-  <xacro:macro name="box_inertial" params="x y z mass">
-    <inertial>
-      <mass value="${mass}" />
-      <origin xyz="0 0 0" />
-      <inertia ixx="${0.0833333 * mass * (y*y + z*z)}" ixy="0.0" ixz="0.0"
-        iyy="${0.0833333 * mass * (x*x + z*z)}" iyz="0.0"
-        izz="${0.0833333 * mass * (x*x + y*y)}" />
-    </inertial>
-  </xacro:macro>
   <xacro:macro name="sick_lms100" params="prefix:=base">
-    <joint name="${prefix}_laser_joint" type="fixed">
-      <origin xyz="0.07 0 0.17" rpy="0 0 0" />
-      <parent link="${prefix}_laser_mount_link" />
-      <child link="${prefix}_laser" />
-    </joint>
     <link name="${prefix}_laser">
-      <xacro:box_inertial x="${laser_x}" y="${laser_y}" z="${laser_z}" mass="${laser_mass}" />
+      <inertial>
+        <mass value="${laser_mass}" />
+        <origin xyz="0 0 0" />
+        <inertia ixx="${0.0833333 * laser_mass * (laser_y*laser_y + laser_z*laser_z)}" ixy="0.0" ixz="0.0"
+          iyy="${0.0833333 * laser_mass * (laser_x*laser_x + laser_z*laser_z)}" iyz="0.0"
+          izz="${0.0833333 * laser_mass * (laser_x*laser_x + laser_y*laser_y)}" />
+      </inertial>
       <visual>
         <origin xyz="0 0 0" rpy="0 0 0" />
@@ -52,5 +44,5 @@
           <mesh filename="package://husky_description/meshes/accessories/sick_lms100.stl" />
         </geometry>
-        <material name="Grey" />
+        <material name="DarkGrey" />
       </visual>
       <collision>

File: urdf/husky.urdf.xacro (robot description, xacro)
@@ -64,8 +64,13 @@
       </visual>
       <collision>
-        <origin xyz="0 0 ${0.1578 - wheel_vertical_offset}" rpy="0 0 0" />
+        <origin xyz="0 0 ${base_z_size/4}" rpy="0 0 0" />
         <geometry>
-          <!-- Make collision box slightly bigger in x and z directions. -->
-          <box size = "${base_x_size+0.02} ${base_y_size} ${base_z_size + 0.02}"/>
+          <box size="${base_x_size} ${base_y_size} ${base_z_size/2}"/>
+        </geometry>
+      </collision>
+      <collision>
+        <origin xyz="0 0 ${base_z_size*3/4}" rpy="0 0 0" />
+        <geometry>
+          <box size="${base_x_size*4/5} ${base_y_size} ${base_z_size/2}"/>
         </geometry>
       </collision>
@@ -123,17 +128,8 @@
     </xacro:if>
     <xacro:if value="$(arg laser_enabled)">
-      <link name="base_laser_mount_link">
-        <visual>
-          <geometry>
-            <mesh filename="package://husky_description/meshes/accessories/lidar_mount.stl" />
-          </geometry>
-          <material name="DarkGrey" />
-        </visual>
-      </link>
-      <!-- TODO find better place for laser -->
       <joint name="base_laser_mount" type="fixed">
-        <origin xyz="0 0 -0.05" rpy="0 0 0" />
+        <origin xyz="-0.07 0 0.1" rpy="0 0 0" />
         <parent link="front_bumper_link" />
-        <child link="base_laser_mount_link" />
+        <child link="base_laser" />
       </joint>
       <xacro:sick_lms100 prefix="base" />
@@ -144,5 +140,4 @@
         </xacro:sensor_arch>
         <joint name="kinect_frame_joint" type="fixed">
-          <!-- TODO Fix x y z so kinect is not floating -->
           <origin xyz="0 0 0" rpy="0 ${M_PI/8} ${M_PI}"/>
           <parent link="sensor_arch_mount_link"/>
