Commit message: husky_description/urdf: add material color for better visualization for collision objects

File: husky_description/urdf/accessories/kinect_camera.urdf.xacro (robot description, xacro)
@@ -36,4 +36,7 @@
           <mesh filename="package://husky_description/meshes/accessories/kinect.dae" />
         </geometry>
+        <material name="LightGrey">
+          <color rgba="0.6 0.6 0.6 1.0"/>
+        </material>
       </visual>
       <collision>

File: husky_description/urdf/accessories/sensor_arch.urdf.xacro (robot description, xacro)
@@ -9,4 +9,7 @@
                      <mesh filename="package://husky_description/meshes/accessories/${size}_mm_sensor_arch.dae" />
                  </geometry>
+                 <material name="LightGrey">
+                   <color rgba="0.6 0.6 0.6 1.0"/>
+                 </material>
              </visual>
              <collision>

File: husky_description/urdf/decorations.urdf.xacro (robot description, xacro)
@@ -30,4 +30,7 @@
           <mesh filename="package://husky_description/meshes/top_chassis.dae" />
         </geometry>
+        <material name="LightGrey">
+          <color rgba="0.6 0.6 0.6 1.0"/>
+        </material>
       </visual>
     </link>
@@ -43,4 +46,7 @@
           <mesh filename="package://husky_description/meshes/user_rail.dae" />
         </geometry>
+        <material name="LightGrey">
+          <color rgba="0.6 0.6 0.6 1.0"/>
+        </material>
       </visual>
     </link>
@@ -57,4 +63,7 @@
           <mesh filename="package://husky_description/meshes/bumper.dae" />
         </geometry>
+        <material name="LightGrey">
+          <color rgba="0.6 0.6 0.6 1.0"/>
+        </material>
       </visual>
     </link>
@@ -71,4 +80,7 @@
           <mesh filename="package://husky_description/meshes/bumper.dae" />
         </geometry>
+        <material name="LightGrey">
+          <color rgba="0.6 0.6 0.6 1.0"/>
+        </material>
       </visual>
     </link>
@@ -87,4 +99,7 @@
             <mesh filename="package://husky_description/meshes/top_plate.dae" />
           </geometry>
+          <material name="LightGrey">
+            <color rgba="0.6 0.6 0.6 1.0"/>
+          </material>
         </visual>
         <collision>

File: husky_description/urdf/husky.urdf.xacro (robot description, xacro)
@@ -50,4 +50,7 @@
           <mesh filename="package://husky_description/meshes/base_link.dae" />
         </geometry>
+        <material name="LightGrey">
+          <color rgba="0.6 0.6 0.6 1.0"/>
+        </material>
       </visual>
       <collision>

File: husky_description/urdf/wheel.urdf.xacro (robot description, xacro)
@@ -34,4 +34,7 @@
 					<mesh filename="package://husky_description/meshes/wheel.dae" />
 				</geometry>
+                                <material name="LightGrey">
+                                  <color rgba="0.6 0.6 0.6 1.0"/>
+                                </material>
 			</visual>
 			<collision>
