Commit message: Use the STL from realsense2_description, rotated as necessary. Add realsense2_description to the dependencies

File: husky_description/urdf/accessories/intel_realsense.urdf.xacro (robot description, xacro)
@@ -71,8 +71,12 @@
     <link name="${prefix}_realsense_lens">
       <visual>
-        <origin xyz="0 0 0" rpy="0 0 0" />
+        <!--
+          the model's origin is in the middle & it's rotated to lie in
+          the optical standard with X left, Y up, and Z forward
+        -->
+        <origin xyz="0.0115 0 0.0100" rpy="1.570796 0 1.570796" />
         <geometry>
           <!-- Origin of this mesh is the base of the bracket. -->
-          <mesh filename="package://husky_description/meshes/accessories/intel_realsense_d415.stl" />
+          <mesh filename="package://realsense2_description/meshes/d415.stl" />
         </geometry>
         <material name="white" />
