Commit message: Start adding out-of-the-box support for the Hokuyo UST10

File: husky_description/urdf/accessories/hokuyo_ust10.urdf.xacro (robot description, xacro)
@@ -53,5 +53,5 @@
         <geometry>
           <!-- Origin of this mesh is the base of the bracket. -->
-          <mesh filename="package://husky_description/meshes/accessories/hokuyo_ust10.stl" />
+          <mesh filename="package://jackal_description/meshes/hokuyo_ust10.stl" />
         </geometry>
         <material name="dark_grey" />
@@ -60,5 +60,5 @@
     <joint name="${prefix}_laser_joint" type="fixed">
       <!-- This offset is from the base of the bracket to the LIDAR's focal point. -->
-      <origin xyz="0 0 0" rpy="0 0 0" />
+      <origin xyz="0 0 0.149" rpy="0 0 0" />
       <parent link="${prefix}_laser_mount" />
       <child link="${prefix}_laser" />

Commit message: Fix the package for the ust10 mesh

File: husky_description/urdf/accessories/hokuyo_ust10.urdf.xacro (robot description, xacro)
@@ -53,5 +53,5 @@
         <geometry>
           <!-- Origin of this mesh is the base of the bracket. -->
-          <mesh filename="package://jackal_description/meshes/hokuyo_ust10.stl" />
+          <mesh filename="package://husky_description/meshes/hokuyo_ust10.stl" />
         </geometry>
         <material name="dark_grey" />

Commit message: Added UST10 mesh

File: husky_description/urdf/accessories/hokuyo_ust10.urdf.xacro (robot description, xacro)
@@ -58,5 +58,5 @@
         <geometry>
           <!-- Origin of this mesh is the base of the bracket. -->
-          <mesh filename="package://jackal_description/meshes/hokuyo_ust10.stl" />
+          <mesh filename="package://husky_description/meshes/accessories/hokuyo_ust10.stl" />
         </geometry>
         <material name="dark_grey" />
