Commit message: Remove the prefix's trailing underscore in the vlp16 mount to make it consistent. Fix an inconsistent envar for the sensor arch, add an arg to explicitly enable it, to stay internally consistent with the rest of Husky.

File: husky_description/urdf/accessories/vlp16_mount.urdf.xacro (robot description, xacro)
@@ -6,6 +6,6 @@
       The VLP16 is mounted to a pair of extrusion rods on top of the main sensor arch
     -->
-    <link name="${prefix}_vlp16_mount_base_link" />
-    <link name="${prefix}_vlp16_mount_left_support">
+    <link name="${prefix}vlp16_mount_base_link" />
+    <link name="${prefix}vlp16_mount_left_support">
       <visual>
         <geometry>
@@ -24,5 +24,5 @@
       </collision>
     </link>
-    <link name="${prefix}_vlp16_mount_right_support">
+    <link name="${prefix}vlp16_mount_right_support">
       <visual>
         <geometry>
@@ -41,20 +41,20 @@
       </collision>
     </link>
-    <joint name="${prefix}_vlp16_mount_base_link_joint" type="fixed">
+    <joint name="${prefix}vlp16_mount_base_link_joint" type="fixed">
       <parent link="${parent_link}" />
-      <child link="${prefix}_vlp16_mount_base_link" />
+      <child link="${prefix}vlp16_mount_base_link" />
       <xacro:insert_block name="origin" />
     </joint>
-    <joint name="${prefix}_vlp16_mount_left_support_joint" type="fixed">
-      <parent link="${prefix}_vlp16_mount_base_link" />
-      <child link="${prefix}_vlp16_mount_left_support" />
+    <joint name="${prefix}vlp16_mount_left_support_joint" type="fixed">
+      <parent link="${prefix}vlp16_mount_base_link" />
+      <child link="${prefix}vlp16_mount_left_support" />
       <origin xyz="0 0.04 ${height/2}" rpy="0 0 0"/>
     </joint>
-    <joint name="${prefix}_vlp16_mount_right_support_joint" type="fixed">
-      <parent link="${prefix}_vlp16_mount_base_link" />
-      <child link="${prefix}_vlp16_mount_right_support" />
+    <joint name="${prefix}vlp16_mount_right_support_joint" type="fixed">
+      <parent link="${prefix}vlp16_mount_base_link" />
+      <child link="${prefix}vlp16_mount_right_support" />
       <origin xyz="0 -0.04 ${height/2}" rpy="0 0 0"/>
     </joint>
-    <xacro:VLP-16 parent="${prefix}_vlp16_mount_base_link" topic="${topic}">
+    <xacro:VLP-16 parent="${prefix}vlp16_mount_base_link" topic="${topic}">
       <origin xyz="0 0 ${height}" rpy="0 0 0" />
     </xacro:VLP-16>

File: husky_description/urdf/husky.urdf.xacro (robot description, xacro)
@@ -39,4 +39,5 @@
   <!-- Height of the sensor arch in mm.  Must be either 510 or 300 -->
   <xacro:arg name="sensor_arch_height"  default="$(optenv HUSKY_SENSOR_ARCH_HEIGHT 510)" />
+  <xacro:arg name="sensor_arch"         default="$(optenv HUSKY_SENSOR_ARCH 0)" />
   <xacro:arg name="robot_namespace" default="/" />
   <xacro:arg name="urdf_extras" default="empty.urdf" />
@@ -150,7 +151,7 @@
     requires it for mounting
   -->
-  <xacro:property name="sensorbar_user_enabled"     value="$(optenv HUSKY_SENSOR_ARCH 0)" />
+  <xacro:property name="sensorbar_user_enabled"     value="$(arg sensor_arch)" />
   <xacro:property name="sensorbar_needed_realsense" value="$(arg realsense_enabled)" />
-  <xacro:property name="sensorbar_needed_lidar"     value="$(optenv HUSKY_LASER_3D 0)" />
+  <xacro:property name="sensorbar_needed_lidar"     value="$(arg laser_3d_enabled)" />
   <xacro:if value="${sensorbar_needed_realsense or sensorbar_user_enabled or sensorbar_needed_lidar}">
     <xacro:sensor_arch prefix="" parent="top_plate_link" size="$(arg sensor_arch_height)">

Commit message: Update mount support dimensions and spacing to better represent real-world measurements

File: husky_description/urdf/accessories/vlp16_mount.urdf.xacro (robot description, xacro)
@@ -10,7 +10,7 @@
       <visual>
         <geometry>
-          <box size="0.012 0.012 ${height}" />
+          <box size="0.04 0.02 ${height}" />
         </geometry>
-        <material name="white">
+        <material name="black">
           <color rgba="1 1 1 1" />
         </material>
@@ -19,5 +19,5 @@
       <collision>
         <geometry>
-          <box size="0.012 0.012 ${height}" />
+          <box size="0.04 0.02 ${height}" />
         </geometry>
         <origin xyz="0 0 0" rpy="0 0 0" />
@@ -27,7 +27,7 @@
       <visual>
         <geometry>
-          <box size="0.012 0.012 ${height}" />
+          <box size="0.04 0.02 ${height}" />
         </geometry>
-        <material name="white">
+        <material name="black">
           <color rgba="1 1 1 1" />
         </material>
@@ -36,5 +36,5 @@
       <collision>
         <geometry>
-          <box size="0.012 0.012 ${height}" />
+          <box size="0.04 0.02 ${height}" />
         </geometry>
         <origin xyz="0 0 0" rpy="0 0 0" />
@@ -49,10 +49,10 @@
       <parent link="${prefix}vlp16_mount_base_link" />
       <child link="${prefix}vlp16_mount_left_support" />
-      <origin xyz="0 0.04 ${height/2}" rpy="0 0 0"/>
+      <origin xyz="0 0.06 ${height/2}" rpy="0 0 0"/>
     </joint>
     <joint name="${prefix}vlp16_mount_right_support_joint" type="fixed">
       <parent link="${prefix}vlp16_mount_base_link" />
       <child link="${prefix}vlp16_mount_right_support" />
-      <origin xyz="0 -0.04 ${height/2}" rpy="0 0 0"/>
+      <origin xyz="0 -0.06 ${height/2}" rpy="0 0 0"/>
     </joint>
     <xacro:VLP-16 parent="${prefix}vlp16_mount_base_link" topic="${topic}">

Commit message: Create visual geometry of vlp16_mount_base_link

File: husky_description/urdf/accessories/vlp16_mount.urdf.xacro (robot description, xacro)
@@ -6,5 +6,21 @@
       The VLP16 is mounted to a pair of extrusion rods on top of the main sensor arch
     -->
-    <link name="${prefix}vlp16_mount_base_link" />
+    <link name="${prefix}vlp16_mount_base_link">
+      <visual>
+        <geometry>
+          <box size="0.04 0.141 0.0063" />
+        </geometry>
+        <material name="black">
+          <color rgba="1 1 1 1" />
+        </material>
+        <origin xyz="0 0 0" rpy="0 0 0" />
+      </visual>
+      <collision>
+        <geometry>
+          <box size="0.04 0.02 ${height}" />
+        </geometry>
+        <origin xyz="0 0 0" rpy="0 0 0" />
+      </collision>
+    </link>
     <link name="${prefix}vlp16_mount_left_support">
       <visual>
@@ -44,18 +60,18 @@
       <parent link="${parent_link}" />
       <child link="${prefix}vlp16_mount_base_link" />
-      <xacro:insert_block name="origin" />
+      <origin xyz="0 0 ${height}" rpy="0 0 0"/>
     </joint>
     <joint name="${prefix}vlp16_mount_left_support_joint" type="fixed">
       <parent link="${prefix}vlp16_mount_base_link" />
       <child link="${prefix}vlp16_mount_left_support" />
-      <origin xyz="0 0.06 ${height/2}" rpy="0 0 0"/>
+      <origin xyz="0 0.06 -${height/2}" rpy="0 0 0"/>
     </joint>
     <joint name="${prefix}vlp16_mount_right_support_joint" type="fixed">
       <parent link="${prefix}vlp16_mount_base_link" />
       <child link="${prefix}vlp16_mount_right_support" />
-      <origin xyz="0 -0.06 ${height/2}" rpy="0 0 0"/>
+      <origin xyz="0 -0.06 -${height/2}" rpy="0 0 0"/>
     </joint>
     <xacro:VLP-16 parent="${prefix}vlp16_mount_base_link" topic="${topic}">
-      <origin xyz="0 0 ${height}" rpy="0 0 0" />
+      <origin xyz="0 0 0" rpy="0 0 0" />
     </xacro:VLP-16>
   </xacro:macro>

Commit message: Revert changes to mount_base_link to preserve use of origin argument; instead, simply created an additional plate link that sits between the supports and VLP16

File: husky_description/urdf/accessories/vlp16_mount.urdf.xacro (robot description, xacro)
@@ -6,5 +6,6 @@
       The VLP16 is mounted to a pair of extrusion rods on top of the main sensor arch
     -->
-    <link name="${prefix}vlp16_mount_base_link">
+    <link name="${prefix}vlp16_mount_base_link" />
+    <link name="${prefix}vlp16_mount_plate">
       <visual>
         <geometry>
@@ -60,17 +61,22 @@
       <parent link="${parent_link}" />
       <child link="${prefix}vlp16_mount_base_link" />
-      <origin xyz="0 0 ${height}" rpy="0 0 0"/>
+      <xacro:insert_block name="origin" />
     </joint>
     <joint name="${prefix}vlp16_mount_left_support_joint" type="fixed">
       <parent link="${prefix}vlp16_mount_base_link" />
       <child link="${prefix}vlp16_mount_left_support" />
-      <origin xyz="0 0.06 -${height/2}" rpy="0 0 0"/>
+      <origin xyz="0 0.06 ${height/2}" rpy="0 0 0"/>
     </joint>
     <joint name="${prefix}vlp16_mount_right_support_joint" type="fixed">
       <parent link="${prefix}vlp16_mount_base_link" />
       <child link="${prefix}vlp16_mount_right_support" />
-      <origin xyz="0 -0.06 -${height/2}" rpy="0 0 0"/>
+      <origin xyz="0 -0.06 ${height/2}" rpy="0 0 0"/>
     </joint>
-    <xacro:VLP-16 parent="${prefix}vlp16_mount_base_link" topic="${topic}">
+    <joint name="${prefix}vlp16_mount_plate_joint" type="fixed">
+      <parent link="${prefix}vlp16_mount_base_link" />
+      <child link="${prefix}vlp16_mount_plate" />
+      <origin xyz="0 0 ${height}" rpy="0 0 0"/>
+    </joint>
+    <xacro:VLP-16 parent="${prefix}vlp16_mount_plate" topic="${topic}">
       <origin xyz="0 0 0" rpy="0 0 0" />
     </xacro:VLP-16>

Commit message: First commit

File: husky_description/urdf/accessories/vlp16_mount.urdf.xacro (robot description, xacro)
@@ -1,4 +1,5 @@
 <?xml version="1.0"?>
 <robot xmlns:xacro="http://wiki.ros.org/xacro">
+  <xacro:property name="M_PI" value="3.1415926535897931" />
   <xacro:include filename="$(find velodyne_description)/urdf/VLP-16.urdf.xacro" />
   <xacro:macro name="vlp16_mount" params="prefix parent_link topic height:=0.12 *origin">
@@ -56,6 +57,11 @@
       <origin xyz="0 -0.04 ${height/2}" rpy="0 0 0"/>
     </joint>
+<<<<<<< HEAD
     <xacro:VLP-16 parent="${prefix}vlp16_mount_base_link" topic="${topic}">
       <origin xyz="0 0 ${height}" rpy="0 0 0" />
+=======
+    <xacro:VLP-16 parent="${prefix}vlp16_mount_plate" topic="${topic}" gpu="true">
+      <origin xyz="0 0 0" rpy="0 0 0" />
+>>>>>>> c14491e... First commit
     </xacro:VLP-16>
   </xacro:macro>

File: husky_description/urdf/husky.urdf.xacro (robot description, xacro)
@@ -126,4 +126,13 @@
   <gazebo reference="imu_link">
   </gazebo>
+  <!-- GPS Link is the standard mounting position for the GPS-->
+  <link name="gps_link"/>
+  <joint name="gps_joint" type="fixed">
+    <origin xyz="$(optenv HUSKY_GPS_XYZ 0.0 0.0 0.5)" rpy="$(optenv HUSKY_GPS_RPY 0 0 0)" />
+    <parent link="base_link" />
+    <child link="gps_link" />
+  </joint>
+  <gazebo reference="gps_link">
+  </gazebo>
   <!-- Husky wheel macros -->
   <xacro:husky_wheel wheel_prefix="front_left">
@@ -227,11 +236,11 @@
     <plugin name="gps_controller" filename="libhector_gazebo_ros_gps.so">
       <robotNamespace>$(arg robot_namespace)</robotNamespace>
-      <updateRate>40</updateRate>
-      <bodyName>base_link</bodyName>
-      <frameId>base_link</frameId>
+      <updateRate>40.0</updateRate>
+      <bodyName>gps_link</bodyName>
+      <frameId>gps_link</frameId>
       <topicName>navsat/fix</topicName>
       <velocityTopicName>navsat/vel</velocityTopicName>
-      <referenceLatitude>49.9</referenceLatitude>
-      <referenceLongitude>8.9</referenceLongitude>
+      <referenceLatitude>48.711254</referenceLatitude>
+      <referenceLongitude>2.217765</referenceLongitude>
       <referenceHeading>0</referenceHeading>
       <referenceAltitude>0</referenceAltitude>

Commit message: Update vlp16_mount.urdf.xacro

File: husky_description/urdf/accessories/vlp16_mount.urdf.xacro (robot description, xacro)
@@ -57,11 +57,6 @@
       <origin xyz="0 -0.04 ${height/2}" rpy="0 0 0"/>
     </joint>
-<<<<<<< HEAD
-    <xacro:VLP-16 parent="${prefix}vlp16_mount_base_link" topic="${topic}">
-      <origin xyz="0 0 ${height}" rpy="0 0 0" />
-=======
     <xacro:VLP-16 parent="${prefix}vlp16_mount_plate" topic="${topic}" gpu="true">
       <origin xyz="0 0 0" rpy="0 0 0" />
->>>>>>> c14491e... First commit
     </xacro:VLP-16>
   </xacro:macro>

Commit message: Fixes for velodyne prefix

File: husky_description/urdf/accessories/vlp16_mount.urdf.xacro (robot description, xacro)
@@ -15,5 +15,5 @@
           <color rgba="1 1 1 1" />
         </material>
-        <origin xyz="0 0 0" rpy="0 0 0" />
+        <origin xyz="0 0 0.00315" rpy="0 0 0" />
       </visual>
       <collision>
@@ -79,5 +79,5 @@
     </joint>
     <xacro:VLP-16 parent="${prefix}vlp16_mount_plate" topic="${topic}" name="${prefix}velodyne">
-      <origin xyz="0 0 0" rpy="0 0 0" />
+      <origin xyz="0 0 0.0063" rpy="0 0 0" />
     </xacro:VLP-16>
   </xacro:macro>

File: husky_description/urdf/husky.urdf.xacro (robot description, xacro)
@@ -56,5 +56,5 @@
   <xacro:arg name="laser_3d_topic"                default="$(optenv HUSKY_LASER_3D_TOPIC points)"/>
   <xacro:arg name="laser_3d_tower"                default="$(optenv HUSKY_LASER_3D_TOWER 1)"/>
-  <xacro:arg name="laser_3d_prefix"               default="$(optenv HUSKY_LASER_3D_PREFIX '')"/>
+  <xacro:arg name="laser_3d_prefix"               default="$(optenv HUSKY_LASER_3D_PREFIX )"/>
   <xacro:arg name="laser_3d_parent"               default="$(optenv HUSKY_LASER_3D_PARENT top_plate_link)"/>
   <xacro:arg name="laser_3d_xyz"                  default="$(optenv HUSKY_LASER_3D_XYZ 0 0 0)" />
@@ -284,5 +284,5 @@
     </xacro:if>
     <xacro:unless value="$(arg laser_3d_tower)">
-      <xacro:VLP-16 parent="$(arg laser_3d_parent)" topic="$(arg laser_3d_topic)" name="$(arg laser_3d_prefix)_velodyne">
+      <xacro:VLP-16 parent="$(arg laser_3d_parent)" topic="$(arg laser_3d_topic)" name="$(arg laser_3d_prefix)velodyne">
         <origin xyz="$(arg laser_3d_xyz)" rpy="$(arg laser_3d_rpy)" />
       </xacro:VLP-16>
