Commit message: Minor bugfix for wheelconfig

File: husky_description_mbzirc/urdf/description.xacro (robot description, xacro)
@@ -25,5 +25,6 @@
   <xacro:arg name="ur5_enabled" default="false" />
   <xacro:arg name="kinect_enabled" default="false" />
+  <xacro:arg name="wheelconfig_full" default="true"/> <!-- true: 4wheel, false: 2wheel -->
   <xacro:include filename="$(find husky_description_mbzirc)/urdf/husky.urdf.xacro" />
-  <xacro:husky_robot />
+  <xacro:husky_robot wheelconfig_full="$(arg wheelconfig_full)" />
 </robot>

File: husky_description_mbzirc/urdf/husky.urdf.xacro (robot description, xacro)
@@ -39,5 +39,5 @@
   <xacro:property name="wheel_length" value="0.1143" />
   <xacro:property name="wheel_radius" value="0.17775" />
-  <xacro:macro name="husky_robot" params="wheelconfig">
+  <xacro:macro name="husky_robot" params="wheelconfig_full">
     <!-- Base link is the center of the robot's bottom plate -->
     <link name="base_link">
