Commit message: Allow projection of rear wheel inertias onto front wheels.

File: husky_description_mbzirc/urdf/husky.urdf.xacro (robot description, xacro)
@@ -92,23 +92,29 @@
     </gazebo>
     <!-- Husky wheel macros -->
-    <xacro:husky_wheel wheel_prefix="front_left" fixed="false">
-      <origin xyz="${wheelbase/2} ${track/2} ${wheel_vertical_offset}" rpy="0 0 0" />
-    </xacro:husky_wheel>
-    <xacro:husky_wheel wheel_prefix="front_right" fixed="false">
-      <origin xyz="${wheelbase/2} ${-track/2} ${wheel_vertical_offset}" rpy="0 0 0" />
-    </xacro:husky_wheel>
     <xacro:if value="${wheelconfig_full}">
-	    <xacro:husky_wheel wheel_prefix="rear_left" fixed="false">
+      <xacro:husky_wheel wheel_prefix="front_left" fixed="false" double_inertia="false">
+        <origin xyz="${wheelbase/2} ${track/2} ${wheel_vertical_offset}" rpy="0 0 0" />
+      </xacro:husky_wheel>
+      <xacro:husky_wheel wheel_prefix="front_right" fixed="false" double_inertia="false">
+        <origin xyz="${wheelbase/2} ${-track/2} ${wheel_vertical_offset}" rpy="0 0 0" />
+      </xacro:husky_wheel>
+	    <xacro:husky_wheel wheel_prefix="rear_left" fixed="false" double_inertia="false">
 	      <origin xyz="${-wheelbase/2} ${track/2} ${wheel_vertical_offset}" rpy="0 0 0" />
 	    </xacro:husky_wheel>
-	    <xacro:husky_wheel wheel_prefix="rear_right" fixed="false">
+	    <xacro:husky_wheel wheel_prefix="rear_right" fixed="false" double_inertia="false">
 	      <origin xyz="${-wheelbase/2} ${-track/2} ${wheel_vertical_offset}" rpy="0 0 0" />
 	    </xacro:husky_wheel>
 	  </xacro:if>
 	  <xacro:unless value="${wheelconfig_full}">
-      <xacro:husky_wheel wheel_prefix="rear_left" fixed="true">
+      <xacro:husky_wheel wheel_prefix="front_left" fixed="false" double_inertia="true">
+        <origin xyz="${wheelbase/2} ${track/2} ${wheel_vertical_offset}" rpy="0 0 0" />
+      </xacro:husky_wheel>
+      <xacro:husky_wheel wheel_prefix="front_right" fixed="false" double_inertia="true">
+        <origin xyz="${wheelbase/2} ${-track/2} ${wheel_vertical_offset}" rpy="0 0 0" />
+      </xacro:husky_wheel>
+      <xacro:husky_wheel wheel_prefix="rear_left" fixed="true" double_inertia="false">
         <origin xyz="${-wheelbase/2} ${track/2} ${wheel_vertical_offset}" rpy="0 0 0" />
       </xacro:husky_wheel>
-      <xacro:husky_wheel wheel_prefix="rear_right" fixed="true">
+      <xacro:husky_wheel wheel_prefix="rear_right" fixed="true" double_inertia="false">
         <origin xyz="${-wheelbase/2} ${-track/2} ${wheel_vertical_offset}" rpy="0 0 0" />
       </xacro:husky_wheel>

File: husky_description_mbzirc/urdf/wheel.urdf.xacro (robot description, xacro)
@@ -22,10 +22,15 @@
 -->
 <robot xmlns:xacro="http://ros.org/wiki/xacro" name="husky_wheel">
-	<xacro:macro name="husky_wheel" params="wheel_prefix fixed *joint_pose">
+	<xacro:macro name="husky_wheel" params="wheel_prefix fixed double_inertia *joint_pose">
 		<link name="${wheel_prefix}_wheel_link">
 			<inertial>
 				<mass value="2.637" />
 				<origin xyz="0 0 0" />
-				<inertia  ixx="0.02467" ixy="0" ixz="0" iyy="0.02467" iyz="0" izz="0.04411" />
+        <xacro:if value="${double_inertia}">
+          <inertia  ixx="0.02467" ixy="0" ixz="0" iyy="${2*0.02467}" iyz="0" izz="0.04411" />
+        </xacro:if>
+        <xacro:unless value="${double_inertia}">
+          <inertia  ixx="0.02467" ixy="0" ixz="0" iyy="0.02467" iyz="0" izz="0.04411" />
+        </xacro:unless>
 			</inertial>
 			<visual>

Commit message: Remove kinect parameter and inclusion

File: husky_description_mbzirc/urdf/husky.urdf.xacro (robot description, xacro)
@@ -121,15 +121,4 @@
 	  </xacro:unless>
     <xacro:husky_decorate />
-    <xacro:if value="$(arg kinect_enabled)">
-      <xacro:sensor_arch prefix="" parent="top_plate_link">
-        <origin xyz="-0.35 0 0.51" rpy="0 0 -3.14"/>
-      </xacro:sensor_arch>
-      <joint name="kinect_frame_joint" type="fixed">
-        <origin xyz="$(optenv HUSKY_KINECT_XYZ 0 0 0)" rpy="$(optenv HUSKY_KINECT_RPY 0 0.18 3.14)" />
-        <parent link="sensor_arch_mount_link"/>
-        <child link="camera_link"/>
-      </joint>
-      <xacro:kinect_camera prefix="camera"/>
-    </xacro:if>
   </xacro:macro>
 </robot>

Commit message: Husky description: Add GPS and IMU controllers + mounting

File: husky_description_mbzirc/urdf/husky.urdf.xacro (robot description, xacro)
@@ -121,4 +121,51 @@
 	  </xacro:unless>
     <xacro:husky_decorate />
+    <!-- Attaching additional sensors and frames to husky -->
+    <!-- GPS mounting position -->
+    <link name="gps_mount_link"/>
+    <joint name="gps_joint" type="fixed">
+      <origin xyz="-0.14 -0.20 0.65" rpy="0 0 0" />
+      <parent link="base_link" />
+      <child link="gps_mount_link" />
+    </joint>
+    <gazebo reference="gps_mount_link">
+    </gazebo>
+    <!-- GPS controller plugin for gazebo -->
+    <xacro:if value="$(arg simulation)">
+      <gazebo>
+        <plugin name="gps_controller" filename="libhector_gazebo_ros_gps.so">
+          <updateRate>40</updateRate>
+          <robotNamespace>/</robotNamespace>
+          <bodyName>base_link</bodyName>
+          <frameId>base_link</frameId>
+          <topicName>navsat/fix</topicName>
+          <velocityTopicName>navsat/vel</velocityTopicName>
+          <referenceLatitude>49.9</referenceLatitude>
+          <referenceLongitude>8.9</referenceLongitude>
+          <referenceHeading>0</referenceHeading>
+          <referenceAltitude>0</referenceAltitude>
+          <drift>0.0001 0.0001 0.0001</drift>
+        </plugin>
+      </gazebo>
+    </xacro:if>
+    <!-- IMU controller plugin for gazebo -->
+    <xacro:if value="$(arg simulation)">
+      <gazebo>
+        <plugin name="imu_controller" filename="libhector_gazebo_ros_imu.so">
+          <robotNamespace>/</robotNamespace>
+          <updateRate>50.0</updateRate>
+          <bodyName>base_link</bodyName>
+          <topicName>imu/data</topicName>
+          <accelDrift>0.005 0.005 0.005</accelDrift>
+          <accelGaussianNoise>0.005 0.005 0.005</accelGaussianNoise>
+          <rateDrift>0.005 0.005 0.005 </rateDrift>
+          <rateGaussianNoise>0.005 0.005 0.005 </rateGaussianNoise>
+          <headingDrift>0.005</headingDrift>
+          <headingGaussianNoise>0.005</headingGaussianNoise>
+          <xyzOffset>0 0 0</xyzOffset>
+          <rpyOffset>0 0 0</rpyOffset>
+        </plugin>
+      </gazebo>
+    </xacro:if>
   </xacro:macro>
 </robot>

Commit message: introduce velodyne mount link

File: husky_description_mbzirc/urdf/husky.urdf.xacro (robot description, xacro)
@@ -122,4 +122,13 @@
     <xacro:husky_decorate />
     <!-- Attaching additional sensors and frames to husky -->
+    <!-- Velodyne laser -->
+    <link name="velodyne_mount_link"/>
+    <joint name="velodyne_joint" type="fixed">
+      <origin xyz="0.23 0 0.35" rpy="0 0 ${PI}" />
+      <parent link="base_link" />
+      <child link="velodyne_mount_link" />
+    </joint>
+    <gazebo reference="velodyne_mount_link">
+    </gazebo>
     <!-- GPS mounting position -->
     <link name="gps_mount_link"/>

Commit message: updated description (new box)

File: husky_description_mbzirc/urdf/husky.urdf.xacro (robot description, xacro)
@@ -125,5 +125,5 @@
     <link name="velodyne_mount_link"/>
     <joint name="velodyne_joint" type="fixed">
-      <origin xyz="0.23 0 0.35" rpy="0 0 ${PI}" />
+      <origin xyz="0.23 0 0.48" rpy="0 0 ${PI}" />
       <parent link="base_link" />
       <child link="velodyne_mount_link" />
@@ -134,6 +134,6 @@
     <link name="gps_mount_link"/>
     <joint name="gps_joint" type="fixed">
-      <origin xyz="-0.14 -0.20 0.65" rpy="0 0 0" />
-      <parent link="base_link" />
+      <origin xyz="-0.30 0.20 0.125" rpy="0 0 0" />
+      <parent link="top_plate_link" />
       <child link="gps_mount_link" />
     </joint>

Commit message: fix gps mount link.

File: husky_description_mbzirc/urdf/husky.urdf.xacro (robot description, xacro)
@@ -134,5 +134,5 @@
     <link name="gps_mount_link"/>
     <joint name="gps_joint" type="fixed">
-      <origin xyz="-0.24 0.20 0.125" rpy="0 0 0" />
+      <origin xyz="-0.24 0.20 0.145" rpy="0 0 0" />
       <parent link="top_plate_link" />
       <child link="gps_mount_link" />
